File: PONG_Display/IOinterface.sch (KiCad schematic (older format))
At the start: 5 parts

Commit message: V2
Parts:
- added J?: ESP_Conn, symbol Connector_Generic:Conn_02x04_Odd_Even
- added J?: ESP_Prog_Conn, symbol Connector_Generic:Conn_01x04
- added J?: PIR_Sensor_Conn, symbol Connector_Generic:Conn_01x03
Connections:
- net +12V: now reaches J?.1 (Pin_1)
- net +12V: now also J?.1 (Pin_1)
- net LED_DATA: now reaches J?.2 (Pin_2)
- net GND: now reaches J?.3 (Pin_3)
- net GND: now also J?.10 (GND), J?.2 (Pin_2), J?.3 (Pin_3), J?.4 (GND), J?.6 (GND), J?.8 (GND), J?.2 (Pin_2), J?.3 (Pin_3), J?.8 (Pin_8)
- net +5V: now reaches J?.1 (Pin_1)
- net +5V: now also J?.2 (VCC), J?.1 (Pin_1)
- net DHT22_DATA: now reaches J?.2 (Pin_2)
- net LIGHT_SENSOR_IN: now reaches J?.1 (Pin_1)
- net LIGHT_SENSOR_OUT: now reaches J?.2 (Pin_2)
- net uC_MOSI: now reaches J?.1 (MOSI)
- net uC_RST: now reaches J?.5 (~RST)
- net uC_SCK: now reaches J?.7 (SCK)
- net uC_MISO: now reaches J?.9 (MISO)
- new net +3.3V: J?.1 (Pin_1), J?.1 (Pin_1)
- new net ESP_CH_PD: J?.5 (Pin_5)
- new net ESP_GPIO0: J?.4 (Pin_4)
- new net ESP_GPIO2: J?.6 (Pin_6)
- new net ESP_RST: J?.3 (Pin_3)
- new net ESP_RX: J?.2 (Pin_2), J?.3 (Pin_3)
- new net ESP_TX: J?.4 (Pin_4), J?.7 (Pin_7)
- new net PIR_OUT: J?.2 (Pin_2)
Other:
- note added: "Interfejs złączy urządzenia"
Changed lines of the file:
@@
 	1    0    0    -1
 $EndComp
+Text GLabel 2300 1850 2    50   Input ~ 0
++12V
+Text GLabel 2300 1950 2    50   Input ~ 0
+GND
+Text GLabel 1950 3950 1    50   Input ~ 0
++5V
+Text GLabel 1950 5250 3    50   Input ~ 0
+GND
+Text GLabel 2700 4450 2    50   BiDi ~ 0
+uC_MISO
+Text GLabel 2700 4550 2    50   BiDi ~ 0
+uC_MOSI
+Text GLabel 2700 4650 2    50   BiDi ~ 0
+uC_SCK
+Text GLabel 2700 4750 2    50   BiDi ~ 0
+uC_RST
+Text GLabel 9400 1700 0    50   Input ~ 0
++12V
+Text GLabel 9400 1800 0    50   Input ~ 0
+LED_DATA
+Text GLabel 9400 1900 0    50   Input ~ 0
+GND
+Wire Wire Line
+	9400 1700 9500 1700
+Wire Wire Line
+	9400 1800 9500 1800
+Wire Wire Line
+	9400 1900 9500 1900
+Wire Wire Line
+	2150 1850 2300 1850
+Wire Wire Line
+	2150 1950 2300 1950
+Wire Wire Line
+	1950 3950 1950 4150
+Wire Wire Line
+	1950 5050 1950 5250
+Wire Wire Line
+	2450 4750 2700 4750
+Wire Wire Line
+	2450 4650 2700 4650
+Wire Wire Line
+	2450 4550 2700 4550
+Wire Wire Line
+	2450 4450 2700 4450
+Text GLabel 9400 3200 0    50   Input ~ 0
++5V
+Text GLabel 9400 3300 0    50   Output ~ 0
+DHT22_DATA
+Text GLabel 9400 3400 0    50   Input ~ 0
+GND
+Wire Wire Line
+	9550 3200 9400 3200
+Wire Wire Line
+	9400 3300 9550 3300
+Wire Wire Line
+	9400 3400 9550 3400
+Text GLabel 9400 4050 0    50   Input ~ 0
+LIGHT_SENSOR_IN
+Text GLabel 9400 4150 0    50   Output ~ 0
+LIGHT_SENSOR_OUT
+Wire Wire Line
+	9400 4050 9550 4050
+Wire Wire Line
+	9400 4150 9550 4150
+Text GLabel 6050 1800 2    50   Input ~ 0
++3.3V
+Text GLabel 6050 1900 2    50   Input ~ 0
+ESP_RST
+Text GLabel 6050 2000 2    50   Input ~ 0
+ESP_CH_PD
+Text GLabel 6050 2100 2    50   BiDi ~ 0
+ESP_TX
+Text GLabel 5300 1800 0    50   BiDi ~ 0
+ESP_RX
+Text GLabel 5300 1900 0    50   BiDi ~ 0
+ESP_GPIO0
+Text GLabel 5300 2000 0    50   BiDi ~ 0
+ESP_GPIO2
+Text GLabel 5300 2100 0    50   Input ~ 0
+GND
+$Comp
+L Connector_Generic:Conn_02x04_Odd_Even J?
+U 1 1 5E819A97
+P 5750 1900
+F 0 "J?" H 5800 2217 50  0000 C CNN
+F 1 "ESP_Conn" H 5800 2126 50  0000 C CNN
+F 2 "" H 5750 1900 50  0001 C CNN
+F 3 "~" H 5750 1900 50  0001 C CNN
+	1    5750 1900
+	-1   0    0    -1
+$EndComp
+Wire Wire Line
+	5950 1800 6050 1800
+Wire Wire Line
+	5950 1900 6050 1900
+Wire Wire Line
+	5950 2000 6050 2000
+Wire Wire Line
+	5950 2100 6050 2100
+Wire Wire Line
+	5300 1800 5450 1800
+Wire Wire Line
+	5300 1900 5450 1900
+Wire Wire Line
+	5450 2000 5300 2000
+Wire Wire Line
+	5300 2100 5450 2100
+$Comp
+L Connector_Generic:Conn_01x04 J?
+U 1 1 5E81D2F5
+P 5700 2750
+F 0 "J?" H 5780 2742 50  0000 L CNN
+F 1 "ESP_Prog_Conn" H 5780 2651 50  0000 L CNN
+F 2 "" H 5700 2750 50  0001 C CNN
+F 3 "~" H 5700 2750 50  0001 C CNN
+	1    5700 2750
+	1    0    0    -1
+$EndComp
+Text GLabel 5350 2650 0    50   Input ~ 0
++3.3V
+Text GLabel 5350 2750 0    50   Input ~ 0
+GND
+Wire Wire Line
+	5350 2650 5500 2650
+Wire Wire Line
+	5350 2750 5500 2750
+Wire Wire Line
+	5350 2850 5500 2850
+Wire Wire Line
+	5350 2950 5500 2950
+Text Notes 7800 7500 0    50   ~ 0
+Interfejs złączy urządzenia
+Text GLabel 5350 2950 0    50   BiDi ~ 0
+ESP_TX
+Text GLabel 5350 2850 0    50   BiDi ~ 0
+ESP_RX
+$Comp
+L Connector_Generic:Conn_01x03 J?
+U 1 1 5E822EF1
+P 9750 4750
+F 0 "J?" H 9830 4792 50  0000 L CNN
+F 1 "PIR_Sensor_Conn" H 9830 4701 50  0000 L CNN
+F 2 "" H 9750 4750 50  0001 C CNN
+F 3 "~" H 9750 4750 50  0001 C CNN
+	1    9750 4750
+	1    0    0    -1
+$EndComp
+Text GLabel 9400 4650 0    50   Input ~ 0
++5V
+Text GLabel 9400 4750 0    50   Output ~ 0
+PIR_OUT
+Text GLabel 9400 4850 0    50   Input ~ 0
+GND
+Wire Wire Line
+	9400 4650 9550 4650
+Wire Wire Line
+	9400 4750 9550 4750
+Wire Wire Line
+	9400 4850 9550 4850
 $EndSCHEMATC
