File: PONG_Display/PONG_Display.sch (KiCad schematic (older format))
At the start: 4 parts

Commit message: po obgadaniu
Other:
- note added: "1)wybór 5V czy 12V\n2)Poziomy logiczne TX i RX\n3)stany na pinach -\n> czy programowo\n4)Jakie piny na GPIO uC\n5)GPIO od ESP czy potrzebne \n6)Jaka prędkość I2C \n->rezystory 2k/10k\n7)Przypisać piny ESP"
- note added: "Wybór 5V czy 12V"
- note removed: "1)Nie przypisany LED_DATA\n\n2)Poziomy logiczne TX i RX\n\n3)Jakie GPIO z klocka \n\n4)Czy pot do przetwornicy\n\n5)5,6,21 pin Atmegi\n\n6)RTC może brać 5V\n\n7)RTC sprawdzić\n\n8)Przypisać piny ESP\n\n9)Reset klocka i ESP ten sam?\n\n10)Omówić klocek\n\n11)Reset ESP\n\n12)Programator ESP\n"
Changed lines of the file:
@@
 EESchema Schematic File Version 4
+LIBS:PONG_Display-cache
 EELAYER 30 0
 EELAYER END
@@
 Text Notes 950  1150 0    197  Italic 39
 To do:\n
-Text Notes 700  4350 0    79   ~ 0
-1)Nie przypisany LED_DATA\n\n2)Poziomy logiczne TX i RX\n\n3)Jakie GPIO z klocka \n\n4)Czy pot do przetwornicy\n\n5)5,6,21 pin Atmegi\n\n6)RTC może brać 5V\n\n7)RTC sprawdzić\n\n8)Przypisać piny ESP\n\n9)Reset klocka i ESP ten sam?\n\n10)Omówić klocek\n\n11)Reset ESP\n\n12)Programator ESP\n
+Text Notes 700  2500 0    79   ~ 0
+1)wybór 5V czy 12V\n2)Poziomy logiczne TX i RX\n3)stany na pinach -\n> czy programowo\n4)Jakie piny na GPIO uC\n5)GPIO od ESP czy potrzebne \n6)Jaka prędkość I2C \n->rezystory 2k/10k\n7)Przypisać piny ESP
+Text Notes 3800 1200 0    394  Italic 79
+Wybór 5V czy 12V
 $EndSCHEMATC

Commit message: jeszcze do przekminienia
Changed lines of the file:
@@
 EESchema Schematic File Version 4
+LIBS:PONG_Display-cache
 EELAYER 30 0
 EELAYER END
@@
 F3 "PIR_SENSOR_OUT" I L 5400 2800 50
 F4 "DHT22_DATA" I L 5400 2650 50
-F5 "ESP_TX" I R 7200 2500 50
-F6 "ESP_RX" I R 7200 2350 50
-F7 "ESP_RST" I R 7200 2950 50
-F8 "LED_DATA" I R 7200 3300 50
+F5 "ESP_RST" I R 7200 2950 50
+F6 "LED_DATA" I R 7200 3300 50
+F7 "ESP_TX_HIGH" I R 7200 2500 50
+F8 "ESP_RX_HIGH" I R 7200 2350 50
 $EndSheet
 Wire Wire Line
@@
 F0 "Moduł WiFi" 50
 F1 "esp.sch" 50
-F2 "ESP_RX" I L 8400 2350 50
-F3 "ESP_TX" I L 8400 2500 50
-F4 "ESP_RST" I L 8400 2950 50
-F5 "ESP_CH_PD" I L 8400 3100 50
-F6 "ESP_GPIO0" I L 8400 2650 50
-F7 "ESP_GPIO2" I L 8400 2800 50
+F2 "ESP_RST" I L 8400 2950 50
+F3 "ESP_CH_PD" I L 8400 3100 50
+F4 "ESP_GPIO0" I L 8400 2650 50
+F5 "ESP_GPIO2" I L 8400 2800 50
+F6 "ESP_RX_HIGH" I L 8400 2350 50
+F7 "ESP_TX_HIGH" I L 8400 2500 50
 $EndSheet
 Text Notes 950  1150 0    197  Italic 39

Commit message: wybrane 5V
Other:
- note removed: "Wybór 5V czy 12V"
Changed lines of the file:
@@
 Text Notes 700  2500 0    79   ~ 0
 1)wybór 5V czy 12V\n2)Poziomy logiczne TX i RX\n3)stany na pinach -\n> czy programowo\n4)Jakie piny na GPIO uC\n5)GPIO od ESP czy potrzebne \n6)Jaka prędkość I2C \n->rezystory 2k/10k\n7)Przypisać piny ESP
-Text Notes 3800 1200 0    394  Italic 79
-Wybór 5V czy 12V
 $EndSCHEMATC
