File: PONG_Display/Power_supply.sch (KiCad schematic (older format))
At the start: 0 parts

Commit message: V2
Parts:
- added C?: 470u, symbol Device:CP
- added C?: 100n, symbol Device:C
- added C?: 10u, symbol Device:C
- added C?: 100n, symbol Device:CP
- added J?: Input_Supply+12V, symbol Connector_Generic:Conn_01x02
- added U?: LD1117S33TR_SOT223, Package_TO_SOT_SMD:SOT-223-3_TabPin2, symbol Regulator_Linear:LD1117S33TR_SOT223
Connections:
- new net +12V: J?.1 (Pin_1)
- new net +3V3: C?.1, C?.1, U?.2 (VO)
- new net +5V: C?.1, C?.1, U?.3 (VI)
- new net GND: C?.2, C?.2, C?.2, C?.2, J?.2 (Pin_2), U?.1 (GND)
Other:
- note added: "Schemat układu zasilania"
Changed lines of the file:
@@
 $Descr A4 11693 8268
 encoding utf-8
-Sheet 3 7
+Sheet 6 6
 Title ""
 Date ""
@@
 Comment4 ""
 $EndDescr
+$Comp
+L Connector_Generic:Conn_01x02 J?
+U 1 1 5E83DA30
+P 1750 1750
+AR Path="/5E80CCDD/5E83DA30" Ref="J?"  Part="1"
+AR Path="/5E80B14C/5E83DA30" Ref="J?"  Part="1"
+AR Path="/5E83DA30" Ref="J?"  Part="1"
+F 0 "J?" H 1668 1967 50  0000 C CNN
+F 1 "Input_Supply+12V" H 1668 1876 50  0000 C CNN
+F 2 "" H 1750 1750 50  0001 C CNN
+F 3 "~" H 1750 1750 50  0001 C CNN
+	1    1750 1750
+	-1   0    0    -1
+$EndComp
+Text Notes 7850 7500 0    50   ~ 0
+Schemat układu zasilania
+$Comp
+L power:+12V #PWR?
+U 1 1 5E85C905
+P 2400 1600
+F 0 "#PWR?" H 2400 1450 50  0001 C CNN
+F 1 "+12V" H 2415 1773 50  0000 C CNN
+F 2 "" H 2400 1600 50  0001 C CNN
+F 3 "" H 2400 1600 50  0001 C CNN
+	1    2400 1600
+	-1   0    0    -1
+$EndComp
+$Comp
+L power:GND #PWR?
+U 1 1 5E85CD82
+P 2400 2000
+F 0 "#PWR?" H 2400 1750 50  0001 C CNN
+F 1 "GND" H 2405 1827 50  0000 C CNN
+F 2 "" H 2400 2000 50  0001 C CNN
+F 3 "" H 2400 2000 50  0001 C CNN
+	1    2400 2000
+	-1   0    0    -1
+$EndComp
+Wire Wire Line
+	2400 1600 2400 1750
+Wire Wire Line
+	2400 1750 1950 1750
+Wire Wire Line
+	2400 1850 2400 2000
+Wire Wire Line
+	2400 1850 1950 1850
+$Comp
+L Regulator_Linear:LD1117S33TR_SOT223 U?
+U 1 1 5E860E17
+P 8200 1650
+F 0 "U?" H 8200 1892 50  0000 C CNN
+F 1 "LD1117S33TR_SOT223" H 8200 1801 50  0000 C CNN
+F 2 "Package_TO_SOT_SMD:SOT-223-3_TabPin2" H 8200 1850 50  0001 C CNN
+F 3 "http://www.st.com/st-web-ui/static/active/en/resource/technical/document/datasheet/CD00000544.pdf" H 8300 1400 50  0001 C CNN
+	1    8200 1650
+	1    0    0    -1
+$EndComp
+$Comp
+L power:GND #PWR?
+U 1 1 5E862C71
+P 8200 2100
+F 0 "#PWR?" H 8200 1850 50  0001 C CNN
+F 1 "GND" H 8205 1927 50  0000 C CNN
+F 2 "" H 8200 2100 50  0001 C CNN
+F 3 "" H 8200 2100 50  0001 C CNN
+	1    8200 2100
+	1    0    0    -1
+$EndComp
+$Comp
+L power:+5V #PWR?
+U 1 1 5E862F46
+P 7000 1500
+F 0 "#PWR?" H 7000 1350 50  0001 C CNN
+F 1 "+5V" H 7015 1673 50  0000 C CNN
+F 2 "" H 7000 1500 50  0001 C CNN
+F 3 "" H 7000 1500 50  0001 C CNN
+	1    7000 1500
+	1    0    0    -1
+$EndComp
+$Comp
+L power:+3.3V #PWR?
+U 1 1 5E8636C0
+P 9300 1500
+F 0 "#PWR?" H 9300 1350 50  0001 C CNN
+F 1 "+3.3V" H 9315 1673 50  0000 C CNN
+F 2 "" H 9300 1500 50  0001 C CNN
+F 3 "" H 9300 1500 50  0001 C CNN
+	1    9300 1500
+	1    0    0    -1
+$EndComp
+Wire Wire Line
+	8200 1950 8200 2100
+Wire Wire Line
+	8500 1650 8700 1650
+Wire Wire Line
+	9300 1650 9300 1500
+Wire Wire Line
+	7000 1500 7000 1650
+Wire Wire Line
+	7000 1650 7200 1650
+$Comp
+L Device:CP C?
+U 1 1 5E864BF2
+P 7200 1900
+F 0 "C?" H 7318 1946 50  0000 L CNN
+F 1 "470u" H 7318 1855 50  0000 L CNN
+F 2 "" H 7238 1750 50  0001 C CNN
+F 3 "~" H 7200 1900 50  0001 C CNN
+	1    7200 1900
+	1    0    0    -1
+$EndComp
+$Comp
+L Device:C C?
+U 1 1 5E86541E
+P 7600 1900
+F 0 "C?" H 7715 1946 50  0000 L CNN
+F 1 "100n" H 7715 1855 50  0000 L CNN
+F 2 "" H 7638 1750 50  0001 C CNN
+F 3 "~" H 7600 1900 50  0001 C CNN
+	1    7600 1900
+	1    0    0    -1
+$EndComp
+$Comp
+L Device:C C?
+U 1 1 5E8658D9
+P 8700 1900
+F 0 "C?" H 8815 1946 50  0000 L CNN
+F 1 "10u" H 8815 1855 50  0000 L CNN
+F 2 "" H 8738 1750 50  0001 C CNN
+F 3 "~" H 8700 1900 50  0001 C CNN
+	1    8700 1900
+	1    0    0    -1
+$EndComp
+$Comp
+L Device:CP C?
+U 1 1 5E8660CC
+P 9050 1900
+F 0 "C?" H 9168 1946 50  0000 L CNN
+F 1 "100n" H 9168 1855 50  0000 L CNN
+F 2 "" H 9088 1750 50  0001 C CNN
+F 3 "~" H 9050 1900 50  0001 C CNN
+	1    9050 1900
+	1    0    0    -1
+$EndComp
+$Comp
+L power:GND #PWR?
+U 1 1 5E866491
+P 7200 2150
+F 0 "#PWR?" H 7200 1900 50  0001 C CNN
+F 1 "GND" H 7205 1977 50  0000 C CNN
+F 2 "" H 7200 2150 50  0001 C CNN
+F 3 "" H 7200 2150 50  0001 C CNN
+	1    7200 2150
+	1    0    0    -1
+$EndComp
+$Comp
+L power:GND #PWR?
+U 1 1 5E8668A3
+P 7600 2150
+F 0 "#PWR?" H 7600 1900 50  0001 C CNN
+F 1 "GND" H 7605 1977 50  0000 C CNN
+F 2 "" H 7600 2150 50  0001 C CNN
+F 3 "" H 7600 2150 50  0001 C CNN
+	1    7600 2150
+	1    0    0    -1
+$EndComp
+$Comp
+L power:GND #PWR?
+U 1 1 5E866DAE
+P 8700 2150
+F 0 "#PWR?" H 8700 1900 50  0001 C CNN
+F 1 "GND" H 8705 1977 50  0000 C CNN
+F 2 "" H 8700 2150 50  0001 C CNN
+F 3 "" H 8700 2150 50  0001 C CNN
+	1    8700 2150
+	1    0    0    -1
+$EndComp
+$Comp
+L power:GND #PWR?
+U 1 1 5E8670D0
+P 9050 2150
+F 0 "#PWR?" H 9050 1900 50  0001 C CNN
+F 1 "GND" H 9055 1977 50  0000 C CNN
+F 2 "" H 9050 2150 50  0001 C CNN
+F 3 "" H 9050 2150 50  0001 C CNN
+	1    9050 2150
+	1    0    0    -1
+$EndComp
+Wire Wire Line
+	9050 2050 9050 2150
+Wire Wire Line
+	8700 2050 8700 2150
+Wire Wire Line
+	7600 2050 7600 2150
+Wire Wire Line
+	7200 2050 7200 2150
+Wire Wire Line
+	7200 1650 7200 1750
+Connection ~ 7200 1650
+Wire Wire Line
+	7200 1650 7600 1650
+Wire Wire Line
+	7600 1650 7600 1750
+Connection ~ 7600 1650
+Wire Wire Line
+	7600 1650 7900 1650
+Wire Wire Line
+	8700 1650 8700 1750
+Connection ~ 8700 1650
+Wire Wire Line
+	8700 1650 9050 1650
+Wire Wire Line
+	9050 1650 9050 1750
+Connection ~ 9050 1650
+Wire Wire Line
+	9050 1650 9300 1650
 $EndSCHEMATC

Commit message: V3
Parts:
- added C?: 1u, symbol Device:CP
- added C? (x4): 10u, symbol Device:CP
- added C?: 100n, symbol Device:C
- added D?: RED_LED, symbol Device:LED
- added D?: YELLOW_LED, symbol Device:LED
- added D?: GREEN_LED, symbol Device:LED
- added L?: 22u, symbol Device:L
- added R?: 470R, symbol Device:R
- added R?: 82R, symbol Device:R
- added R?: 5R, symbol Device:R
- added RV?: 100k, symbol Device:R_POT
- added U?: MCP16311MS, Package_SO:MSOP-8_3x3mm_P0.65mm, symbol Regulator_Switching:MCP16311MS
Connections:
- net +12V: now also C?.1, C?.1, R?.1, U?.3 (EN), U?.4 (Vin)
- net +3V3: now also R?.1
- net +5V: now also C?.1, C?.1, L?.2, R?.1
- net GND: now also C?.2, C?.2, C?.2, C?.2, C?.2, D?.1 (K), D?.1 (K), D?.1 (K), RV?.1, U?.5 (PGND), U?.8 (AGND)
- new net: D?.2 (A), R?.2 (x3)
- new net: RV?.2, U?.1 (Vfb)
- new net: C?.1, U?.2 (Vcc)
- new net: C?.2, L?.1, RV?.3, U?.6 (SW)
- new net: C?.1, U?.7 (BOOST)
Other:
- note added: "Przetwornica DC/DC 12V/5V"
- note added: "Stabilizator LDO 3.3V"
- note added: "Wskaźnik działania zasilania"
- note added: "Złącze zasilania CON WAGO 580 x2"
- moved on the sheet: C?, U?

Commit message: Dodane footprinty
Parts:
- C10, C4, C6, C7: renamed from C?; footprint (none) -> Capacitor_THT:CP_Axial_L10.0mm_D4.5mm_P15.00mm_Horizontal
- C11, C5, C9: renamed from C?; footprint (none) -> Capacitor_SMD:C_1206_3216Metric_Pad1.42x1.75mm_HandSolder
- C2, C3, C8: renamed from C?; footprint (none) -> Capacitor_THT:CP_Axial_L10.0mm_D6.0mm_P15.00mm_Horizontal
- D1, D2, D3: renamed from D?; footprint (none) -> Diode_SMD:D_1206_3216Metric_Pad1.42x1.75mm_HandSolder
- R2, R3, R4: renamed from R?; footprint (none) -> Resistor_SMD:R_1206_3216Metric_Pad1.42x1.75mm_HandSolder
- RV1: renamed from RV?; footprint (none) -> Resistor_SMD:R_1206_3216Metric_Pad1.42x1.75mm_HandSolder
- gave numbers to parts that had none: 4
Changed lines of the file:
@@
 P 1750 1750
 AR Path="/5E80CCDD/5E83DA30" Ref="J?"  Part="1"
-AR Path="/5E80B14C/5E83DA30" Ref="J?"  Part="1"
+AR Path="/5E80B14C/5E83DA30" Ref="J2"  Part="1"
 AR Path="/5E83DA30" Ref="J?"  Part="1"
-F 0 "J?" H 1668 1967 50  0000 C CNN
+F 0 "J2" H 1668 1967 50  0000 C CNN
 F 1 "Input_Supply+12V" H 1668 1876 50  0000 C CNN
 F 2 "" H 1750 1750 50  0001 C CNN
@@
 	2400 1850 1950 1850
 $Comp
-L Regulator_Linear:LD1117S33TR_SOT223 U?
+L Regulator_Linear:LD1117S33TR_SOT223 U3
 U 1 1 5E860E17
 P 8300 1650
-F 0 "U?" H 8300 1892 50  0000 C CNN
+F 0 "U3" H 8300 1892 50  0000 C CNN
 F 1 "LD1117S33TR_SOT223" H 8300 1801 50  0000 C CNN
 F 2 "Package_TO_SOT_SMD:SOT-223-3_TabPin2" H 8300 1850 50  0001 C CNN
@@
 	7100 1650 7300 1650
 $Comp
-L Device:CP C?
+L Device:CP C8
 U 1 1 5E864BF2
 P 7300 1900
-F 0 "C?" H 7418 1946 50  0000 L CNN
+F 0 "C8" H 7418 1946 50  0000 L CNN
 F 1 "470u" H 7418 1855 50  0000 L CNN
-F 2 "" H 7338 1750 50  0001 C CNN
+F 2 "Capacitor_THT:CP_Axial_L10.0mm_D6.0mm_P15.00mm_Horizontal" H 7338 1750 50  0001 C CNN
 F 3 "~" H 7300 1900 50  0001 C CNN
 	1    7300 1900
@@
 $EndComp
 $Comp
-L Device:C C?
+L Device:C C9
 U 1 1 5E86541E
 P 7700 1900
-F 0 "C?" H 7815 1946 50  0000 L CNN
+F 0 "C9" H 7815 1946 50  0000 L CNN
 F 1 "100n" H 7815 1855 50  0000 L CNN
-F 2 "" H 7738 1750 50  0001 C CNN
+F 2 "Capacitor_SMD:C_1206_3216Metric_Pad1.42x1.75mm_HandSolder" H 7738 1750 50  0001 C CNN
 F 3 "~" H 7700 1900 50  0001 C CNN
 	1    7700 1900
@@
 $EndComp
 $Comp
-L Device:C C?
+L Device:C C10
 U 1 1 5E8658D9
 P 8800 1900
-F 0 "C?" H 8915 1946 50  0000 L CNN
+F 0 "C10" H 8915 1946 50  0000 L CNN
 F 1 "10u" H 8915 1855 50  0000 L CNN
-F 2 "" H 8838 1750 50  0001 C CNN
+F 2 "Capacitor_THT:CP_Axial_L10.0mm_D4.5mm_P15.00mm_Horizontal" H 8838 1750 50  0001 C CNN
 F 3 "~" H 8800 1900 50  0001 C CNN
 	1    8800 1900
@@
 $EndComp
 $Comp
-L Device:CP C?
+L Device:CP C11
 U 1 1 5E8660CC
 P 9150 1900
-F 0 "C?" H 9268 1946 50  0000 L CNN
+F 0 "C11" H 9268 1946 50  0000 L CNN
 F 1 "100n" H 9268 1855 50  0000 L CNN
-F 2 "" H 9188 1750 50  0001 C CNN
+F 2 "Capacitor_SMD:C_1206_3216Metric_Pad1.42x1.75mm_HandSolder" H 9188 1750 50  0001 C CNN
 F 3 "~" H 9150 1900 50  0001 C CNN
 	1    9150 1900
@@
 $EndComp
 $Comp
-L Device:R R?
+L Device:R R2
 U 1 1 5E8EF261
 P 3850 1850
-F 0 "R?" H 3920 1896 50  0000 L CNN
+F 0 "R2" H 3920 1896 50  0000 L CNN
 F 1 "470R" H 3920 1805 50  0000 L CNN
-F 2 "" V 3780 1850 50  0001 C CNN
+F 2 "Resistor_SMD:R_1206_3216Metric_Pad1.42x1.75mm_HandSolder" V 3780 1850 50  0001 C CNN
 F 3 "~" H 3850 1850 50  0001 C CNN
 	1    3850 1850
@@
 $EndComp
 $Comp
-L Device:R R?
+L Device:R R3
 U 1 1 5E8EF860
 P 4500 1850
-F 0 "R?" H 4570 1896 50  0000 L CNN
+F 0 "R3" H 4570 1896 50  0000 L CNN
 F 1 "82R" H 4570 1805 50  0000 L CNN
-F 2 "" V 4430 1850 50  0001 C CNN
+F 2 "Resistor_SMD:R_1206_3216Metric_Pad1.42x1.75mm_HandSolder" V 4430 1850 50  0001 C CNN
 F 3 "~" H 4500 1850 50  0001 C CNN
 	1    4500 1850
@@
 $EndComp
 $Comp
-L Device:R R?
+L Device:R R4
 U 1 1 5E8F00A4
 P 5200 1850
-F 0 "R?" H 5270 1896 50  0000 L CNN
+F 0 "R4" H 5270 1896 50  0000 L CNN
 F 1 "5R" H 5270 1805 50  0000 L CNN
-F 2 "" V 5130 1850 50  0001 C CNN
+F 2 "Resistor_SMD:R_1206_3216Metric_Pad1.42x1.75mm_HandSolder" V 5130 1850 50  0001 C CNN
 F 3 "~" H 5200 1850 50  0001 C CNN
 	1    5200 1850
@@
 $EndComp
 $Comp
-L Device:LED D?
+L Device:LED D1
 U 1 1 5E8F075F
 P 3850 2300
-F 0 "D?" V 3889 2182 50  0000 R CNN
+F 0 "D1" V 3889 2182 50  0000 R CNN
 F 1 "RED_LED" V 3798 2182 50  0000 R CNN
-F 2 "" H 3850 2300 50  0001 C CNN
+F 2 "Diode_SMD:D_1206_3216Metric_Pad1.42x1.75mm_HandSolder" H 3850 2300 50  0001 C CNN
 F 3 "~" H 3850 2300 50  0001 C CNN
 	1    3850 2300
@@
 $EndComp
 $Comp
-L Device:LED D?
+L Device:LED D2
 U 1 1 5E8F11B2
 P 4500 2300
-F 0 "D?" V 4539 2183 50  0000 R CNN
+F 0 "D2" V 4539 2183 50  0000 R CNN
 F 1 "YELLOW_LED" V 4448 2183 50  0000 R CNN
-F 2 "" H 4500 2300 50  0001 C CNN
+F 2 "Diode_SMD:D_1206_3216Metric_Pad1.42x1.75mm_HandSolder" H 4500 2300 50  0001 C CNN
 F 3 "~" H 4500 2300 50  0001 C CNN
 	1    4500 2300
@@
 $EndComp
 $Comp
-L Device:LED D?
+L Device:LED D3
 U 1 1 5E8F1C29
 P 5200 2300
-F 0 "D?" V 5239 2182 50  0000 R CNN
+F 0 "D3" V 5239 2182 50  0000 R CNN
 F 1 "GREEN_LED" V 5148 2182 50  0000 R CNN
-F 2 "" H 5200 2300 50  0001 C CNN
+F 2 "Diode_SMD:D_1206_3216Metric_Pad1.42x1.75mm_HandSolder" H 5200 2300 50  0001 C CNN
 F 3 "~" H 5200 2300 50  0001 C CNN
 	1    5200 2300
@@
 Przetwornica DC/DC 12V/5V
 $Comp
-L Regulator_Switching:MCP16311MS U?
+L Regulator_Switching:MCP16311MS U2
 U 1 1 5E9D393E
 P 3250 5700
-F 0 "U?" H 3250 6267 50  0000 C CNN
+F 0 "U2" H 3250 6267 50  0000 C CNN
 F 1 "MCP16311MS" H 3250 6176 50  0000 C CNN
 F 2 "Package_SO:MSOP-8_3x3mm_P0.65mm" H 3400 5450 50  0001 L CNN
@@
 $EndComp
 $Comp
-L Device:CP C?
+L Device:CP C4
 U 1 1 5E9D4E40
 P 2700 6000
-F 0 "C?" H 2818 6046 50  0000 L CNN
+F 0 "C4" H 2818 6046 50  0000 L CNN
 F 1 "1u" H 2818 5955 50  0000 L CNN
-F 2 "" H 2738 5850 50  0001 C CNN
+F 2 "Capacitor_THT:CP_Axial_L10.0mm_D4.5mm_P15.00mm_Horizontal" H 2738 5850 50  0001 C CNN
 F 3 "~" H 2700 6000 50  0001 C CNN
 	1    2700 6000
@@
 $EndComp
 $Comp
-L Device:CP C?
+L Device:CP C3
 U 1 1 5E9D7DF8
 P 2350 5650
-F 0 "C?" H 2468 5696 50  0000 L CNN
+F 0 "C3" H 2468 5696 50  0000 L CNN
 F 1 "10u" H 2468 5605 50  0000 L CNN
-F 2 "" H 2388 5500 50  0001 C CNN
+F 2 "Capacitor_THT:CP_Axial_L10.0mm_D6.0mm_P15.00mm_Horizontal" H 2388 5500 50  0001 C CNN
 F 3 "~" H 2350 5650 50  0001 C CNN
 	1    2350 5650
@@
 $EndComp
 $Comp
-L Device:CP C?
+L Device:CP C2
 U 1 1 5E9D9473
 P 2000 5650
-F 0 "C?" H 2118 5696 50  0000 L CNN
+F 0 "C2" H 2118 5696 50  0000 L CNN
 F 1 "10u" H 2118 5605 50  0000 L CNN
-F 2 "" H 2038 5500 50  0001 C CNN
+F 2 "Capacitor_THT:CP_Axial_L10.0mm_D6.0mm_P15.00mm_Horizontal" H 2038 5500 50  0001 C CNN
 F 3 "~" H 2000 5650 50  0001 C CNN
 	1    2000 5650
@@
 	2700 5500 2350 5500
 $Comp
-L Device:C C?
+L Device:C C5
 U 1 1 5E9DD7F1
 P 3950 5400
-F 0 "C?" V 4202 5400 50  0000 C CNN
+F 0 "C5" V 4202 5400 50  0000 C CNN
 F 1 "100n" V 4111 5400 50  0000 C CNN
-F 2 "" H 3988 5250 50  0001 C CNN
+F 2 "Capacitor_SMD:C_1206_3216Metric_Pad1.42x1.75mm_HandSolder" H 3988 5250 50  0001 C CNN
 F 3 "~" H 3950 5400 50  0001 C CNN
 	1    3950 5400
@@
 $EndComp
 $Comp
-L Device:CP C?
+L Device:CP C6
 U 1 1 5E9E1C89
 P 4950 5650
-F 0 "C?" H 5068 5696 50  0000 L CNN
+F 0 "C6" H 5068 5696 50  0000 L CNN
 F 1 "10u" H 5068 5605 50  0000 L CNN
-F 2 "" H 4988 5500 50  0001 C CNN
+F 2 "Capacitor_THT:CP_Axial_L10.0mm_D4.5mm_P15.00mm_Horizontal" H 4988 5500 50  0001 C CNN
 F 3 "~" H 4950 5650 50  0001 C CNN
 	1    4950 5650
@@
 $EndComp
 $Comp
-L Device:CP C?
+L Device:CP C7
 U 1 1 5E9E2732
 P 5350 5650
-F 0 "C?" H 5468 5696 50  0000 L CNN
+F 0 "C7" H 5468 5696 50  0000 L CNN
 F 1 "10u" H 5468 5605 50  0000 L CNN
-F 2 "" H 5388 5500 50  0001 C CNN
+F 2 "Capacitor_THT:CP_Axial_L10.0mm_D4.5mm_P15.00mm_Horizontal" H 5388 5500 50  0001 C CNN
 F 3 "~" H 5350 5650 50  0001 C CNN
 	1    5350 5650
@@
 $EndComp
 $Comp
-L Device:L L?
+L Device:L L1
 U 1 1 5E9E3110
 P 4650 5500
-F 0 "L?" V 4840 5500 50  0000 C CNN
+F 0 "L1" V 4840 5500 50  0000 C CNN
 F 1 "22u" V 4749 5500 50  0000 C CNN
 F 2 "" H 4650 5500 50  0001 C CNN
@@
 	5350 5800 5350 5900
 $Comp
-L Device:R_POT RV?
+L Device:R_POT RV1
 U 1 1 5E9F22F8
 P 4300 5700
-F 0 "RV?" H 4230 5654 50  0000 R CNN
+F 0 "RV1" H 4230 5654 50  0000 R CNN
 F 1 "100k" H 4230 5745 50  0000 R CNN
-F 2 "" H 4300 5700 50  0001 C CNN
+F 2 "Resistor_SMD:R_1206_3216Metric_Pad1.42x1.75mm_HandSolder" H 4300 5700 50  0001 C CNN
 F 3 "~" H 4300 5700 50  0001 C CNN
 	1    4300 5700

Commit message: v2
Parts:
- C10, C6, C7: footprint Capacitor_THT:CP_Axial_L10.0mm_D4.5mm_P15.00mm_Horizontal -> Capacitor_THT:CP_Radial_D6.3mm_P2.50mm
- C2, C3: footprint Capacitor_THT:CP_Axial_L10.0mm_D6.0mm_P15.00mm_Horizontal -> Capacitor_THT:CP_Radial_D6.3mm_P2.50mm
- C8: footprint Capacitor_THT:CP_Axial_L10.0mm_D6.0mm_P15.00mm_Horizontal -> Capacitor_SMD:C_Elec_10x10.2
- L1: footprint (none) -> Inductor_SMD:L_12x12mm_H4.5mm
Changed lines of the file:
@@
 F 0 "C8" H 7418 1946 50  0000 L CNN
 F 1 "470u" H 7418 1855 50  0000 L CNN
-F 2 "Capacitor_THT:CP_Axial_L10.0mm_D6.0mm_P15.00mm_Horizontal" H 7338 1750 50  0001 C CNN
+F 2 "Capacitor_SMD:C_Elec_10x10.2" H 7338 1750 50  0001 C CNN
 F 3 "~" H 7300 1900 50  0001 C CNN
 	1    7300 1900
@@
 F 0 "C10" H 8915 1946 50  0000 L CNN
 F 1 "10u" H 8915 1855 50  0000 L CNN
-F 2 "Capacitor_THT:CP_Axial_L10.0mm_D4.5mm_P15.00mm_Horizontal" H 8838 1750 50  0001 C CNN
+F 2 "Capacitor_THT:CP_Radial_D6.3mm_P2.50mm" H 8838 1750 50  0001 C CNN
 F 3 "~" H 8800 1900 50  0001 C CNN
 	1    8800 1900
@@
 F 0 "C3" H 2468 5696 50  0000 L CNN
 F 1 "10u" H 2468 5605 50  0000 L CNN
-F 2 "Capacitor_THT:CP_Axial_L10.0mm_D6.0mm_P15.00mm_Horizontal" H 2388 5500 50  0001 C CNN
+F 2 "Capacitor_THT:CP_Radial_D6.3mm_P2.50mm" H 2388 5500 50  0001 C CNN
 F 3 "~" H 2350 5650 50  0001 C CNN
 	1    2350 5650
@@
 F 0 "C2" H 2118 5696 50  0000 L CNN
 F 1 "10u" H 2118 5605 50  0000 L CNN
-F 2 "Capacitor_THT:CP_Axial_L10.0mm_D6.0mm_P15.00mm_Horizontal" H 2038 5500 50  0001 C CNN
+F 2 "Capacitor_THT:CP_Radial_D6.3mm_P2.50mm" H 2038 5500 50  0001 C CNN
 F 3 "~" H 2000 5650 50  0001 C CNN
 	1    2000 5650
@@
 F 0 "C6" H 5068 5696 50  0000 L CNN
 F 1 "10u" H 5068 5605 50  0000 L CNN
-F 2 "Capacitor_THT:CP_Axial_L10.0mm_D4.5mm_P15.00mm_Horizontal" H 4988 5500 50  0001 C CNN
+F 2 "Capacitor_THT:CP_Radial_D6.3mm_P2.50mm" H 4988 5500 50  0001 C CNN
 F 3 "~" H 4950 5650 50  0001 C CNN
 	1    4950 5650
@@
 F 0 "C7" H 5468 5696 50  0000 L CNN
 F 1 "10u" H 5468 5605 50  0000 L CNN
-F 2 "Capacitor_THT:CP_Axial_L10.0mm_D4.5mm_P15.00mm_Horizontal" H 5388 5500 50  0001 C CNN
+F 2 "Capacitor_THT:CP_Radial_D6.3mm_P2.50mm" H 5388 5500 50  0001 C CNN
 F 3 "~" H 5350 5650 50  0001 C CNN
 	1    5350 5650
@@
 F 0 "L1" V 4840 5500 50  0000 C CNN
 F 1 "22u" V 4749 5500 50  0000 C CNN
-F 2 "" H 4650 5500 50  0001 C CNN
+F 2 "Inductor_SMD:L_12x12mm_H4.5mm" H 4650 5500 50  0001 C CNN
 F 3 "~" H 4650 5500 50  0001 C CNN
 	1    4650 5500

Commit message: Drobne zmiany
Parts:
- J2: footprint (none) -> TerminalBlock:TerminalBlock_bornier-2_P5.08mm
Other:
- moved on the sheet: C11
Changed lines of the file:
@@
 F 0 "J2" H 1668 1967 50  0000 C CNN
 F 1 "Input_Supply+12V" H 1668 1876 50  0000 C CNN
-F 2 "" H 1750 1750 50  0001 C CNN
+F 2 "TerminalBlock:TerminalBlock_bornier-2_P5.08mm" H 1750 1750 50  0001 C CNN
 F 3 "~" H 1750 1750 50  0001 C CNN
 	1    1750 1750
@@
 L Device:CP C11
 U 1 1 5E8660CC
-P 9150 1900
-F 0 "C11" H 9268 1946 50  0000 L CNN
-F 1 "100n" H 9268 1855 50  0000 L CNN
-F 2 "Capacitor_SMD:C_1206_3216Metric_Pad1.42x1.75mm_HandSolder" H 9188 1750 50  0001 C CNN
-F 3 "~" H 9150 1900 50  0001 C CNN
-	1    9150 1900
+P 9200 1900
+F 0 "C11" H 9318 1946 50  0000 L CNN
+F 1 "100n" H 9318 1855 50  0000 L CNN
+F 2 "Capacitor_SMD:C_1206_3216Metric_Pad1.42x1.75mm_HandSolder" H 9238 1750 50  0001 C CNN
+F 3 "~" H 9200 1900 50  0001 C CNN
+	1    9200 1900
 	1    0    0    -1
 $EndComp
@@
 L power:GND #PWR0114
 U 1 1 5E8670D0
-P 9150 2150
-F 0 "#PWR0114" H 9150 1900 50  0001 C CNN
-F 1 "GND" H 9155 1977 50  0000 C CNN
-F 2 "" H 9150 2150 50  0001 C CNN
-F 3 "" H 9150 2150 50  0001 C CNN
-	1    9150 2150
-	1    0    0    -1
-$EndComp
-Wire Wire Line
-	9150 2050 9150 2150
+P 9200 2150
+F 0 "#PWR0114" H 9200 1900 50  0001 C CNN
+F 1 "GND" H 9205 1977 50  0000 C CNN
+F 2 "" H 9200 2150 50  0001 C CNN
+F 3 "" H 9200 2150 50  0001 C CNN
+	1    9200 2150
+	1    0    0    -1
+$EndComp
+Wire Wire Line
+	9200 2050 9200 2150
 Wire Wire Line
 	8800 2050 8800 2150
@@
 Connection ~ 8800 1650
 Wire Wire Line
-	8800 1650 9150 1650
-Wire Wire Line
-	9150 1650 9150 1750
-Connection ~ 9150 1650
-Wire Wire Line
-	9150 1650 9400 1650
+	8800 1650 9200 1650
+Wire Wire Line
+	9200 1650 9200 1750
+Connection ~ 9200 1650
+Wire Wire Line
+	9200 1650 9400 1650
 $Comp
 L power:+12V #PWR0115

Commit message: Zmiany
Parts:
- R3: value 82R -> 150R
- R4: value 5R -> 5R1
Connections:
- net +5V: now also RV1.3
- net at C5.2, L1.1, U2.6 (SW): no longer RV1.3
Other:
- moved on the sheet: L1, RV1
Changed lines of the file:
@@
 P 4500 1850
 F 0 "R3" H 4570 1896 50  0000 L CNN
-F 1 "82R" H 4570 1805 50  0000 L CNN
+F 1 "150R" H 4570 1805 50  0000 L CNN
 F 2 "Resistor_SMD:R_1206_3216Metric_Pad1.42x1.75mm_HandSolder" V 4430 1850 50  0001 C CNN
 F 3 "~" H 4500 1850 50  0001 C CNN
@@
 P 5200 1850
 F 0 "R4" H 5270 1896 50  0000 L CNN
-F 1 "5R" H 5270 1805 50  0000 L CNN
+F 1 "5R1" H 5270 1805 50  0000 L CNN
 F 2 "Resistor_SMD:R_1206_3216Metric_Pad1.42x1.75mm_HandSolder" V 5130 1850 50  0001 C CNN
 F 3 "~" H 5200 1850 50  0001 C CNN
@@
 $EndComp
 $Comp
-L Device:L L1
-U 1 1 5E9E3110
-P 4650 5500
-F 0 "L1" V 4840 5500 50  0000 C CNN
-F 1 "22u" V 4749 5500 50  0000 C CNN
-F 2 "Inductor_SMD:L_12x12mm_H4.5mm" H 4650 5500 50  0001 C CNN
-F 3 "~" H 4650 5500 50  0001 C CNN
-	1    4650 5500
-	0    -1   -1   0
-$EndComp
-$Comp
 L power:GND #PWR0122
 U 1 1 5E9E41EC
@@
 L power:GND #PWR0125
 U 1 1 5E9E641F
-P 4300 5950
-F 0 "#PWR0125" H 4300 5700 50  0001 C CNN
-F 1 "GND" H 4305 5777 50  0000 C CNN
-F 2 "" H 4300 5950 50  0001 C CNN
-F 3 "" H 4300 5950 50  0001 C CNN
-	1    4300 5950
+P 4600 5950
+F 0 "#PWR0125" H 4600 5700 50  0001 C CNN
+F 1 "GND" H 4605 5777 50  0000 C CNN
+F 2 "" H 4600 5950 50  0001 C CNN
+F 3 "" H 4600 5950 50  0001 C CNN
+	1    4600 5950
 	1    0    0    -1
 $EndComp
@@
 L power:+5V #PWR0128
 U 1 1 5E9E832A
-P 5800 5350
-F 0 "#PWR0128" H 5800 5200 50  0001 C CNN
-F 1 "+5V" H 5815 5523 50  0000 C CNN
-F 2 "" H 5800 5350 50  0001 C CNN
-F 3 "" H 5800 5350 50  0001 C CNN
-	1    5800 5350
+P 4950 5350
+F 0 "#PWR0128" H 4950 5200 50  0001 C CNN
+F 1 "+5V" H 4965 5523 50  0000 C CNN
+F 2 "" H 4950 5350 50  0001 C CNN
+F 3 "" H 4950 5350 50  0001 C CNN
+	1    4950 5350
 	1    0    0    -1
 $EndComp
@@
 	4100 5500 3650 5500
 Wire Wire Line
-	4100 5500 4300 5500
-Connection ~ 4100 5500
-Wire Wire Line
-	4800 5500 4950 5500
-Wire Wire Line
 	4950 5500 5350 5500
-Connection ~ 4950 5500
-Wire Wire Line
-	5350 5500 5800 5500
-Wire Wire Line
-	5800 5500 5800 5350
-Connection ~ 5350 5500
+Wire Wire Line
+	4950 5500 4950 5350
 Wire Wire Line
 	4950 5800 4950 5900
@@
 L Device:R_POT RV1
 U 1 1 5E9F22F8
-P 4300 5700
-F 0 "RV1" H 4230 5654 50  0000 R CNN
-F 1 "100k" H 4230 5745 50  0000 R CNN
-F 2 "Resistor_SMD:R_1206_3216Metric_Pad1.42x1.75mm_HandSolder" H 4300 5700 50  0001 C CNN
-F 3 "~" H 4300 5700 50  0001 C CNN
-	1    4300 5700
+P 4600 5700
+F 0 "RV1" H 4530 5654 50  0000 R CNN
+F 1 "100k" H 4530 5745 50  0000 R CNN
+F 2 "Resistor_SMD:R_1206_3216Metric_Pad1.42x1.75mm_HandSolder" H 4600 5700 50  0001 C CNN
+F 3 "~" H 4600 5700 50  0001 C CNN
+	1    4600 5700
 	-1   0    0    1
 $EndComp
 Wire Wire Line
-	3650 5700 4150 5700
-Wire Wire Line
-	4300 5550 4300 5500
-Connection ~ 4300 5500
-Wire Wire Line
-	4300 5500 4500 5500
-Wire Wire Line
-	4300 5950 4300 5850
+	3650 5700 4450 5700
+Wire Wire Line
+	4600 5550 4600 5500
+Wire Wire Line
+	4600 5950 4600 5850
 Wire Wire Line
 	2000 5800 2000 5950
@@
 Wire Wire Line
 	3350 6000 3350 6100
+Connection ~ 4950 5500
+$Comp
+L Device:L L1
+U 1 1 5E9E3110
+P 4350 5500
+F 0 "L1" V 4540 5500 50  0000 C CNN
+F 1 "22u" V 4449 5500 50  0000 C CNN
+F 2 "Inductor_SMD:L_12x12mm_H4.5mm" H 4350 5500 50  0001 C CNN
+F 3 "~" H 4350 5500 50  0001 C CNN
+	1    4350 5500
+	0    -1   -1   0
+$EndComp
+Wire Wire Line
+	4600 5500 4950 5500
+Wire Wire Line
+	4500 5500 4600 5500
+Connection ~ 4600 5500
+Wire Wire Line
+	4100 5500 4200 5500
+Connection ~ 4100 5500
 $EndSCHEMATC
