File: PONG_Display/Power_supply.sch (KiCad schematic (older format))
At the start: 22 parts, among them J2 Input_Supply+12V, U2 MCP16311MS, U3 LD1117S33TR_SOT223

Commit message: Zmianaa
Parts:
- F1: renamed from F?; footprint (none) -> Fuse:Fuseholder_Cylinder-5x20mm_Schurter_FAB_0031-355x_Horizontal_Closed
- RV1: footprint Resistor_SMD:R_1206_3216Metric_Pad1.42x1.75mm_HandSolder -> Potentiometer_THT:Potentiometer_Piher_PT-6-V_Vertical
Changed lines of the file:
@@
 F 0 "RV1" H 4530 5654 50  0000 R CNN
 F 1 "100k" H 4530 5745 50  0000 R CNN
-F 2 "Resistor_SMD:R_1206_3216Metric_Pad1.42x1.75mm_HandSolder" H 4600 5700 50  0001 C CNN
+F 2 "Potentiometer_THT:Potentiometer_Piher_PT-6-V_Vertical" H 4600 5700 50  0001 C CNN
 F 3 "~" H 4600 5700 50  0001 C CNN
 	1    4600 5700
@@
 Connection ~ 4100 5500
 $Comp
-L Device:Fuse F?
+L Device:Fuse F1
 U 1 1 5EA039B3
 P 2400 1750
-F 0 "F?" V 2203 1750 50  0000 C CNN
+F 0 "F1" V 2203 1750 50  0000 C CNN
 F 1 "Fuse" V 2294 1750 50  0000 C CNN
-F 2 "" V 2330 1750 50  0001 C CNN
+F 2 "Fuse:Fuseholder_Cylinder-5x20mm_Schurter_FAB_0031-355x_Horizontal_Closed" V 2330 1750 50  0001 C CNN
 F 3 "~" H 2400 1750 50  0001 C CNN
 	1    2400 1750

Commit message: 2
Parts:
- C10, C2, C3, C6, C7: footprint Capacitor_THT:CP_Radial_D6.3mm_P2.50mm -> Capacitor_THT:CP_Radial_D4.0mm_P2.00mm
- C4: footprint Capacitor_THT:CP_Radial_D8.0mm_P3.50mm -> Capacitor_THT:CP_Radial_D4.0mm_P2.00mm
Changed lines of the file:
@@
 EESchema Schematic File Version 4
-LIBS:PONG_Display-cache
 EELAYER 30 0
 EELAYER END
@@
 F 0 "C10" H 8915 1946 50  0000 L CNN
 F 1 "10u" H 8915 1855 50  0000 L CNN
-F 2 "Capacitor_THT:CP_Radial_D6.3mm_P2.50mm" H 8838 1750 50  0001 C CNN
+F 2 "Capacitor_THT:CP_Radial_D4.0mm_P2.00mm" H 8838 1750 50  0001 C CNN
 F 3 "~" H 8800 1900 50  0001 C CNN
 	1    8800 1900
@@
 F 0 "C4" H 2818 6046 50  0000 L CNN
 F 1 "1u" H 2818 5955 50  0000 L CNN
-F 2 "Capacitor_THT:CP_Radial_D8.0mm_P3.50mm" H 2738 5850 50  0001 C CNN
+F 2 "Capacitor_THT:CP_Radial_D4.0mm_P2.00mm" H 2738 5850 50  0001 C CNN
 F 3 "~" H 2700 6000 50  0001 C CNN
 	1    2700 6000
@@
 F 0 "C3" H 2468 5696 50  0000 L CNN
 F 1 "10u" H 2468 5605 50  0000 L CNN
-F 2 "Capacitor_THT:CP_Radial_D6.3mm_P2.50mm" H 2388 5500 50  0001 C CNN
+F 2 "Capacitor_THT:CP_Radial_D4.0mm_P2.00mm" H 2388 5500 50  0001 C CNN
 F 3 "~" H 2350 5650 50  0001 C CNN
 	1    2350 5650
@@
 F 0 "C2" H 2118 5696 50  0000 L CNN
 F 1 "10u" H 2118 5605 50  0000 L CNN
-F 2 "Capacitor_THT:CP_Radial_D6.3mm_P2.50mm" H 2038 5500 50  0001 C CNN
+F 2 "Capacitor_THT:CP_Radial_D4.0mm_P2.00mm" H 2038 5500 50  0001 C CNN
 F 3 "~" H 2000 5650 50  0001 C CNN
 	1    2000 5650
@@
 F 0 "C6" H 5068 5696 50  0000 L CNN
 F 1 "10u" H 5068 5605 50  0000 L CNN
-F 2 "Capacitor_THT:CP_Radial_D6.3mm_P2.50mm" H 4988 5500 50  0001 C CNN
+F 2 "Capacitor_THT:CP_Radial_D4.0mm_P2.00mm" H 4988 5500 50  0001 C CNN
 F 3 "~" H 4950 5650 50  0001 C CNN
 	1    4950 5650
@@
 F 0 "C7" H 5468 5696 50  0000 L CNN
 F 1 "10u" H 5468 5605 50  0000 L CNN
-F 2 "Capacitor_THT:CP_Radial_D6.3mm_P2.50mm" H 5388 5500 50  0001 C CNN
+F 2 "Capacitor_THT:CP_Radial_D4.0mm_P2.00mm" H 5388 5500 50  0001 C CNN
 F 3 "~" H 5350 5650 50  0001 C CNN
 	1    5350 5650

Commit message: 5v
Parts:
- removed C2, C3, C6, C7: 10u, Capacitor_THT:CP_Radial_D4.0mm_P2.00mm, symbol Device:CP
- removed C4: 1u, Capacitor_THT:CP_Radial_D4.0mm_P2.00mm, symbol Device:CP
- removed C5: 100n, Capacitor_SMD:C_1206_3216Metric_Pad1.42x1.75mm_HandSolder, symbol Device:C
- removed D2: YELLOW_LED, Diode_SMD:D_1206_3216Metric_Pad1.42x1.75mm_HandSolder, symbol Device:LED
- removed L1: 22u, Inductor_SMD:L_12x12mm_H4.5mm, symbol Device:L
- removed R3: 150R, Resistor_SMD:R_1206_3216Metric_Pad1.42x1.75mm_HandSolder, symbol Device:R
- removed RV1: 100k, Potentiometer_THT:Potentiometer_Piher_PT-6-V_Vertical, symbol Device:R_POT
- removed U2: MCP16311MS, Package_SO:MSOP-8_3x3mm_P0.65mm, symbol Regulator_Switching:MCP16311MS
- renumbered C8 to C2, C9 to C3, C10 to C4, C11 to C5, D3 to D2, R4 to R3, U3 to U2
Connections:
- net +12V is gone; now on net +5V: F1.1, R2.1
Other:
- note removed: "Przetwornica DC/DC 12V/5V"
- moved on the sheet: D1, D2, R2, R3

Commit message: layout v1
Parts:
- C3, C5: footprint Capacitor_SMD:C_1206_3216Metric_Pad1.42x1.75mm_HandSolder -> Capacitor_SMD:C_0603_1608Metric_Pad1.05x0.95mm_HandSolder
- C4: footprint Capacitor_THT:CP_Radial_D4.0mm_P2.00mm -> Capacitor_SMD:C_1206_3216Metric_Pad1.42x1.75mm_HandSolder
- F1: footprint Fuse:Fuseholder_Cylinder-5x20mm_Schurter_FAB_0031-355x_Horizontal_Closed -> Fuse:Fuseholder_Cylinder-5x20mm_Schurter_0031_8201_Horizontal_Open
Changed lines of the file:
@@
 EESchema Schematic File Version 4
-LIBS:PONG_Display-cache
 EELAYER 30 0
 EELAYER END
@@
 F 0 "C3" H 7815 1946 50  0000 L CNN
 F 1 "100n" H 7815 1855 50  0000 L CNN
-F 2 "Capacitor_SMD:C_1206_3216Metric_Pad1.42x1.75mm_HandSolder" H 7738 1750 50  0001 C CNN
+F 2 "Capacitor_SMD:C_0603_1608Metric_Pad1.05x0.95mm_HandSolder" H 7738 1750 50  0001 C CNN
 F 3 "~" H 7700 1900 50  0001 C CNN
 	1    7700 1900
@@
 F 0 "C4" H 8915 1946 50  0000 L CNN
 F 1 "10u" H 8915 1855 50  0000 L CNN
-F 2 "Capacitor_THT:CP_Radial_D4.0mm_P2.00mm" H 8838 1750 50  0001 C CNN
+F 2 "Capacitor_SMD:C_1206_3216Metric_Pad1.42x1.75mm_HandSolder" H 8838 1750 50  0001 C CNN
 F 3 "~" H 8800 1900 50  0001 C CNN
 	1    8800 1900
@@
 F 0 "C5" H 9318 1946 50  0000 L CNN
 F 1 "100n" H 9318 1855 50  0000 L CNN
-F 2 "Capacitor_SMD:C_1206_3216Metric_Pad1.42x1.75mm_HandSolder" H 9238 1750 50  0001 C CNN
+F 2 "Capacitor_SMD:C_0603_1608Metric_Pad1.05x0.95mm_HandSolder" H 9238 1750 50  0001 C CNN
 F 3 "~" H 9200 1900 50  0001 C CNN
 	1    9200 1900
@@
 F 0 "F1" V 2203 1750 50  0000 C CNN
 F 1 "Fuse" V 2294 1750 50  0000 C CNN
-F 2 "Fuse:Fuseholder_Cylinder-5x20mm_Schurter_FAB_0031-355x_Horizontal_Closed" V 2330 1750 50  0001 C CNN
+F 2 "Fuse:Fuseholder_Cylinder-5x20mm_Schurter_0031_8201_Horizontal_Open" V 2330 1750 50  0001 C CNN
 F 3 "~" H 2400 1750 50  0001 C CNN
 	1    2400 1750

Commit message: l
Parts:
- R2, R3: footprint Resistor_SMD:R_1206_3216Metric_Pad1.42x1.75mm_HandSolder -> Resistor_SMD:R_0603_1608Metric_Pad1.05x0.95mm_HandSolder
Changed lines of the file:
@@
 F 0 "R2" H 4270 1896 50  0000 L CNN
 F 1 "470R" H 4270 1805 50  0000 L CNN
-F 2 "Resistor_SMD:R_1206_3216Metric_Pad1.42x1.75mm_HandSolder" V 4130 1850 50  0001 C CNN
+F 2 "Resistor_SMD:R_0603_1608Metric_Pad1.05x0.95mm_HandSolder" V 4130 1850 50  0001 C CNN
 F 3 "~" H 4200 1850 50  0001 C CNN
 	1    4200 1850
@@
 F 0 "R3" H 5120 1896 50  0000 L CNN
 F 1 "5R1" H 5120 1805 50  0000 L CNN
-F 2 "Resistor_SMD:R_1206_3216Metric_Pad1.42x1.75mm_HandSolder" V 4980 1850 50  0001 C CNN
+F 2 "Resistor_SMD:R_0603_1608Metric_Pad1.05x0.95mm_HandSolder" V 4980 1850 50  0001 C CNN
 F 3 "~" H 5050 1850 50  0001 C CNN
 	1    5050 1850
