File: PONG_Display/Power_supply.sch (KiCad schematic (older format))
At the start: 11 parts, among them J2 Input_Supply+12V, U2 LD1117S33TR_SOT223

Commit message: layout4
Parts:
- F1: footprint Fuse:Fuseholder_Cylinder-5x20mm_Schurter_0031_8201_Horizontal_Open -> Fuse:Fuse_Littelfuse_372_D8.50mm
- J2: value Input_Supply+12V -> Input_Supply+5V
Connections:
- net +5VA: now reaches F1.2, J2.1 (Pin_1)
Changed lines of the file:
@@
 AR Path="/5E83DA30" Ref="J?"  Part="1"
 F 0 "J2" H 1668 1967 50  0000 C CNN
-F 1 "Input_Supply+12V" H 1668 1876 50  0000 C CNN
+F 1 "Input_Supply+5V" H 1668 1876 50  0000 C CNN
 F 2 "TerminalBlock:TerminalBlock_bornier-2_P5.08mm" H 1750 1750 50  0001 C CNN
 F 3 "~" H 1750 1750 50  0001 C CNN
@@
 F 0 "F1" V 2203 1750 50  0000 C CNN
 F 1 "Fuse" V 2294 1750 50  0000 C CNN
-F 2 "Fuse:Fuseholder_Cylinder-5x20mm_Schurter_0031_8201_Horizontal_Open" V 2330 1750 50  0001 C CNN
+F 2 "Fuse:Fuse_Littelfuse_372_D8.50mm" V 2330 1750 50  0001 C CNN
 F 3 "~" H 2400 1750 50  0001 C CNN
 	1    2400 1750
@@
 	2550 1750 2850 1750
 Wire Wire Line
-	2250 1750 1950 1750
+	2250 1750 2200 1750
 $Comp
 L power:+5V #PWR06
@@
 	1    0    0    -1
 $EndComp
+$Comp
+L power:+5VA #PWR0111
+U 1 1 5EA465DD
+P 2200 1600
+F 0 "#PWR0111" H 2200 1450 50  0001 C CNN
+F 1 "+5VA" H 2215 1773 50  0000 C CNN
+F 2 "" H 2200 1600 50  0001 C CNN
+F 3 "" H 2200 1600 50  0001 C CNN
+	1    2200 1600
+	1    0    0    -1
+$EndComp
+Wire Wire Line
+	2200 1600 2200 1750
+Connection ~ 2200 1750
+Wire Wire Line
+	2200 1750 1950 1750
 $EndSCHEMATC

Commit message: laayout6
Parts:
- J2: footprint TerminalBlock:TerminalBlock_bornier-2_P5.08mm -> TerminalBlock_RND:TerminalBlock_RND_205-00001_1x02_P5.00mm_Horizontal
Changed lines of the file:
@@
 F 0 "J2" H 1668 1967 50  0000 C CNN
 F 1 "Input_Supply+5V" H 1668 1876 50  0000 C CNN
-F 2 "TerminalBlock:TerminalBlock_bornier-2_P5.08mm" H 1750 1750 50  0001 C CNN
+F 2 "TerminalBlock_RND:TerminalBlock_RND_205-00001_1x02_P5.00mm_Horizontal" H 1750 1750 50  0001 C CNN
 F 3 "~" H 1750 1750 50  0001 C CNN
 	1    1750 1750

Commit message: Layout 11
Parts:
- D1, D2: footprint Diode_SMD:D_1206_3216Metric_Pad1.42x1.75mm_HandSolder -> Diode_SMD:D_0805_2012Metric_Pad1.15x1.40mm_HandSolder
Changed lines of the file:
@@
 F 0 "D1" V 4239 2182 50  0000 R CNN
 F 1 "RED_LED" V 4148 2182 50  0000 R CNN
-F 2 "Diode_SMD:D_1206_3216Metric_Pad1.42x1.75mm_HandSolder" H 4200 2300 50  0001 C CNN
+F 2 "Diode_SMD:D_0805_2012Metric_Pad1.15x1.40mm_HandSolder" H 4200 2300 50  0001 C CNN
 F 3 "~" H 4200 2300 50  0001 C CNN
 	1    4200 2300
@@
 F 0 "D2" V 5089 2182 50  0000 R CNN
 F 1 "GREEN_LED" V 4998 2182 50  0000 R CNN
-F 2 "Diode_SMD:D_1206_3216Metric_Pad1.42x1.75mm_HandSolder" H 5050 2300 50  0001 C CNN
+F 2 "Diode_SMD:D_0805_2012Metric_Pad1.15x1.40mm_HandSolder" H 5050 2300 50  0001 C CNN
 F 3 "~" H 5050 2300 50  0001 C CNN
 	1    5050 2300
