File: PONG_Display/esp.sch (KiCad schematic (older format))
At the start: 4 parts, among them J7 ESP_Conn, J8 ESP_Prog_Conn, SW2 SW_Push_SPDT, SW3 SW_Push_SPDT

Commit message: 23
Parts:
- added C?: 100n, Capacitor_SMD:C_1206_3216Metric_Pad1.42x1.75mm_HandSolder, symbol Device:C
- added D?: D_Zener, Diode_THT:D_DO-34_SOD68_P7.62mm_Horizontal, symbol Device:D_Zener
- added R?: 10k, Resistor_SMD:R_1206_3216Metric_Pad1.42x1.75mm_HandSolder, symbol Device:R
- added R?: 330R, Resistor_SMD:R_1206_3216Metric_Pad1.42x1.75mm_HandSolder, symbol Device:R
- added SW?: SW_Push, Button_Switch_THT:SW_PUSH_6mm, symbol Switch:SW_Push
Connections:
- net ESP_RST: now also C?.1, D?.2 (A), R?.2, SW?.1
- net GND: now also C?.2, R?.2
- new net: R?.1, SW?.2
- new net +5V: D?.1 (K), R?.1
Changed lines of the file:
@@
 NoConn ~ 9050 2350
 NoConn ~ 9050 2800
+$Comp
+L power:+5V #PWR?
+U 1 1 5E9DFF82
+P 4700 5250
+F 0 "#PWR?" H 4700 5100 50  0001 C CNN
+F 1 "+5V" H 4715 5423 50  0000 C CNN
+F 2 "" H 4700 5250 50  0001 C CNN
+F 3 "" H 4700 5250 50  0001 C CNN
+	1    4700 5250
+	1    0    0    -1
+$EndComp
+$Comp
+L power:GND #PWR?
+U 1 1 5E9DFF88
+P 4700 6250
+F 0 "#PWR?" H 4700 6000 50  0001 C CNN
+F 1 "GND" H 4705 6077 50  0000 C CNN
+F 2 "" H 4700 6250 50  0001 C CNN
+F 3 "" H 4700 6250 50  0001 C CNN
+	1    4700 6250
+	1    0    0    -1
+$EndComp
+$Comp
+L Device:C C?
+U 1 1 5E9DFF8E
+P 4700 6000
+F 0 "C?" H 4815 6046 50  0000 L CNN
+F 1 "100n" H 4815 5955 50  0000 L CNN
+F 2 "Capacitor_SMD:C_1206_3216Metric_Pad1.42x1.75mm_HandSolder" H 4738 5850 50  0001 C CNN
+F 3 "~" H 4700 6000 50  0001 C CNN
+	1    4700 6000
+	1    0    0    -1
+$EndComp
+$Comp
+L Device:R R?
+U 1 1 5E9DFF94
+P 4550 5500
+F 0 "R?" H 4620 5546 50  0000 L CNN
+F 1 "10k" H 4620 5455 50  0000 L CNN
+F 2 "Resistor_SMD:R_1206_3216Metric_Pad1.42x1.75mm_HandSolder" V 4480 5500 50  0001 C CNN
+F 3 "~" H 4550 5500 50  0001 C CNN
+	1    4550 5500
+	1    0    0    -1
+$EndComp
+$Comp
+L Device:D_Zener D?
+U 1 1 5E9DFF9A
+P 4800 5500
+F 0 "D?" V 4754 5579 50  0000 L CNN
+F 1 "D_Zener" V 4845 5579 50  0000 L CNN
+F 2 "Diode_THT:D_DO-34_SOD68_P7.62mm_Horizontal" H 4800 5500 50  0001 C CNN
+F 3 "~" H 4800 5500 50  0001 C CNN
+	1    4800 5500
+	0    1    1    0
+$EndComp
+Wire Wire Line
+	4700 5250 4800 5250
+Wire Wire Line
+	4800 5250 4800 5350
+Wire Wire Line
+	4700 5250 4550 5250
+Wire Wire Line
+	4550 5250 4550 5350
+Connection ~ 4700 5250
+Wire Wire Line
+	4550 5650 4550 5750
+Wire Wire Line
+	4800 5750 4800 5650
+Wire Wire Line
+	4700 6250 4700 6150
+Wire Wire Line
+	4550 5750 4050 5750
+Connection ~ 4550 5750
+$Comp
+L Device:R R?
+U 1 1 5E9DFFAA
+P 5850 6100
+F 0 "R?" H 5920 6146 50  0000 L CNN
+F 1 "330R" H 5920 6055 50  0000 L CNN
+F 2 "Resistor_SMD:R_1206_3216Metric_Pad1.42x1.75mm_HandSolder" V 5780 6100 50  0001 C CNN
+F 3 "~" H 5850 6100 50  0001 C CNN
+	1    5850 6100
+	1    0    0    -1
+$EndComp
+$Comp
+L power:GND #PWR?
+U 1 1 5E9DFFB0
+P 5850 6500
+F 0 "#PWR?" H 5850 6250 50  0001 C CNN
+F 1 "GND" H 5855 6327 50  0000 C CNN
+F 2 "" H 5850 6500 50  0001 C CNN
+F 3 "" H 5850 6500 50  0001 C CNN
+	1    5850 6500
+	1    0    0    -1
+$EndComp
+Wire Wire Line
+	5850 6250 5850 6500
+Wire Wire Line
+	4550 5750 4700 5750
+Wire Wire Line
+	4700 5750 4700 5850
+Connection ~ 4700 5750
+Wire Wire Line
+	4700 5750 4800 5750
+$Comp
+L Switch:SW_Push SW?
+U 1 1 5E9DFFBB
+P 5400 5750
+F 0 "SW?" H 5400 6035 50  0000 C CNN
+F 1 "SW_Push" H 5400 5944 50  0000 C CNN
+F 2 "Button_Switch_THT:SW_PUSH_6mm" H 5400 5950 50  0001 C CNN
+F 3 "~" H 5400 5950 50  0001 C CNN
+	1    5400 5750
+	1    0    0    -1
+$EndComp
+Wire Wire Line
+	4800 5750 5200 5750
+Connection ~ 4800 5750
+Wire Wire Line
+	5850 5750 5850 5950
+Wire Wire Line
+	5600 5750 5850 5750
+Text HLabel 4050 5750 0    50   Input ~ 0
+ESP_RST
 $EndSCHEMATC

Commit message: po obgadaniu
Parts:
- gave numbers to parts that had none: 5
Connections:
- net +3V3: now also J7.2 (Pin_2); no longer J7.1 (Pin_1)
- net ESP_CH_PD: now also J7.6 (Pin_6); no longer J7.5 (Pin_5)
- net ESP_GPIO0: now also J7.3 (Pin_3); no longer J7.4 (Pin_4)
- net ESP_GPIO2: now also J7.5 (Pin_5); no longer J7.6 (Pin_6)
- net ESP_RST: now also J7.4 (Pin_4); no longer J7.3 (Pin_3)
- net ESP_RX: now also J7.1 (Pin_1); no longer J7.2 (Pin_2)
- net ESP_TX: now also J7.8 (Pin_8); no longer J7.7 (Pin_7)
- net GND: now also J7.7 (Pin_7); no longer J7.8 (Pin_8)
Changed lines of the file:
@@
 EESchema Schematic File Version 4
+LIBS:PONG_Display-cache
 EELAYER 30 0
 EELAYER END
@@
 L Connector_Generic:Conn_02x04_Odd_Even J?
 U 1 1 5E838274
-P 4400 2150
+P 4300 2150
 AR Path="/5E80CCDD/5E838274" Ref="J?"  Part="1"
 AR Path="/5E80B1F8/5E838274" Ref="J7"  Part="1"
-F 0 "J7" H 4450 2467 50  0000 C CNN
-F 1 "ESP_Conn" H 4450 2376 50  0000 C CNN
-F 2 "Connector_PinHeader_2.54mm:PinHeader_2x04_P2.54mm_Vertical" H 4400 2150 50  0001 C CNN
-F 3 "~" H 4400 2150 50  0001 C CNN
-	1    4400 2150
-	-1   0    0    -1
+F 0 "J7" H 4350 2467 50  0000 C CNN
+F 1 "ESP_Conn" H 4350 2376 50  0000 C CNN
+F 2 "Connector_PinHeader_2.54mm:PinHeader_2x04_P2.54mm_Vertical" H 4300 2150 50  0001 C CNN
+F 3 "~" H 4300 2150 50  0001 C CNN
+	1    4300 2150
+	1    0    0    -1
 $EndComp
 Wire Wire Line
@@
 Wire Wire Line
 	4800 1900 4800 2050
-Wire Wire Line
-	4600 2050 4800 2050
 Wire Wire Line
 	3850 2350 3850 2500
@@
 NoConn ~ 9050 2800
 $Comp
-L power:+5V #PWR?
+L power:+5V #PWR0177
 U 1 1 5E9DFF82
 P 4700 5250
-F 0 "#PWR?" H 4700 5100 50  0001 C CNN
+F 0 "#PWR0177" H 4700 5100 50  0001 C CNN
 F 1 "+5V" H 4715 5423 50  0000 C CNN
 F 2 "" H 4700 5250 50  0001 C CNN
@@
 $EndComp
 $Comp
-L power:GND #PWR?
+L power:GND #PWR0178
 U 1 1 5E9DFF88
 P 4700 6250
-F 0 "#PWR?" H 4700 6000 50  0001 C CNN
+F 0 "#PWR0178" H 4700 6000 50  0001 C CNN
 F 1 "GND" H 4705 6077 50  0000 C CNN
 F 2 "" H 4700 6250 50  0001 C CNN
@@
 $EndComp
 $Comp
-L Device:C C?
+L Device:C C28
 U 1 1 5E9DFF8E
 P 4700 6000
-F 0 "C?" H 4815 6046 50  0000 L CNN
+F 0 "C28" H 4815 6046 50  0000 L CNN
 F 1 "100n" H 4815 5955 50  0000 L CNN
 F 2 "Capacitor_SMD:C_1206_3216Metric_Pad1.42x1.75mm_HandSolder" H 4738 5850 50  0001 C CNN
@@
 $EndComp
 $Comp
-L Device:R R?
+L Device:R R9
 U 1 1 5E9DFF94
 P 4550 5500
-F 0 "R?" H 4620 5546 50  0000 L CNN
+F 0 "R9" H 4620 5546 50  0000 L CNN
 F 1 "10k" H 4620 5455 50  0000 L CNN
 F 2 "Resistor_SMD:R_1206_3216Metric_Pad1.42x1.75mm_HandSolder" V 4480 5500 50  0001 C CNN
@@
 $EndComp
 $Comp
-L Device:D_Zener D?
+L Device:D_Zener D5
 U 1 1 5E9DFF9A
 P 4800 5500
-F 0 "D?" V 4754 5579 50  0000 L CNN
+F 0 "D5" V 4754 5579 50  0000 L CNN
 F 1 "D_Zener" V 4845 5579 50  0000 L CNN
 F 2 "Diode_THT:D_DO-34_SOD68_P7.62mm_Horizontal" H 4800 5500 50  0001 C CNN
@@
 Connection ~ 4550 5750
 $Comp
-L Device:R R?
+L Device:R R10
 U 1 1 5E9DFFAA
 P 5850 6100
-F 0 "R?" H 5920 6146 50  0000 L CNN
+F 0 "R10" H 5920 6146 50  0000 L CNN
 F 1 "330R" H 5920 6055 50  0000 L CNN
 F 2 "Resistor_SMD:R_1206_3216Metric_Pad1.42x1.75mm_HandSolder" V 5780 6100 50  0001 C CNN
@@
 $EndComp
 $Comp
-L power:GND #PWR?
+L power:GND #PWR0179
 U 1 1 5E9DFFB0
 P 5850 6500
-F 0 "#PWR?" H 5850 6250 50  0001 C CNN
+F 0 "#PWR0179" H 5850 6250 50  0001 C CNN
 F 1 "GND" H 5855 6327 50  0000 C CNN
 F 2 "" H 5850 6500 50  0001 C CNN
@@
 	4700 5750 4800 5750
 $Comp
-L Switch:SW_Push SW?
+L Switch:SW_Push SW4
 U 1 1 5E9DFFBB
 P 5400 5750
-F 0 "SW?" H 5400 6035 50  0000 C CNN
+F 0 "SW4" H 5400 6035 50  0000 C CNN
 F 1 "SW_Push" H 5400 5944 50  0000 C CNN
 F 2 "Button_Switch_THT:SW_PUSH_6mm" H 5400 5950 50  0001 C CNN
@@
 Text HLabel 4050 5750 0    50   Input ~ 0
 ESP_RST
+Wire Wire Line
+	4600 2050 4800 2050
 $EndSCHEMATC

Commit message: 5v
Parts:
- renumbered C28 to C22, D5 to D4, J7 to J8, J8 to J9, R9 to R8, R10 to R9, SW4 to SW2, SW2 to SW3, SW3 to SW4
Changed lines of the file:
@@
 EESchema Schematic File Version 4
-LIBS:PONG_Display-cache
 EELAYER 30 0
 EELAYER END
@@
 P 4300 2150
 AR Path="/5E80CCDD/5E838274" Ref="J?"  Part="1"
-AR Path="/5E80B1F8/5E838274" Ref="J7"  Part="1"
-F 0 "J7" H 4350 2467 50  0000 C CNN
+AR Path="/5E80B1F8/5E838274" Ref="J8"  Part="1"
+F 0 "J8" H 4350 2467 50  0000 C CNN
 F 1 "ESP_Conn" H 4350 2376 50  0000 C CNN
 F 2 "Connector_PinHeader_2.54mm:PinHeader_2x04_P2.54mm_Vertical" H 4300 2150 50  0001 C CNN
@@
 P 4700 3150
 AR Path="/5E80CCDD/5E838282" Ref="J?"  Part="1"
-AR Path="/5E80B1F8/5E838282" Ref="J8"  Part="1"
-F 0 "J8" H 4780 3142 50  0000 L CNN
+AR Path="/5E80B1F8/5E838282" Ref="J9"  Part="1"
+F 0 "J9" H 4780 3142 50  0000 L CNN
 F 1 "ESP_Prog_Conn" H 4780 3051 50  0000 L CNN
 F 2 "Connector_PinHeader_2.54mm:PinHeader_1x04_P2.54mm_Vertical" H 4700 3150 50  0001 C CNN
@@
 Schemat modułu WiFi
 $Comp
-L power:+3.3V #PWR0173
+L power:+3.3V #PWR066
 U 1 1 5E858E36
 P 4800 1900
-F 0 "#PWR0173" H 4800 1750 50  0001 C CNN
+F 0 "#PWR066" H 4800 1750 50  0001 C CNN
 F 1 "+3.3V" H 4815 2073 50  0000 C CNN
 F 2 "" H 4800 1900 50  0001 C CNN
@@
 $EndComp
 $Comp
-L power:GND #PWR0174
+L power:GND #PWR061
 U 1 1 5E85942E
 P 3850 2500
-F 0 "#PWR0174" H 3850 2250 50  0001 C CNN
+F 0 "#PWR061" H 3850 2250 50  0001 C CNN
 F 1 "GND" H 3855 2327 50  0000 C CNN
 F 2 "" H 3850 2500 50  0001 C CNN
@@
 	3850 2350 4100 2350
 $Comp
-L power:+3.3V #PWR0175
+L power:+3.3V #PWR062
 U 1 1 5E859CE6
 P 4350 2900
-F 0 "#PWR0175" H 4350 2750 50  0001 C CNN
+F 0 "#PWR062" H 4350 2750 50  0001 C CNN
 F 1 "+3.3V" H 4365 3073 50  0000 C CNN
 F 2 "" H 4350 2900 50  0001 C CNN
@@
 $EndComp
 $Comp
-L power:GND #PWR0176
+L power:GND #PWR063
 U 1 1 5E85A6F5
 P 4350 3600
-F 0 "#PWR0176" H 4350 3350 50  0001 C CNN
+F 0 "#PWR063" H 4350 3350 50  0001 C CNN
 F 1 "GND" H 4355 3427 50  0000 C CNN
 F 2 "" H 4350 3600 50  0001 C CNN
@@
 Przełączniki programowania ESP przez RS232
 $Comp
-L power:+3.3V #PWR01
+L power:+3.3V #PWR068
 U 1 1 5E9D6E89
 P 9550 1900
-F 0 "#PWR01" H 9550 1750 50  0001 C CNN
+F 0 "#PWR068" H 9550 1750 50  0001 C CNN
 F 1 "+3.3V" H 9565 2073 50  0000 C CNN
 F 2 "" H 9550 1900 50  0001 C CNN
@@
 $EndComp
 $Comp
-L power:GND #PWR02
+L power:GND #PWR069
 U 1 1 5E9D779A
 P 9550 3050
-F 0 "#PWR02" H 9550 2800 50  0001 C CNN
+F 0 "#PWR069" H 9550 2800 50  0001 C CNN
 F 1 "GND" H 9555 2877 50  0000 C CNN
 F 2 "" H 9550 3050 50  0001 C CNN
@@
 	8300 2700 8650 2700
 $Comp
-L Switch:SW_Push_SPDT SW2
+L Switch:SW_Push_SPDT SW3
 U 1 1 5E9E35EF
 P 8850 2250
-F 0 "SW2" H 8850 2535 50  0000 C CNN
+F 0 "SW3" H 8850 2535 50  0000 C CNN
 F 1 "SW_Push_SPDT" H 8850 2444 50  0000 C CNN
 F 2 "LIB_PONG_Display:SPDT_switch" H 8850 2250 50  0001 C CNN
@@
 $EndComp
 $Comp
-L Switch:SW_Push_SPDT SW3
+L Switch:SW_Push_SPDT SW4
 U 1 1 5E9E3E9D
 P 8850 2700
-F 0 "SW3" H 8850 2985 50  0000 C CNN
+F 0 "SW4" H 8850 2985 50  0000 C CNN
 F 1 "SW_Push_SPDT" H 8850 2894 50  0000 C CNN
 F 2 "LIB_PONG_Display:SPDT_switch" H 8850 2700 50  0001 C CNN
@@
 NoConn ~ 9050 2800
 $Comp
-L power:+5V #PWR0177
+L power:+5V #PWR064
 U 1 1 5E9DFF82
 P 4700 5250
-F 0 "#PWR0177" H 4700 5100 50  0001 C CNN
+F 0 "#PWR064" H 4700 5100 50  0001 C CNN
 F 1 "+5V" H 4715 5423 50  0000 C CNN
 F 2 "" H 4700 5250 50  0001 C CNN
@@
 $EndComp
 $Comp
-L power:GND #PWR0178
+L power:GND #PWR065
 U 1 1 5E9DFF88
 P 4700 6250
-F 0 "#PWR0178" H 4700 6000 50  0001 C CNN
+F 0 "#PWR065" H 4700 6000 50  0001 C CNN
 F 1 "GND" H 4705 6077 50  0000 C CNN
 F 2 "" H 4700 6250 50  0001 C CNN
@@
 $EndComp
 $Comp
-L Device:C C28
+L Device:C C22
 U 1 1 5E9DFF8E
 P 4700 6000
-F 0 "C28" H 4815 6046 50  0000 L CNN
+F 0 "C22" H 4815 6046 50  0000 L CNN
 F 1 "100n" H 4815 5955 50  0000 L CNN
 F 2 "Capacitor_SMD:C_1206_3216Metric_Pad1.42x1.75mm_HandSolder" H 4738 5850 50  0001 C CNN
@@
 $EndComp
 $Comp
-L Device:R R9
+L Device:R R8
 U 1 1 5E9DFF94
 P 4550 5500
-F 0 "R9" H 4620 5546 50  0000 L CNN
+F 0 "R8" H 4620 5546 50  0000 L CNN
 F 1 "10k" H 4620 5455 50  0000 L CNN
 F 2 "Resistor_SMD:R_1206_3216Metric_Pad1.42x1.75mm_HandSolder" V 4480 5500 50  0001 C CNN
@@
 $EndComp
 $Comp
-L Device:D_Zener D5
+L Device:D_Zener D4
 U 1 1 5E9DFF9A
 P 4800 5500
-F 0 "D5" V 4754 5579 50  0000 L CNN
+F 0 "D4" V 4754 5579 50  0000 L CNN
 F 1 "D_Zener" V 4845 5579 50  0000 L CNN
 F 2 "Diode_THT:D_DO-34_SOD68_P7.62mm_Horizontal" H 4800 5500 50  0001 C CNN
@@
 Connection ~ 4550 5750
 $Comp
-L Device:R R10
+L Device:R R9
 U 1 1 5E9DFFAA
 P 5850 6100
-F 0 "R10" H 5920 6146 50  0000 L CNN
+F 0 "R9" H 5920 6146 50  0000 L CNN
 F 1 "330R" H 5920 6055 50  0000 L CNN
 F 2 "Resistor_SMD:R_1206_3216Metric_Pad1.42x1.75mm_HandSolder" V 5780 6100 50  0001 C CNN
@@
 $EndComp
 $Comp
-L power:GND #PWR0179
+L power:GND #PWR067
 U 1 1 5E9DFFB0
 P 5850 6500
-F 0 "#PWR0179" H 5850 6250 50  0001 C CNN
+F 0 "#PWR067" H 5850 6250 50  0001 C CNN
 F 1 "GND" H 5855 6327 50  0000 C CNN
 F 2 "" H 5850 6500 50  0001 C CNN
@@
 	4700 5750 4800 5750
 $Comp
-L Switch:SW_Push SW4
+L Switch:SW_Push SW2
 U 1 1 5E9DFFBB
 P 5400 5750
-F 0 "SW4" H 5400 6035 50  0000 C CNN
+F 0 "SW2" H 5400 6035 50  0000 C CNN
 F 1 "SW_Push" H 5400 5944 50  0000 C CNN
 F 2 "Button_Switch_THT:SW_PUSH_6mm" H 5400 5950 50  0001 C CNN

Commit message: jeszcze do przekminienia
Parts:
- added Q? (x2): 2N7000, symbol Device:Q_NMOS_DGS
- added R? (x4): 10k, Resistor_SMD:R_1206_3216Metric_Pad1.42x1.75mm_HandSolder, symbol Device:R
Connections:
- net +3V3: now also D4.1 (K), R8.1, Q?.2 (G), Q?.2 (G), R?.1, R?.1
- net +5V: now also R?.1, R?.1; no longer D4.1 (K), R8.1
- net ESP_RX: now also Q?.3 (S), R?.2
- net ESP_TX: now also Q?.3 (S), R?.2
- new net ESP_RX_HIGH: Q?.1 (D), R?.2
- new net ESP_TX_HIGH: Q?.1 (D), R?.2
Other:
- note added: "konwerter stanów logicznych\n"
Changed lines of the file:
@@
 EESchema Schematic File Version 4
+LIBS:PONG_Display-cache
 EELAYER 30 0
 EELAYER END
@@
 	1    0    0    -1
 $EndComp
-Text HLabel 3950 2050 0    50   Input ~ 0
-ESP_RX
-Text HLabel 4700 2350 2    50   Input ~ 0
-ESP_TX
 Text HLabel 4700 2150 2    50   Input ~ 0
 ESP_RST
@@
 Text HLabel 3950 2250 0    50   Input ~ 0
 ESP_GPIO2
-Text HLabel 4350 3150 0    50   Input ~ 0
-ESP_RX
-Text HLabel 4350 3250 0    50   Input ~ 0
-ESP_TX
 Text HLabel 8300 2250 0    50   Input ~ 0
 ESP_CH_PD
@@
 NoConn ~ 9050 2350
 NoConn ~ 9050 2800
-$Comp
-L power:+5V #PWR064
-U 1 1 5E9DFF82
-P 4700 5250
-F 0 "#PWR064" H 4700 5100 50  0001 C CNN
-F 1 "+5V" H 4715 5423 50  0000 C CNN
-F 2 "" H 4700 5250 50  0001 C CNN
-F 3 "" H 4700 5250 50  0001 C CNN
-	1    4700 5250
-	1    0    0    -1
-$EndComp
 $Comp
 L power:GND #PWR065
@@
 $EndComp
 Wire Wire Line
-	4700 5250 4800 5250
-Wire Wire Line
 	4800 5250 4800 5350
 Wire Wire Line
-	4700 5250 4550 5250
-Wire Wire Line
 	4550 5250 4550 5350
-Connection ~ 4700 5250
 Wire Wire Line
 	4550 5650 4550 5750
@@
 Wire Wire Line
 	4600 2050 4800 2050
+Text Label 4700 2350 0    50   ~ 0
+ESP_TX
+Text Label 3950 2050 2    50   ~ 0
+ESP_RX
+Text Label 4350 3250 2    50   ~ 0
+ESP_TX
+Text Label 4350 3150 2    50   ~ 0
+ESP_RX
+Text HLabel 10050 5050 2    50   Input ~ 0
+ESP_RX_HIGH
+Text HLabel 10050 6100 2    50   Input ~ 0
+ESP_TX_HIGH
+Text Label 8050 5050 2    50   ~ 0
+ESP_RX
+Text Label 8050 6100 2    50   ~ 0
+ESP_TX
+$Comp
+L Device:Q_NMOS_DGS Q?
+U 1 1 5E9CF246
+P 9100 4950
+F 0 "Q?" V 9351 4950 50  0000 C CNN
+F 1 "2N7000" V 9442 4950 50  0000 C CNN
+F 2 "" H 9300 5050 50  0001 C CNN
+F 3 "~" H 9100 4950 50  0001 C CNN
+	1    9100 4950
+	0    1    1    0
+$EndComp
+$Comp
+L Device:Q_NMOS_DGS Q?
+U 1 1 5E9D0B65
+P 9100 6000
+F 0 "Q?" V 9351 6000 50  0000 C CNN
+F 1 "2N7000" V 9442 6000 50  0000 C CNN
+F 2 "" H 9300 6100 50  0001 C CNN
+F 3 "~" H 9100 6000 50  0001 C CNN
+	1    9100 6000
+	0    1    1    0
+$EndComp
+Wire Wire Line
+	8050 5050 8650 5050
+Wire Wire Line
+	8050 6100 8650 6100
+Wire Wire Line
+	9300 6100 9650 6100
+Wire Wire Line
+	9300 5050 9650 5050
+$Comp
+L power:+3.3V #PWR?
+U 1 1 5E9D4B92
+P 8650 4600
+F 0 "#PWR?" H 8650 4450 50  0001 C CNN
+F 1 "+3.3V" H 8665 4773 50  0000 C CNN
+F 2 "" H 8650 4600 50  0001 C CNN
+F 3 "" H 8650 4600 50  0001 C CNN
+	1    8650 4600
+	1    0    0    -1
+$EndComp
+$Comp
+L power:+3.3V #PWR?
+U 1 1 5E9D533A
+P 8650 5650
+F 0 "#PWR?" H 8650 5500 50  0001 C CNN
+F 1 "+3.3V" H 8665 5823 50  0000 C CNN
+F 2 "" H 8650 5650 50  0001 C CNN
+F 3 "" H 8650 5650 50  0001 C CNN
+	1    8650 5650
+	1    0    0    -1
+$EndComp
+$Comp
+L Device:R R?
+U 1 1 5E9D5B4F
+P 8650 5850
+F 0 "R?" H 8720 5896 50  0000 L CNN
+F 1 "10k" H 8720 5805 50  0000 L CNN
+F 2 "Resistor_SMD:R_1206_3216Metric_Pad1.42x1.75mm_HandSolder" V 8580 5850 50  0001 C CNN
+F 3 "~" H 8650 5850 50  0001 C CNN
+	1    8650 5850
+	1    0    0    -1
+$EndComp
+Wire Wire Line
+	8650 4950 8650 5050
+Connection ~ 8650 5050
+Wire Wire Line
+	8650 5050 8900 5050
+Wire Wire Line
+	8650 4600 8650 4650
+Wire Wire Line
+	8650 6000 8650 6100
+Connection ~ 8650 6100
+Wire Wire Line
+	8650 6100 8900 6100
+Wire Wire Line
+	8650 5650 8650 5700
+$Comp
+L Device:R R?
+U 1 1 5E9D56BD
+P 8650 4800
+F 0 "R?" H 8720 4846 50  0000 L CNN
+F 1 "10k" H 8720 4755 50  0000 L CNN
+F 2 "Resistor_SMD:R_1206_3216Metric_Pad1.42x1.75mm_HandSolder" V 8580 4800 50  0001 C CNN
+F 3 "~" H 8650 4800 50  0001 C CNN
+	1    8650 4800
+	1    0    0    -1
+$EndComp
+$Comp
+L power:+5V #PWR?
+U 1 1 5E9D8E3B
+P 9650 4600
+F 0 "#PWR?" H 9650 4450 50  0001 C CNN
+F 1 "+5V" H 9665 4773 50  0000 C CNN
+F 2 "" H 9650 4600 50  0001 C CNN
+F 3 "" H 9650 4600 50  0001 C CNN
+	1    9650 4600
+	1    0    0    -1
+$EndComp
+$Comp
+L power:+5V #PWR?
+U 1 1 5E9D96BA
+P 9650 5650
+F 0 "#PWR?" H 9650 5500 50  0001 C CNN
+F 1 "+5V" H 9665 5823 50  0000 C CNN
+F 2 "" H 9650 5650 50  0001 C CNN
+F 3 "" H 9650 5650 50  0001 C CNN
+	1    9650 5650
+	1    0    0    -1
+$EndComp
+$Comp
+L Device:R R?
+U 1 1 5E9D99AA
+P 9650 4800
+F 0 "R?" H 9720 4846 50  0000 L CNN
+F 1 "10k" H 9720 4755 50  0000 L CNN
+F 2 "Resistor_SMD:R_1206_3216Metric_Pad1.42x1.75mm_HandSolder" V 9580 4800 50  0001 C CNN
+F 3 "~" H 9650 4800 50  0001 C CNN
+	1    9650 4800
+	1    0    0    -1
+$EndComp
+$Comp
+L Device:R R?
+U 1 1 5E9D9C8C
+P 9650 5850
+F 0 "R?" H 9720 5896 50  0000 L CNN
+F 1 "10k" H 9720 5805 50  0000 L CNN
+F 2 "Resistor_SMD:R_1206_3216Metric_Pad1.42x1.75mm_HandSolder" V 9580 5850 50  0001 C CNN
+F 3 "~" H 9650 5850 50  0001 C CNN
+	1    9650 5850
+	1    0    0    -1
+$EndComp
+Wire Wire Line
+	9650 4600 9650 4650
+Wire Wire Line
+	9650 4950 9650 5050
+Connection ~ 9650 5050
+Wire Wire Line
+	9650 5050 10050 5050
+Wire Wire Line
+	9650 5650 9650 5700
+Wire Wire Line
+	9650 6000 9650 6100
+Connection ~ 9650 6100
+Wire Wire Line
+	9650 6100 10050 6100
+Wire Wire Line
+	4550 5250 4700 5250
+$Comp
+L power:+3.3V #PWR?
+U 1 1 5E9DD25C
+P 4700 5250
+F 0 "#PWR?" H 4700 5100 50  0001 C CNN
+F 1 "+3.3V" H 4715 5423 50  0000 C CNN
+F 2 "" H 4700 5250 50  0001 C CNN
+F 3 "" H 4700 5250 50  0001 C CNN
+	1    4700 5250
+	1    0    0    -1
+$EndComp
+Connection ~ 4700 5250
+Wire Wire Line
+	4700 5250 4800 5250
+$Comp
+L power:+3.3V #PWR?
+U 1 1 5E9E0D36
+P 9100 4600
+F 0 "#PWR?" H 9100 4450 50  0001 C CNN
+F 1 "+3.3V" H 9115 4773 50  0000 C CNN
+F 2 "" H 9100 4600 50  0001 C CNN
+F 3 "" H 9100 4600 50  0001 C CNN
+	1    9100 4600
+	1    0    0    -1
+$EndComp
+$Comp
+L power:+3.3V #PWR?
+U 1 1 5E9E0F18
+P 9100 5650
+F 0 "#PWR?" H 9100 5500 50  0001 C CNN
+F 1 "+3.3V" H 9115 5823 50  0000 C CNN
+F 2 "" H 9100 5650 50  0001 C CNN
+F 3 "" H 9100 5650 50  0001 C CNN
+	1    9100 5650
+	1    0    0    -1
+$EndComp
+Wire Wire Line
+	9100 4600 9100 4750
+Wire Wire Line
+	9100 5650 9100 5800
+Text Notes 8550 4250 0    50   ~ 0
+konwerter stanów logicznych\n
+Wire Notes Line
+	7000 4050 10700 4050
+Wire Notes Line
+	10700 4050 10700 6500
+Wire Notes Line
+	10700 6500 7000 6500
+Wire Notes Line
+	7000 6500 7000 4050
 $EndSCHEMATC

Commit message: wywalone rezystory
Parts:
- removed R? (x2): 10k, Resistor_SMD:R_1206_3216Metric_Pad1.42x1.75mm_HandSolder, symbol Device:R
Changed lines of the file:
@@
 	8050 5050 8650 5050
 Wire Wire Line
-	8050 6100 8650 6100
-Wire Wire Line
 	9300 6100 9650 6100
-Wire Wire Line
-	9300 5050 9650 5050
 $Comp
 L power:+3.3V #PWR?
@@
 	1    0    0    -1
 $EndComp
-$Comp
-L power:+3.3V #PWR?
-U 1 1 5E9D533A
-P 8650 5650
-F 0 "#PWR?" H 8650 5500 50  0001 C CNN
-F 1 "+3.3V" H 8665 5823 50  0000 C CNN
-F 2 "" H 8650 5650 50  0001 C CNN
-F 3 "" H 8650 5650 50  0001 C CNN
-	1    8650 5650
-	1    0    0    -1
-$EndComp
-$Comp
-L Device:R R?
-U 1 1 5E9D5B4F
-P 8650 5850
-F 0 "R?" H 8720 5896 50  0000 L CNN
-F 1 "10k" H 8720 5805 50  0000 L CNN
-F 2 "Resistor_SMD:R_1206_3216Metric_Pad1.42x1.75mm_HandSolder" V 8580 5850 50  0001 C CNN
-F 3 "~" H 8650 5850 50  0001 C CNN
-	1    8650 5850
-	1    0    0    -1
-$EndComp
 Wire Wire Line
 	8650 4950 8650 5050
@@
 Wire Wire Line
 	8650 4600 8650 4650
-Wire Wire Line
-	8650 6000 8650 6100
-Connection ~ 8650 6100
-Wire Wire Line
-	8650 6100 8900 6100
-Wire Wire Line
-	8650 5650 8650 5700
 $Comp
 L Device:R R?
@@
 F 3 "~" H 8650 4800 50  0001 C CNN
 	1    8650 4800
-	1    0    0    -1
-$EndComp
-$Comp
-L power:+5V #PWR?
-U 1 1 5E9D8E3B
-P 9650 4600
-F 0 "#PWR?" H 9650 4450 50  0001 C CNN
-F 1 "+5V" H 9665 4773 50  0000 C CNN
-F 2 "" H 9650 4600 50  0001 C CNN
-F 3 "" H 9650 4600 50  0001 C CNN
-	1    9650 4600
 	1    0    0    -1
 $EndComp
@@
 $Comp
 L Device:R R?
-U 1 1 5E9D99AA
-P 9650 4800
-F 0 "R?" H 9720 4846 50  0000 L CNN
-F 1 "10k" H 9720 4755 50  0000 L CNN
-F 2 "Resistor_SMD:R_1206_3216Metric_Pad1.42x1.75mm_HandSolder" V 9580 4800 50  0001 C CNN
-F 3 "~" H 9650 4800 50  0001 C CNN
-	1    9650 4800
-	1    0    0    -1
-$EndComp
-$Comp
-L Device:R R?
 U 1 1 5E9D9C8C
 P 9650 5850
@@
 	1    0    0    -1
 $EndComp
-Wire Wire Line
-	9650 4600 9650 4650
-Wire Wire Line
-	9650 4950 9650 5050
-Connection ~ 9650 5050
-Wire Wire Line
-	9650 5050 10050 5050
 Wire Wire Line
 	9650 5650 9650 5700
@@
 Wire Notes Line
 	7000 6500 7000 4050
+Wire Wire Line
+	9300 5050 10050 5050
+Wire Wire Line
+	8050 6100 8900 6100
 $EndSCHEMATC
