File: PONG_Display/sensors.sch (KiCad schematic (older format))
At the start: 3 parts

Commit message: V3
Parts:
- added RV?: R_POT, symbol Device:R_POT
Connections:
- net LIGHT_SENSOR_IN is gone; now on net +5V: J?.1 (Pin_1)
- net GND: now also RV?.3
- net LIGHT_SENSOR_OUT: now also RV?.2; no longer J?.2 (Pin_2)
- new net: J?.2 (Pin_2), RV?.1
Other:
- note added: "Złącza do czujników"
- moved on the sheet: J?
Changed lines of the file:
@@
 $Descr A4 11693 8268
 encoding utf-8
-Sheet 3 6
+Sheet 4 6
 Title ""
 Date ""
@@
 L Connector_Generic:Conn_01x03 J?
 U 1 1 5E82C0DD
-P 9550 1800
+P 6250 2650
 AR Path="/5E80CCDD/5E82C0DD" Ref="J?"  Part="1"
 AR Path="/5E80B6DE/5E82C0DD" Ref="J?"  Part="1"
-F 0 "J?" H 9630 1842 50  0000 L CNN
-F 1 "DHT22_Conn" H 9630 1751 50  0000 L CNN
-F 2 "" H 9550 1800 50  0001 C CNN
-F 3 "~" H 9550 1800 50  0001 C CNN
-	1    9550 1800
+F 0 "J?" H 6330 2692 50  0000 L CNN
+F 1 "DHT22_Conn" H 6330 2601 50  0000 L CNN
+F 2 "" H 6250 2650 50  0001 C CNN
+F 3 "~" H 6250 2650 50  0001 C CNN
+	1    6250 2650
 	1    0    0    -1
 $EndComp
@@
 L Connector_Generic:Conn_01x02 J?
 U 1 1 5E82C0E3
-P 9550 2550
+P 6250 3600
 AR Path="/5E80CCDD/5E82C0E3" Ref="J?"  Part="1"
 AR Path="/5E80B6DE/5E82C0E3" Ref="J?"  Part="1"
-F 0 "J?" H 9630 2542 50  0000 L CNN
-F 1 "LightSensor_Conn" H 9630 2451 50  0000 L CNN
-F 2 "" H 9550 2550 50  0001 C CNN
-F 3 "~" H 9550 2550 50  0001 C CNN
-	1    9550 2550
+F 0 "J?" H 6330 3592 50  0000 L CNN
+F 1 "LightSensor_Conn" H 6330 3501 50  0000 L CNN
+F 2 "" H 6250 3600 50  0001 C CNN
+F 3 "~" H 6250 3600 50  0001 C CNN
+	1    6250 3600
 	1    0    0    -1
 $EndComp
-Text GLabel 9200 1800 0    50   Input ~ 0
+Text GLabel 4850 2650 0    50   Input ~ 0
 DHT22_DATA
 Wire Wire Line
-	9200 1800 9350 1800
-Text GLabel 9200 2550 0    50   Input ~ 0
-LIGHT_SENSOR_IN
-Text GLabel 9200 2650 0    50   Output ~ 0
+	4850 2650 6050 2650
+Text GLabel 5050 4150 0    50   Output ~ 0
 LIGHT_SENSOR_OUT
-Wire Wire Line
-	9200 2550 9350 2550
-Wire Wire Line
-	9200 2650 9350 2650
 $Comp
 L Connector_Generic:Conn_01x03 J?
 U 1 1 5E82C0F3
-P 9550 3250
+P 6250 4700
 AR Path="/5E80CCDD/5E82C0F3" Ref="J?"  Part="1"
 AR Path="/5E80B6DE/5E82C0F3" Ref="J?"  Part="1"
-F 0 "J?" H 9630 3292 50  0000 L CNN
-F 1 "PIR_Sensor_Conn" H 9630 3201 50  0000 L CNN
-F 2 "" H 9550 3250 50  0001 C CNN
-F 3 "~" H 9550 3250 50  0001 C CNN
-	1    9550 3250
+F 0 "J?" H 6330 4742 50  0000 L CNN
+F 1 "PIR_Sensor_Conn" H 6330 4651 50  0000 L CNN
+F 2 "" H 6250 4700 50  0001 C CNN
+F 3 "~" H 6250 4700 50  0001 C CNN
+	1    6250 4700
 	1    0    0    -1
 $EndComp
-Text GLabel 9200 3250 0    50   Output ~ 0
+Text GLabel 4750 4700 0    50   Output ~ 0
 PIR_OUT
-Wire Wire Line
-	9200 3250 9350 3250
 Text Notes 7750 7500 0    50   ~ 0
 Schemat układu czujników
 $Comp
-L power:+5V #PWR?
+L power:+5V #PWR0131
 U 1 1 5E853437
-P 9100 1600
-F 0 "#PWR?" H 9100 1450 50  0001 C CNN
-F 1 "+5V" H 9115 1773 50  0000 C CNN
-F 2 "" H 9100 1600 50  0001 C CNN
-F 3 "" H 9100 1600 50  0001 C CNN
-	1    9100 1600
+P 5800 2450
+F 0 "#PWR0131" H 5800 2300 50  0001 C CNN
+F 1 "+5V" H 5815 2623 50  0000 C CNN
+F 2 "" H 5800 2450 50  0001 C CNN
+F 3 "" H 5800 2450 50  0001 C CNN
+	1    5800 2450
 	1    0    0    -1
 $EndComp
 $Comp
-L power:+5V #PWR?
+L power:+5V #PWR0132
 U 1 1 5E853AD5
-P 9100 3050
-F 0 "#PWR?" H 9100 2900 50  0001 C CNN
-F 1 "+5V" H 9115 3223 50  0000 C CNN
-F 2 "" H 9100 3050 50  0001 C CNN
-F 3 "" H 9100 3050 50  0001 C CNN
-	1    9100 3050
+P 5800 4500
+F 0 "#PWR0132" H 5800 4350 50  0001 C CNN
+F 1 "+5V" H 5815 4673 50  0000 C CNN
+F 2 "" H 5800 4500 50  0001 C CNN
+F 3 "" H 5800 4500 50  0001 C CNN
+	1    5800 4500
 	1    0    0    -1
 $EndComp
 $Comp
-L power:GND #PWR?
+L power:GND #PWR0133
 U 1 1 5E854167
-P 9100 3500
-F 0 "#PWR?" H 9100 3250 50  0001 C CNN
-F 1 "GND" H 9105 3327 50  0000 C CNN
-F 2 "" H 9100 3500 50  0001 C CNN
-F 3 "" H 9100 3500 50  0001 C CNN
-	1    9100 3500
+P 5800 4950
+F 0 "#PWR0133" H 5800 4700 50  0001 C CNN
+F 1 "GND" H 5805 4777 50  0000 C CNN
+F 2 "" H 5800 4950 50  0001 C CNN
+F 3 "" H 5800 4950 50  0001 C CNN
+	1    5800 4950
 	1    0    0    -1
 $EndComp
 $Comp
-L power:GND #PWR?
+L power:GND #PWR0134
 U 1 1 5E85474C
-P 9100 2050
-F 0 "#PWR?" H 9100 1800 50  0001 C CNN
-F 1 "GND" H 9105 1877 50  0000 C CNN
-F 2 "" H 9100 2050 50  0001 C CNN
-F 3 "" H 9100 2050 50  0001 C CNN
-	1    9100 2050
+P 5800 2900
+F 0 "#PWR0134" H 5800 2650 50  0001 C CNN
+F 1 "GND" H 5805 2727 50  0000 C CNN
+F 2 "" H 5800 2900 50  0001 C CNN
+F 3 "" H 5800 2900 50  0001 C CNN
+	1    5800 2900
 	1    0    0    -1
 $EndComp
 Wire Wire Line
-	9100 1600 9100 1700
+	5800 2450 5800 2550
 Wire Wire Line
-	9100 1700 9350 1700
+	5800 2550 6050 2550
 Wire Wire Line
-	9100 2050 9100 1900
+	5800 2900 5800 2750
 Wire Wire Line
-	9100 1900 9350 1900
+	5800 2750 6050 2750
 Wire Wire Line
-	9100 3050 9100 3150
+	5800 4500 5800 4600
 Wire Wire Line
-	9100 3150 9350 3150
+	5800 4600 6050 4600
 Wire Wire Line
-	9100 3500 9100 3350
+	5800 4950 5800 4800
 Wire Wire Line
-	9100 3350 9350 3350
+	5800 4800 6050 4800
+Wire Notes Line
+	4000 1900 7750 1900
+Wire Notes Line
+	7750 1900 7750 5350
+Wire Notes Line
+	7750 5350 4000 5350
+Wire Notes Line
+	4000 5350 4000 1900
+Text Notes 4650 2150 0    50   ~ 0
+Złącza do czujników
+$Comp
+L power:+5V #PWR0135
+U 1 1 5E91534B
+P 5800 3500
+F 0 "#PWR0135" H 5800 3350 50  0001 C CNN
+F 1 "+5V" H 5815 3673 50  0000 C CNN
+F 2 "" H 5800 3500 50  0001 C CNN
+F 3 "" H 5800 3500 50  0001 C CNN
+	1    5800 3500
+	1    0    0    -1
+$EndComp
+Wire Wire Line
+	5800 3600 5800 3500
+Wire Wire Line
+	5800 3600 6050 3600
+Wire Wire Line
+	4750 4700 6050 4700
+$Comp
+L Device:R_POT RV?
+U 1 1 5E9C873A
+P 5450 3700
+F 0 "RV?" H 5380 3654 50  0000 R CNN
+F 1 "R_POT" H 5380 3745 50  0000 R CNN
+F 2 "" H 5450 3700 50  0001 C CNN
+F 3 "~" H 5450 3700 50  0001 C CNN
+	1    5450 3700
+	0    1    1    0
+$EndComp
+$Comp
+L power:GND #PWR0136
+U 1 1 5E9CD10E
+P 5100 3750
+F 0 "#PWR0136" H 5100 3500 50  0001 C CNN
+F 1 "GND" H 5105 3577 50  0000 C CNN
+F 2 "" H 5100 3750 50  0001 C CNN
+F 3 "" H 5100 3750 50  0001 C CNN
+	1    5100 3750
+	1    0    0    -1
+$EndComp
+Wire Wire Line
+	5450 3850 5450 4150
+Wire Wire Line
+	5450 4150 5050 4150
+Wire Wire Line
+	5100 3750 5100 3700
+Wire Wire Line
+	5100 3700 5300 3700
+Wire Wire Line
+	5600 3700 6050 3700
 $EndSCHEMATC

Commit message: Dodane footprinty
Parts:
- gave numbers to parts that had none: 4
Changed lines of the file:
@@
 P 6250 2650
 AR Path="/5E80CCDD/5E82C0DD" Ref="J?"  Part="1"
-AR Path="/5E80B6DE/5E82C0DD" Ref="J?"  Part="1"
-F 0 "J?" H 6330 2692 50  0000 L CNN
+AR Path="/5E80B6DE/5E82C0DD" Ref="J3"  Part="1"
+F 0 "J3" H 6330 2692 50  0000 L CNN
 F 1 "DHT22_Conn" H 6330 2601 50  0000 L CNN
 F 2 "" H 6250 2650 50  0001 C CNN
@@
 P 6250 3600
 AR Path="/5E80CCDD/5E82C0E3" Ref="J?"  Part="1"
-AR Path="/5E80B6DE/5E82C0E3" Ref="J?"  Part="1"
-F 0 "J?" H 6330 3592 50  0000 L CNN
+AR Path="/5E80B6DE/5E82C0E3" Ref="J4"  Part="1"
+F 0 "J4" H 6330 3592 50  0000 L CNN
 F 1 "LightSensor_Conn" H 6330 3501 50  0000 L CNN
 F 2 "" H 6250 3600 50  0001 C CNN
@@
 P 6250 4700
 AR Path="/5E80CCDD/5E82C0F3" Ref="J?"  Part="1"
-AR Path="/5E80B6DE/5E82C0F3" Ref="J?"  Part="1"
-F 0 "J?" H 6330 4742 50  0000 L CNN
+AR Path="/5E80B6DE/5E82C0F3" Ref="J5"  Part="1"
+F 0 "J5" H 6330 4742 50  0000 L CNN
 F 1 "PIR_Sensor_Conn" H 6330 4651 50  0000 L CNN
 F 2 "" H 6250 4700 50  0001 C CNN
@@
 	4750 4700 6050 4700
 $Comp
-L Device:R_POT RV?
+L Device:R_POT RV2
 U 1 1 5E9C873A
 P 5450 3700
-F 0 "RV?" H 5380 3654 50  0000 R CNN
+F 0 "RV2" H 5380 3654 50  0000 R CNN
 F 1 "R_POT" H 5380 3745 50  0000 R CNN
 F 2 "" H 5450 3700 50  0001 C CNN

Commit message: v2
Parts:
- J4: footprint (none) -> Connector_Molex:Molex_CLIK-Mate_502382-0270_1x02-1MP_P1.25mm_Vertical
- RV2: footprint (none) -> Potentiometer_THT:Potentiometer_Piher_PT-6-V_Vertical
Changed lines of the file:
@@
 F 0 "J4" H 6330 3592 50  0000 L CNN
 F 1 "LightSensor_Conn" H 6330 3501 50  0000 L CNN
-F 2 "" H 6250 3600 50  0001 C CNN
+F 2 "Connector_Molex:Molex_CLIK-Mate_502382-0270_1x02-1MP_P1.25mm_Vertical" H 6250 3600 50  0001 C CNN
 F 3 "~" H 6250 3600 50  0001 C CNN
 	1    6250 3600
@@
 F 0 "RV2" H 5380 3654 50  0000 R CNN
 F 1 "R_POT" H 5380 3745 50  0000 R CNN
-F 2 "" H 5450 3700 50  0001 C CNN
+F 2 "Potentiometer_THT:Potentiometer_Piher_PT-6-V_Vertical" H 5450 3700 50  0001 C CNN
 F 3 "~" H 5450 3700 50  0001 C CNN
 	1    5450 3700

Commit message: Updated
Parts:
- removed RV2: R_POT, Potentiometer_THT:Potentiometer_Piher_PT-6-V_Vertical, symbol Device:R_POT
Connections:
- net LIGHT_SENSOR_OUT: now also J4.2 (Pin_2)
Changed lines of the file:
@@
 Wire Wire Line
 	4850 2650 6050 2650
-Text GLabel 5050 4150 0    50   Output ~ 0
+Text GLabel 5650 3700 0    50   Output ~ 0
 LIGHT_SENSOR_OUT
 $Comp
@@
 Wire Wire Line
 	4750 4700 6050 4700
-$Comp
-L Device:R_POT RV2
-U 1 1 5E9C873A
-P 5450 3700
-F 0 "RV2" H 5380 3654 50  0000 R CNN
-F 1 "R_POT" H 5380 3745 50  0000 R CNN
-F 2 "Potentiometer_THT:Potentiometer_Piher_PT-6-V_Vertical" H 5450 3700 50  0001 C CNN
-F 3 "~" H 5450 3700 50  0001 C CNN
-	1    5450 3700
-	0    1    1    0
-$EndComp
-$Comp
-L power:GND #PWR0136
-U 1 1 5E9CD10E
-P 5100 3750
-F 0 "#PWR0136" H 5100 3500 50  0001 C CNN
-F 1 "GND" H 5105 3577 50  0000 C CNN
-F 2 "" H 5100 3750 50  0001 C CNN
-F 3 "" H 5100 3750 50  0001 C CNN
-	1    5100 3750
-	1    0    0    -1
-$EndComp
 Wire Wire Line
-	5450 3850 5450 4150
-Wire Wire Line
-	5450 4150 5050 4150
-Wire Wire Line
-	5100 3750 5100 3700
-Wire Wire Line
-	5100 3700 5300 3700
-Wire Wire Line
-	5600 3700 6050 3700
+	6050 3700 5650 3700
 $EndSCHEMATC

Commit message: Drobne zmiany
Parts:
- J3, J5: footprint (none) -> TerminalBlock:TerminalBlock_bornier-3_P5.08mm
Changed lines of the file:
@@
 F 0 "J3" H 6330 2692 50  0000 L CNN
 F 1 "DHT22_Conn" H 6330 2601 50  0000 L CNN
-F 2 "" H 6250 2650 50  0001 C CNN
+F 2 "TerminalBlock:TerminalBlock_bornier-3_P5.08mm" H 6250 2650 50  0001 C CNN
 F 3 "~" H 6250 2650 50  0001 C CNN
 	1    6250 2650
@@
 F 0 "J5" H 6330 4742 50  0000 L CNN
 F 1 "PIR_Sensor_Conn" H 6330 4651 50  0000 L CNN
-F 2 "" H 6250 4700 50  0001 C CNN
+F 2 "TerminalBlock:TerminalBlock_bornier-3_P5.08mm" H 6250 4700 50  0001 C CNN
 F 3 "~" H 6250 4700 50  0001 C CNN
 	1    6250 4700

Commit message: Zmiany
Parts:
- J3, J5: footprint TerminalBlock:TerminalBlock_bornier-3_P5.08mm -> TerminalBlock_Phoenix:TerminalBlock_Phoenix_PT-1,5-3-3.5-H_1x03_P3.50mm_Horizontal
- J4: footprint Connector_Molex:Molex_CLIK-Mate_502382-0270_1x02-1MP_P1.25mm_Vertical -> TerminalBlock_Phoenix:TerminalBlock_Phoenix_PT-1,5-2-3.5-H_1x02_P3.50mm_Horizontal
Changed lines of the file:
@@
 F 0 "J3" H 6330 2692 50  0000 L CNN
 F 1 "DHT22_Conn" H 6330 2601 50  0000 L CNN
-F 2 "TerminalBlock:TerminalBlock_bornier-3_P5.08mm" H 6250 2650 50  0001 C CNN
+F 2 "TerminalBlock_Phoenix:TerminalBlock_Phoenix_PT-1,5-3-3.5-H_1x03_P3.50mm_Horizontal" H 6250 2650 50  0001 C CNN
 F 3 "~" H 6250 2650 50  0001 C CNN
 	1    6250 2650
@@
 F 0 "J4" H 6330 3592 50  0000 L CNN
 F 1 "LightSensor_Conn" H 6330 3501 50  0000 L CNN
-F 2 "Connector_Molex:Molex_CLIK-Mate_502382-0270_1x02-1MP_P1.25mm_Vertical" H 6250 3600 50  0001 C CNN
+F 2 "TerminalBlock_Phoenix:TerminalBlock_Phoenix_PT-1,5-2-3.5-H_1x02_P3.50mm_Horizontal" H 6250 3600 50  0001 C CNN
 F 3 "~" H 6250 3600 50  0001 C CNN
 	1    6250 3600
@@
 F 0 "J5" H 6330 4742 50  0000 L CNN
 F 1 "PIR_Sensor_Conn" H 6330 4651 50  0000 L CNN
-F 2 "TerminalBlock:TerminalBlock_bornier-3_P5.08mm" H 6250 4700 50  0001 C CNN
+F 2 "TerminalBlock_Phoenix:TerminalBlock_Phoenix_PT-1,5-3-3.5-H_1x03_P3.50mm_Horizontal" H 6250 4700 50  0001 C CNN
 F 3 "~" H 6250 4700 50  0001 C CNN
 	1    6250 4700

Commit message: Teraz jest sexy
Connections:
- net +5V: now also J5.3 (Pin_3); no longer J5.1 (Pin_1)
- net GND: now also J5.1 (Pin_1); no longer J5.3 (Pin_3)
Changed lines of the file:
@@
 EESchema Schematic File Version 4
+LIBS:PONG_Display-cache
 EELAYER 30 0
 EELAYER END
@@
 	1    0    0    -1
 $EndComp
-Text GLabel 4850 2650 0    50   Input ~ 0
-DHT22_DATA
 Wire Wire Line
 	4850 2650 6050 2650
-Text GLabel 5650 3700 0    50   Output ~ 0
-LIGHT_SENSOR_OUT
 $Comp
 L Connector_Generic:Conn_01x03 J?
@@
 F 3 "~" H 6250 4700 50  0001 C CNN
 	1    6250 4700
-	1    0    0    -1
+	1    0    0    1
 $EndComp
-Text GLabel 4750 4700 0    50   Output ~ 0
-PIR_OUT
 Text Notes 7750 7500 0    50   ~ 0
 Schemat układu czujników
@@
 Wire Wire Line
 	6050 3700 5650 3700
+Text HLabel 4850 2650 0    50   Input ~ 0
+DHT22_DATA
+Text HLabel 5650 3700 0    50   Input ~ 0
+LIGHT_SENSOR_OUT
+Text HLabel 4750 4700 0    50   Input ~ 0
+PIR_OUT
 $EndSCHEMATC
