File: PONG_Display/sensors.sch (KiCad schematic (older format))
At the start: 3 parts, among them J3 DHT22_Conn, J4 LightSensor_Conn, J5 PIR_Sensor_Conn

Commit message: laayout6
Parts:
- removed J4: LightSensor_Conn, TerminalBlock_Phoenix:TerminalBlock_Phoenix_PT-1,5-2-3.5-H_1x02_P3.50mm_Horizontal, symbol Connector_Generic:Conn_01x02
- added J4: LightSensor_Conn, TerminalBlock_Phoenix:TerminalBlock_Phoenix_PT-1,5-3-3.5-H_1x03_P3.50mm_Horizontal, symbol Connector_Generic:Conn_01x03
Connections:
- net +5V: now also J4.1 (Pin_1)
- net GND: now also J4.3 (Pin_3)
- net LIGHT_SENSOR_OUT: now also J4.2 (Pin_2)
Changed lines of the file:
@@
-	1    0    0    -1
-$EndComp
-$Comp
-L Connector_Generic:Conn_01x02 J?
-U 1 1 5E82C0E3
-P 6250 3600
-AR Path="/5E80CCDD/5E82C0E3" Ref="J?"  Part="1"
-AR Path="/5E80B6DE/5E82C0E3" Ref="J4"  Part="1"
-F 0 "J4" H 6330 3592 50  0000 L CNN
-F 1 "LightSensor_Conn" H 6330 3501 50  0000 L CNN
-F 2 "TerminalBlock_Phoenix:TerminalBlock_Phoenix_PT-1,5-2-3.5-H_1x02_P3.50mm_Horizontal" H 6250 3600 50  0001 C CNN
-F 3 "~" H 6250 3600 50  0001 C CNN
-	1    6250 3600
 	1    0    0    -1
 $EndComp
@@
 Text HLabel 4750 4700 0    50   Input ~ 0
 PIR_OUT
+$Comp
+L Connector_Generic:Conn_01x03 J?
+U 1 1 5EAE2D4C
+P 6250 3700
+AR Path="/5E80CCDD/5EAE2D4C" Ref="J?"  Part="1"
+AR Path="/5E80B6DE/5EAE2D4C" Ref="J4"  Part="1"
+F 0 "J4" H 6330 3742 50  0000 L CNN
+F 1 "LightSensor_Conn" H 6330 3651 50  0000 L CNN
+F 2 "TerminalBlock_Phoenix:TerminalBlock_Phoenix_PT-1,5-3-3.5-H_1x03_P3.50mm_Horizontal" H 6250 3700 50  0001 C CNN
+F 3 "~" H 6250 3700 50  0001 C CNN
+	1    6250 3700
+	1    0    0    -1
+$EndComp
+$Comp
+L power:GND #PWR0112
+U 1 1 5EAE348C
+P 5800 3900
+F 0 "#PWR0112" H 5800 3650 50  0001 C CNN
+F 1 "GND" H 5805 3727 50  0000 C CNN
+F 2 "" H 5800 3900 50  0001 C CNN
+F 3 "" H 5800 3900 50  0001 C CNN
+	1    5800 3900
+	1    0    0    -1
+$EndComp
+Wire Wire Line
+	6050 3800 5800 3800
+Wire Wire Line
+	5800 3800 5800 3900
 $EndSCHEMATC

Commit message: layout8
Connections:
- net +5V: now also J5.1 (Pin_1); no longer J5.3 (Pin_3)
- net GND: now also J5.3 (Pin_3); no longer J5.1 (Pin_1)
Changed lines of the file:
@@
 F 3 "~" H 6250 4700 50  0001 C CNN
 	1    6250 4700
-	1    0    0    1
+	1    0    0    -1
 $EndComp
 Text Notes 7750 7500 0    50   ~ 0
