File: PONG_Display/microcontroler.sch (KiCad schematic (older format))
At the start: 30 parts, among them J6 AVR-ISP-10, SW1 SW_Push, U4 ATmega328P-AU, U5 MCP7940N-xST, Y1 16MHz, Y2 32,768kHz

Commit message: Zmianaa
Connections:
- net uC_RST renamed ESP_RST
Changed lines of the file:
@@
 	6300 4300 6300 4200
 Wire Wire Line
-	6150 3800 5500 3800
+	6150 3800 5650 3800
 Connection ~ 6150 3800
 $Comp
@@
 Wire Wire Line
 	3400 3700 3550 3700
+Text GLabel 5650 3650 1    50   Input ~ 0
+ESP_RST
+Wire Wire Line
+	5650 3650 5650 3800
+Connection ~ 5650 3800
+Wire Wire Line
+	5650 3800 5500 3800
 $EndSCHEMATC

Commit message: Teraz jest sexy
Parts:
- R7, R8: value 10k -> 2k2
Connections:
- no-connect marks 0 -> 13
Changed lines of the file:
@@
 EESchema Schematic File Version 4
+LIBS:PONG_Display-cache
 EELAYER 30 0
 EELAYER END
@@
 	1    0    0    -1
 $EndComp
-Text GLabel 2300 6550 2    50   BiDi ~ 0
-uC_MISO
-Text GLabel 2300 6650 2    50   BiDi ~ 0
-uC_MOSI
-Text GLabel 2300 6750 2    50   BiDi ~ 0
-uC_SCK
-Text GLabel 2300 6850 2    50   BiDi ~ 0
-uC_RST
 Wire Wire Line
 	1550 6050 1550 6250
@@
 Wire Wire Line
 	5200 3100 5350 3100
-Text GLabel 1100 1900 1    50   Input ~ 0
-LIGHT_SENSOR_OUT
 $Comp
 L power:+5V #PWR0142
@@
 Wire Wire Line
 	4300 5900 4300 6100
-Text GLabel 3550 2300 2    50   Output ~ 0
-DHT22_DATA
-Text GLabel 4000 4200 2    50   Input ~ 0
-PIR_SENSOR_OUT
 Wire Wire Line
 	3400 2300 3550 2300
@@
 Wire Wire Line
 	7200 3800 7450 3800
-Text GLabel 5500 3650 1    50   BiDi ~ 0
-uC_RST
-Wire Wire Line
-	5500 3650 5500 3800
-Connection ~ 5500 3800
-Wire Wire Line
-	5500 3800 3400 3800
-Text GLabel 3550 2700 2    50   BiDi ~ 0
-uC_MISO
-Text GLabel 3550 2600 2    50   BiDi ~ 0
-uC_MOSI
-Text GLabel 3550 2800 2    50   BiDi ~ 0
-uC_SCK
 Wire Wire Line
 	3400 2700 3550 2700
@@
 Text Notes 800  5650 0    50   ~ 0
 Złącze programowania mikrokontrolera
-Text GLabel 3550 4100 2    50   BiDi ~ 0
-ESP_RX
-Text GLabel 3550 4000 2    50   BiDi ~ 0
-ESP_TX
 Wire Wire Line
 	3400 4000 3550 4000
@@
 	1    0    0    -1
 $EndComp
-Text GLabel 8250 1700 0    50   BiDi ~ 0
-RTC_SCL
-Text GLabel 8250 1800 0    50   BiDi ~ 0
-RTC_SDA
 Wire Wire Line
 	8250 1700 8650 1700
@@
 P 8650 1150
 F 0 "R7" H 8720 1196 50  0000 L CNN
-F 1 "10k" H 8720 1105 50  0000 L CNN
+F 1 "2k2" H 8720 1105 50  0000 L CNN
 F 2 "Resistor_SMD:R_1206_3216Metric_Pad1.42x1.75mm_HandSolder" V 8580 1150 50  0001 C CNN
 F 3 "~" H 8650 1150 50  0001 C CNN
@@
 P 8900 1450
 F 0 "R8" H 8970 1496 50  0000 L CNN
-F 1 "10k" H 8970 1405 50  0000 L CNN
+F 1 "2k2" H 8970 1405 50  0000 L CNN
 F 2 "Resistor_SMD:R_1206_3216Metric_Pad1.42x1.75mm_HandSolder" V 8830 1450 50  0001 C CNN
 F 3 "~" H 8900 1450 50  0001 C CNN
@@
 Wire Wire Line
 	1250 2500 2200 2500
-Text GLabel 3550 3700 2    50   BiDi ~ 0
-RTC_SCL
-Text GLabel 3550 3600 2    50   BiDi ~ 0
-RTC_SDA
 Wire Wire Line
 	3400 3600 3550 3600
 Wire Wire Line
 	3400 3700 3550 3700
-Text GLabel 5650 3650 1    50   Input ~ 0
-ESP_RST
 Wire Wire Line
 	5650 3650 5650 3800
 Connection ~ 5650 3800
-Wire Wire Line
-	5650 3800 5500 3800
+Text HLabel 1100 1900 1    50   Input ~ 0
+LIGHT_SENSOR_OUT
+Text HLabel 4000 4200 2    50   Input ~ 0
+PIR_SENSOR_OUT
+Text HLabel 3550 2300 2    50   Input ~ 0
+DHT22_DATA
+Text HLabel 3550 4000 2    50   Input ~ 0
+ESP_TX
+Text HLabel 3550 4100 2    50   Input ~ 0
+ESP_RX
+Text Label 3550 3600 0    50   ~ 0
+RTC_SDA
+Text Label 3550 3700 0    50   ~ 0
+RTC_SCL
+Text Label 3550 2800 0    50   ~ 0
+uC_SCK
+Text Label 3550 2700 0    50   ~ 0
+uC_MISO
+Text Label 3550 2600 0    50   ~ 0
+uC_MOSI
+Text Label 2300 6550 0    50   ~ 0
+uC_MISO
+Text Label 2300 6650 0    50   ~ 0
+uC_MOSI
+Text Label 2300 6750 0    50   ~ 0
+uC_SCK
+Text Label 2300 6850 0    50   ~ 0
+uC_RST
+Text Label 5150 3800 0    50   ~ 0
+uC_RST
+Wire Wire Line
+	3400 3800 5650 3800
+Text HLabel 5650 3650 1    50   Input ~ 0
+ESP_RST
+NoConn ~ 2200 2600
+NoConn ~ 3400 2400
+NoConn ~ 3400 2500
+NoConn ~ 3400 3200
+NoConn ~ 3400 3300
+NoConn ~ 3400 3400
+NoConn ~ 3400 3500
+NoConn ~ 3400 4300
+NoConn ~ 3400 4400
+NoConn ~ 3400 4500
+NoConn ~ 3400 4600
+NoConn ~ 3400 4700
+NoConn ~ 9150 2000
+Text Label 8250 1700 0    50   ~ 0
+RTC_SCL
+Text Label 8250 1800 0    50   ~ 0
+RTC_SDA
 $EndSCHEMATC

Commit message: 2
Parts:
- Y2: footprint Crystal:Crystal_C38-LF_D3.0mm_L8.0mm_Horizontal -> Crystal:Crystal_C26-LF_D2.1mm_L6.5mm_Horizontal
Connections:
- net LED_DATA: now reaches U4.13 (PB1)
- no-connect marks 13 -> 12
Changed lines of the file:
@@
 EESchema Schematic File Version 4
-LIBS:PONG_Display-cache
 EELAYER 30 0
 EELAYER END
@@
 F 0 "Y2" V 10104 2031 50  0000 L CNN
 F 1 "32,768kHz" V 10195 2031 50  0000 L CNN
-F 2 "Crystal:Crystal_C38-LF_D3.0mm_L8.0mm_Horizontal" H 10150 1900 50  0001 C CNN
+F 2 "Crystal:Crystal_C26-LF_D2.1mm_L6.5mm_Horizontal" H 10150 1900 50  0001 C CNN
 F 3 "~" H 10150 1900 50  0001 C CNN
 	1    10150 1900
@@
 ESP_RST
 NoConn ~ 2200 2600
-NoConn ~ 3400 2400
 NoConn ~ 3400 2500
 NoConn ~ 3400 3200
@@
 Text Label 8250 1800 0    50   ~ 0
 RTC_SDA
+Text HLabel 3550 2400 2    50   Input ~ 0
+LED_DATA
+Wire Wire Line
+	3550 2400 3400 2400
 $EndSCHEMATC

Commit message: foot
Parts:
- U5: footprint Package_SO:TSSOP-8_4.4x3mm_P0.65mm -> Package_SO:SOIC-8_3.9x4.9mm_P1.27mm
Connections:
- net LED_DATA: no longer U4.13 (PB1)
Changed lines of the file:
@@
 F 0 "U5" H 9850 1400 50  0000 C CNN
 F 1 "MCP7940N-xST" H 9900 1300 50  0000 C CNN
-F 2 "Package_SO:TSSOP-8_4.4x3mm_P0.65mm" H 9550 1900 50  0001 C CNN
+F 2 "Package_SO:SOIC-8_3.9x4.9mm_P1.27mm" H 9550 1900 50  0001 C CNN
 F 3 "http://ww1.microchip.com/downloads/en/DeviceDoc/20005010F.pdf" H 9550 1900 50  0001 C CNN
 	1    9550 1900
@@
 Text HLabel 3550 2400 2    50   Input ~ 0
 LED_DATA
-Wire Wire Line
-	3550 2400 3400 2400
 $EndSCHEMATC

Commit message: 23
Connections:
- net ESP_RST renamed uC_RST
Changed lines of the file:
@@
 Wire Wire Line
 	6300 4300 6300 4200
-Wire Wire Line
-	6150 3800 5650 3800
 Connection ~ 6150 3800
 $Comp
@@
 Wire Wire Line
 	3400 3700 3550 3700
-Wire Wire Line
-	5650 3650 5650 3800
-Connection ~ 5650 3800
 Text HLabel 1100 1900 1    50   Input ~ 0
 LIGHT_SENSOR_OUT
@@
 Text Label 5150 3800 0    50   ~ 0
 uC_RST
-Wire Wire Line
-	3400 3800 5650 3800
-Text HLabel 5650 3650 1    50   Input ~ 0
-ESP_RST
 NoConn ~ 2200 2600
 NoConn ~ 3400 2500
@@
 Text HLabel 3550 2400 2    50   Input ~ 0
 LED_DATA
+Wire Wire Line
+	3400 3800 6150 3800
 $EndSCHEMATC

Commit message: po obgadaniu
Parts:
- added J9: Conn_01x04, symbol Connector_Generic:Conn_01x04
- R7, R8: value 2k2 -> 10k
- U5: value MCP7940N-xST -> MCP79400
Connections:
- net +3V3: no longer U5.8 (VCC)
- net +5V: now also U5.8 (VCC)
- net LED_DATA: now also U4.13 (PB1)
- net uC_GPIO0: now reaches U4.23 (PC0)
- net uC_GPIO0: now also J9.1 (Pin_1)
- net uC_GPIO1: now reaches U4.24 (PC1)
- net uC_GPIO1: now also J9.2 (Pin_2)
- net uC_GPIO2: now reaches U4.25 (PC2)
- net uC_GPIO2: now also J9.3 (Pin_3)
- net uC_GPIO3: now reaches U4.26 (PC3)
- net uC_GPIO3: now also J9.4 (Pin_4)
- no-connect marks 12 -> 8
Changed lines of the file:
@@
 EESchema Schematic File Version 4
+LIBS:PONG_Display-cache
 EELAYER 30 0
 EELAYER END
@@
 P 9550 1900
 F 0 "U5" H 9850 1400 50  0000 C CNN
-F 1 "MCP7940N-xST" H 9900 1300 50  0000 C CNN
+F 1 "MCP79400" H 9900 1300 50  0000 C CNN
 F 2 "Package_SO:SOIC-8_3.9x4.9mm_P1.27mm" H 9550 1900 50  0001 C CNN
 F 3 "http://ww1.microchip.com/downloads/en/DeviceDoc/20005010F.pdf" H 9550 1900 50  0001 C CNN
 	1    9550 1900
-	1    0    0    -1
-$EndComp
-$Comp
-L power:+3.3V #PWR0154
-U 1 1 5E93C01F
-P 9550 1100
-F 0 "#PWR0154" H 9550 950 50  0001 C CNN
-F 1 "+3.3V" H 9565 1273 50  0000 C CNN
-F 2 "" H 9550 1100 50  0001 C CNN
-F 3 "" H 9550 1100 50  0001 C CNN
-	1    9550 1100
 	1    0    0    -1
 $EndComp
@@
 P 8650 1150
 F 0 "R7" H 8720 1196 50  0000 L CNN
-F 1 "2k2" H 8720 1105 50  0000 L CNN
+F 1 "10k" H 8720 1105 50  0000 L CNN
 F 2 "Resistor_SMD:R_1206_3216Metric_Pad1.42x1.75mm_HandSolder" V 8580 1150 50  0001 C CNN
 F 3 "~" H 8650 1150 50  0001 C CNN
@@
 P 8900 1450
 F 0 "R8" H 8970 1496 50  0000 L CNN
-F 1 "2k2" H 8970 1405 50  0000 L CNN
+F 1 "10k" H 8970 1405 50  0000 L CNN
 F 2 "Resistor_SMD:R_1206_3216Metric_Pad1.42x1.75mm_HandSolder" V 8830 1450 50  0001 C CNN
 F 3 "~" H 8900 1450 50  0001 C CNN
@@
 NoConn ~ 2200 2600
 NoConn ~ 3400 2500
-NoConn ~ 3400 3200
-NoConn ~ 3400 3300
-NoConn ~ 3400 3400
-NoConn ~ 3400 3500
 NoConn ~ 3400 4300
 NoConn ~ 3400 4400
@@
 NoConn ~ 3400 4700
 NoConn ~ 9150 2000
-Text Label 8250 1700 0    50   ~ 0
+Text Label 8250 1700 2    50   ~ 0
 RTC_SCL
-Text Label 8250 1800 0    50   ~ 0
+Text Label 8250 1800 2    50   ~ 0
 RTC_SDA
 Text HLabel 3550 2400 2    50   Input ~ 0
@@
 Wire Wire Line
 	3400 3800 6150 3800
+Wire Wire Line
+	3550 2400 3400 2400
+$Comp
+L power:+5V #PWR0154
+U 1 1 5E9BD4A6
+P 9550 1100
+F 0 "#PWR0154" H 9550 950 50  0001 C CNN
+F 1 "+5V" H 9565 1273 50  0000 C CNN
+F 2 "" H 9550 1100 50  0001 C CNN
+F 3 "" H 9550 1100 50  0001 C CNN
+	1    9550 1100
+	1    0    0    -1
+$EndComp
+Text Label 3750 3300 0    50   ~ 0
+uC_GPIO1
+Text Label 3750 3400 0    50   ~ 0
+uC_GPIO2
+Text Label 3750 3500 0    50   ~ 0
+uC_GPIO3
+$Comp
+L Connector_Generic:Conn_01x04 J9
+U 1 1 5E9D6920
+P 4350 3300
+F 0 "J9" H 4430 3292 50  0000 L CNN
+F 1 "Conn_01x04" H 4430 3201 50  0000 L CNN
+F 2 "" H 4350 3300 50  0001 C CNN
+F 3 "~" H 4350 3300 50  0001 C CNN
+	1    4350 3300
+	1    0    0    -1
+$EndComp
+Text Label 3750 3200 0    50   ~ 0
+uC_GPIO0
+Wire Wire Line
+	3400 3200 4150 3200
+Wire Wire Line
+	3400 3300 4150 3300
+Wire Wire Line
+	3400 3400 4150 3400
+Wire Wire Line
+	3400 3500 4150 3500
 $EndSCHEMATC

Commit message: 5v
Parts:
- J7: renamed from J9; footprint (none) -> Connector_PinHeader_2.54mm:PinHeader_1x04_P2.54mm_Vertical
- renumbered C16 to C10, C17 to C11, C18 to C12, C19 to C13, C20 to C14, C21 to C15, C22 to C16, C23 to C17, C24 to C18, C25 to C19, C26 to C20, C27 to C21, C12 to C6, C13 to C7, C14 to C8, C15 to C9, D4 to D3, L2 to L1, R5 to R4, R6 to R5, R7 to R6, R8 to R7, RV2 to RV1, U4 to U3, U5 to U4

Commit message: jeszcze do przekminienia
Connections:
- net ESP_RX renamed ESP_RX_HIGH
- net ESP_TX renamed ESP_TX_HIGH
Changed lines of the file:
@@
 EESchema Schematic File Version 4
+LIBS:PONG_Display-cache
 EELAYER 30 0
 EELAYER END
@@
 DHT22_DATA
 Text HLabel 3550 4000 2    50   Input ~ 0
-ESP_TX
+ESP_TX_HIGH
 Text HLabel 3550 4100 2    50   Input ~ 0
-ESP_RX
+ESP_RX_HIGH
 Text Label 3550 3600 0    50   ~ 0
 RTC_SDA
