File: PONG_Display/microcontroler.sch (KiCad schematic (older format))
At the start: 31 parts, among them J6 AVR-ISP-10, J7 Conn_01x04, SW1 SW_Push, U3 ATmega328P-AU, U4 MCP79400, Y1 16MHz, Y2 32,768kHz

Commit message: layout v1
Parts:
- C10, C11, C12, C13, C14, C17, C18, C19, C6, C7, C8, C9: footprint Capacitor_SMD:C_1206_3216Metric_Pad1.42x1.75mm_HandSolder -> Capacitor_SMD:C_0603_1608Metric_Pad1.05x0.95mm_HandSolder
Changed lines of the file:
@@
 EESchema Schematic File Version 4
-LIBS:PONG_Display-cache
 EELAYER 30 0
 EELAYER END
@@
 F 0 "C9" H 3965 5796 50  0000 L CNN
 F 1 "100n" H 3965 5705 50  0000 L CNN
-F 2 "Capacitor_SMD:C_1206_3216Metric_Pad1.42x1.75mm_HandSolder" H 3888 5600 50  0001 C CNN
+F 2 "Capacitor_SMD:C_0603_1608Metric_Pad1.05x0.95mm_HandSolder" H 3888 5600 50  0001 C CNN
 F 3 "~" H 3850 5750 50  0001 C CNN
 	1    3850 5750
@@
 F 0 "C11" H 4415 5796 50  0000 L CNN
 F 1 "100n" H 4415 5705 50  0000 L CNN
-F 2 "Capacitor_SMD:C_1206_3216Metric_Pad1.42x1.75mm_HandSolder" H 4338 5600 50  0001 C CNN
+F 2 "Capacitor_SMD:C_0603_1608Metric_Pad1.05x0.95mm_HandSolder" H 4338 5600 50  0001 C CNN
 F 3 "~" H 4300 5750 50  0001 C CNN
 	1    4300 5750
@@
 F 0 "C7" H 2065 1646 50  0000 L CNN
 F 1 "100n" H 2065 1555 50  0000 L CNN
-F 2 "Capacitor_SMD:C_1206_3216Metric_Pad1.42x1.75mm_HandSolder" H 1988 1450 50  0001 C CNN
+F 2 "Capacitor_SMD:C_0603_1608Metric_Pad1.05x0.95mm_HandSolder" H 1988 1450 50  0001 C CNN
 F 3 "~" H 1950 1600 50  0001 C CNN
 	1    1950 1600
@@
 F 0 "C6" H 1965 2946 50  0000 L CNN
 F 1 "100n" H 1965 2855 50  0000 L CNN
-F 2 "Capacitor_SMD:C_1206_3216Metric_Pad1.42x1.75mm_HandSolder" H 1888 2750 50  0001 C CNN
+F 2 "Capacitor_SMD:C_0603_1608Metric_Pad1.05x0.95mm_HandSolder" H 1888 2750 50  0001 C CNN
 F 3 "~" H 1850 2900 50  0001 C CNN
 	1    1850 2900
@@
 F 0 "C8" H 3565 1646 50  0000 L CNN
 F 1 "100n" H 3565 1555 50  0000 L CNN
-F 2 "Capacitor_SMD:C_1206_3216Metric_Pad1.42x1.75mm_HandSolder" H 3488 1450 50  0001 C CNN
+F 2 "Capacitor_SMD:C_0603_1608Metric_Pad1.05x0.95mm_HandSolder" H 3488 1450 50  0001 C CNN
 F 3 "~" H 3450 1600 50  0001 C CNN
 	1    3450 1600
@@
 F 0 "C19" H 6415 4096 50  0000 L CNN
 F 1 "100n" H 6415 4005 50  0000 L CNN
-F 2 "Capacitor_SMD:C_1206_3216Metric_Pad1.42x1.75mm_HandSolder" H 6338 3900 50  0001 C CNN
+F 2 "Capacitor_SMD:C_0603_1608Metric_Pad1.05x0.95mm_HandSolder" H 6338 3900 50  0001 C CNN
 F 3 "~" H 6300 4050 50  0001 C CNN
 	1    6300 4050
@@
 F 0 "C13" H 4915 5796 50  0000 L CNN
 F 1 "100n" H 4915 5705 50  0000 L CNN
-F 2 "Capacitor_SMD:C_1206_3216Metric_Pad1.42x1.75mm_HandSolder" H 4838 5600 50  0001 C CNN
+F 2 "Capacitor_SMD:C_0603_1608Metric_Pad1.05x0.95mm_HandSolder" H 4838 5600 50  0001 C CNN
 F 3 "~" H 4800 5750 50  0001 C CNN
 	1    4800 5750
@@
 F 0 "C10" H 3965 7046 50  0000 L CNN
 F 1 "100n" H 3965 6955 50  0000 L CNN
-F 2 "Capacitor_SMD:C_1206_3216Metric_Pad1.42x1.75mm_HandSolder" H 3888 6850 50  0001 C CNN
+F 2 "Capacitor_SMD:C_0603_1608Metric_Pad1.05x0.95mm_HandSolder" H 3888 6850 50  0001 C CNN
 F 3 "~" H 3850 7000 50  0001 C CNN
 	1    3850 7000
@@
 F 0 "C12" H 4465 7046 50  0000 L CNN
 F 1 "100n" H 4465 6955 50  0000 L CNN
-F 2 "Capacitor_SMD:C_1206_3216Metric_Pad1.42x1.75mm_HandSolder" H 4388 6850 50  0001 C CNN
+F 2 "Capacitor_SMD:C_0603_1608Metric_Pad1.05x0.95mm_HandSolder" H 4388 6850 50  0001 C CNN
 F 3 "~" H 4350 7000 50  0001 C CNN
 	1    4350 7000
@@
 F 0 "C14" H 4915 7046 50  0000 L CNN
 F 1 "100n" H 4915 6955 50  0000 L CNN
-F 2 "Capacitor_SMD:C_1206_3216Metric_Pad1.42x1.75mm_HandSolder" H 4838 6850 50  0001 C CNN
+F 2 "Capacitor_SMD:C_0603_1608Metric_Pad1.05x0.95mm_HandSolder" H 4838 6850 50  0001 C CNN
 F 3 "~" H 4800 7000 50  0001 C CNN
 	1    4800 7000
@@
 F 0 "C17" H 5415 5796 50  0000 L CNN
 F 1 "100n" H 5415 5705 50  0000 L CNN
-F 2 "Capacitor_SMD:C_1206_3216Metric_Pad1.42x1.75mm_HandSolder" H 5338 5600 50  0001 C CNN
+F 2 "Capacitor_SMD:C_0603_1608Metric_Pad1.05x0.95mm_HandSolder" H 5338 5600 50  0001 C CNN
 F 3 "~" H 5300 5750 50  0001 C CNN
 	1    5300 5750
@@
 F 0 "C18" H 5415 7046 50  0000 L CNN
 F 1 "100n" H 5415 6955 50  0000 L CNN
-F 2 "Capacitor_SMD:C_1206_3216Metric_Pad1.42x1.75mm_HandSolder" H 5338 6850 50  0001 C CNN
+F 2 "Capacitor_SMD:C_0603_1608Metric_Pad1.05x0.95mm_HandSolder" H 5338 6850 50  0001 C CNN
 F 3 "~" H 5300 7000 50  0001 C CNN
 	1    5300 7000

Commit message: layout2
Connections:
- net +3V3: no longer C10.1
- net +5V: now also C10.1
Changed lines of the file:
@@
 	4800 7150 4800 7350
-$Comp
-L power:+3.3V #PWR035
-U 1 1 5E99B4C6
-P 3850 6700
-F 0 "#PWR035" H 3850 6550 50  0001 C CNN
-F 1 "+3.3V" H 3865 6873 50  0000 C CNN
-F 2 "" H 3850 6700 50  0001 C CNN
-F 3 "" H 3850 6700 50  0001 C CNN
-	1    3850 6700
-	1    0    0    -1
-$EndComp
 $Comp
 L power:+3.3V #PWR039
@@
 Wire Wire Line
 	3400 3500 4150 3500
+$Comp
+L power:+5V #PWR?
+U 1 1 5EAE1A08
+P 3850 6700
+F 0 "#PWR?" H 3850 6550 50  0001 C CNN
+F 1 "+5V" H 3865 6873 50  0000 C CNN
+F 2 "" H 3850 6700 50  0001 C CNN
+F 3 "" H 3850 6700 50  0001 C CNN
+	1    3850 6700
+	1    0    0    -1
+$EndComp
 $EndSCHEMATC

Commit message: l
Parts:
- C15, C16, C20, C21: footprint Capacitor_SMD:C_1206_3216Metric_Pad1.42x1.75mm_HandSolder -> Capacitor_SMD:C_0603_1608Metric_Pad1.05x0.95mm_HandSolder
- R4, R5, R6, R7: footprint Resistor_SMD:R_1206_3216Metric_Pad1.42x1.75mm_HandSolder -> Resistor_SMD:R_0603_1608Metric_Pad1.05x0.95mm_HandSolder
Changed lines of the file:
@@
 F 0 "C15" V 4798 2800 50  0000 C CNN
 F 1 "22p" V 4889 2800 50  0000 C CNN
-F 2 "Capacitor_SMD:C_1206_3216Metric_Pad1.42x1.75mm_HandSolder" H 5088 2650 50  0001 C CNN
+F 2 "Capacitor_SMD:C_0603_1608Metric_Pad1.05x0.95mm_HandSolder" H 5088 2650 50  0001 C CNN
 F 3 "~" H 5050 2800 50  0001 C CNN
 	1    5050 2800
@@
 F 0 "C16" V 4900 3100 50  0000 C CNN
 F 1 "22p" V 4800 3100 50  0000 C CNN
-F 2 "Capacitor_SMD:C_1206_3216Metric_Pad1.42x1.75mm_HandSolder" H 5088 2950 50  0001 C CNN
+F 2 "Capacitor_SMD:C_0603_1608Metric_Pad1.05x0.95mm_HandSolder" H 5088 2950 50  0001 C CNN
 F 3 "~" H 5050 3100 50  0001 C CNN
 	1    5050 3100
@@
 F 0 "R4" H 6220 3596 50  0000 L CNN
 F 1 "10k" H 6220 3505 50  0000 L CNN
-F 2 "Resistor_SMD:R_1206_3216Metric_Pad1.42x1.75mm_HandSolder" V 6080 3550 50  0001 C CNN
+F 2 "Resistor_SMD:R_0603_1608Metric_Pad1.05x0.95mm_HandSolder" V 6080 3550 50  0001 C CNN
 F 3 "~" H 6150 3550 50  0001 C CNN
 	1    6150 3550
@@
 F 0 "R5" H 7520 4196 50  0000 L CNN
 F 1 "330R" H 7520 4105 50  0000 L CNN
-F 2 "Resistor_SMD:R_1206_3216Metric_Pad1.42x1.75mm_HandSolder" V 7380 4150 50  0001 C CNN
+F 2 "Resistor_SMD:R_0603_1608Metric_Pad1.05x0.95mm_HandSolder" V 7380 4150 50  0001 C CNN
 F 3 "~" H 7450 4150 50  0001 C CNN
 	1    7450 4150
@@
 F 0 "C20" V 10048 1600 50  0000 C CNN
 F 1 "22p" V 10139 1600 50  0000 C CNN
-F 2 "Capacitor_SMD:C_1206_3216Metric_Pad1.42x1.75mm_HandSolder" H 10338 1450 50  0001 C CNN
+F 2 "Capacitor_SMD:C_0603_1608Metric_Pad1.05x0.95mm_HandSolder" H 10338 1450 50  0001 C CNN
 F 3 "~" H 10300 1600 50  0001 C CNN
 	1    10300 1600
@@
 F 0 "C21" V 10150 2200 50  0000 C CNN
 F 1 "22p" V 10050 2200 50  0000 C CNN
-F 2 "Capacitor_SMD:C_1206_3216Metric_Pad1.42x1.75mm_HandSolder" H 10338 2050 50  0001 C CNN
+F 2 "Capacitor_SMD:C_0603_1608Metric_Pad1.05x0.95mm_HandSolder" H 10338 2050 50  0001 C CNN
 F 3 "~" H 10300 2200 50  0001 C CNN
 	1    10300 2200
@@
 F 0 "R6" H 8720 1196 50  0000 L CNN
 F 1 "10k" H 8720 1105 50  0000 L CNN
-F 2 "Resistor_SMD:R_1206_3216Metric_Pad1.42x1.75mm_HandSolder" V 8580 1150 50  0001 C CNN
+F 2 "Resistor_SMD:R_0603_1608Metric_Pad1.05x0.95mm_HandSolder" V 8580 1150 50  0001 C CNN
 F 3 "~" H 8650 1150 50  0001 C CNN
 	1    8650 1150
@@
 F 0 "R7" H 8970 1496 50  0000 L CNN
 F 1 "10k" H 8970 1405 50  0000 L CNN
-F 2 "Resistor_SMD:R_1206_3216Metric_Pad1.42x1.75mm_HandSolder" V 8830 1450 50  0001 C CNN
+F 2 "Resistor_SMD:R_0603_1608Metric_Pad1.05x0.95mm_HandSolder" V 8830 1450 50  0001 C CNN
 F 3 "~" H 8900 1450 50  0001 C CNN
 	1    8900 1450
@@
 	3400 3500 4150 3500
 $Comp
-L power:+5V #PWR?
+L power:+5V #PWR0108
 U 1 1 5EAE1A08
 P 3850 6700
-F 0 "#PWR?" H 3850 6550 50  0001 C CNN
+F 0 "#PWR0108" H 3850 6550 50  0001 C CNN
 F 1 "+5V" H 3865 6873 50  0000 C CNN
 F 2 "" H 3850 6700 50  0001 C CNN

Commit message: layout4
Parts:
- removed J6: AVR-ISP-10, Connector_IDC:IDC-Header_2x05_P2.54mm_Vertical, symbol PONG_Display-rescue:AVR-ISP-10-Connector
- added J?: AVR-ISP-6, symbol Connector:AVR-ISP-6
Connections:
- net +5V: now also J?.2 (VCC)
- net GND: now also J?.6 (GND)
- net uC_MISO: now also J?.1 (MISO)
- net uC_MOSI: now also J?.4 (MOSI)
- net uC_RST: now also J?.5 (~RST)
- net uC_SCK: now also J?.3 (SCK)
Changed lines of the file:
@@
 Comment4 ""
 $EndDescr
-$Comp
-L PONG_Display-rescue:AVR-ISP-10-Connector J?
-U 1 1 5E830B15
-P 1650 6750
-AR Path="/5E80CCDD/5E830B15" Ref="J?"  Part="1"
-AR Path="/5E80B18F/5E830B15" Ref="J6"  Part="1"
-AR Path="/5E830B15" Ref="J?"  Part="1"
-F 0 "J6" H 1320 6846 50  0000 R CNN
-F 1 "AVR-ISP-10" H 1320 6755 50  0000 R CNN
-F 2 "Connector_IDC:IDC-Header_2x05_P2.54mm_Vertical" V 1400 6800 50  0001 C CNN
-F 3 " ~" H 375 6200 50  0001 C CNN
-	1    1650 6750
-	1    0    0    -1
-$EndComp
 Wire Wire Line
 	1550 6050 1550 6250
@@
 	1    0    0    -1
 $EndComp
+$Comp
+L Connector:AVR-ISP-6 J?
+U 1 1 5EA88C51
+P 1650 6750
+F 0 "J?" H 1321 6846 50  0000 R CNN
+F 1 "AVR-ISP-6" H 1321 6755 50  0000 R CNN
+F 2 "" V 1400 6800 50  0001 C CNN
+F 3 " ~" H 375 6200 50  0001 C CNN
+	1    1650 6750
+	1    0    0    -1
+$EndComp
