File: PONG_Display/PONG_Display.kicad_pcb (KiCad board)
At the start: 2 copper layers, 61 parts, among them J1 LED_Display_Conn, J2 Input_Supply+12V, J3 DHT22_Conn, J4 LightSensor_Conn, J5 PIR_Sensor_Conn, J6 AVR-ISP-10, J7 Conn_01x04, J8 ESP_Conn, J9 ESP_Prog_Conn, SW1 SW_Push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

Commit message: layout v1
Parts:
- added Q1: BSS138, Package_TO_SOT_SMD:SOT-23, B.Cu at (25.4, 52.1)
- added Q2: BSS138, Package_TO_SOT_SMD:SOT-23, B.Cu at (35.6, 52.1)
- added R10: 10k, Resistor_SMD:R_1206_3216Metric_Pad1.42x1.75mm_HandSolder, B.Cu at (25.2, 48.3)
- added R11: 10k, Resistor_SMD:R_1206_3216Metric_Pad1.42x1.75mm_HandSolder, B.Cu at (35.6, 48.3)
- added R12: 10k, Resistor_SMD:R_1206_3216Metric_Pad1.42x1.75mm_HandSolder, B.Cu at (25.4, 57.1)
- added R13: 10k, Resistor_SMD:R_1206_3216Metric_Pad1.42x1.75mm_HandSolder, B.Cu at (35.8, 57.1)
- C1, C5, C9: footprint Capacitor_SMD:C_1206_3216Metric_Pad1.42x1.75mm_HandSolder -> Capacitor_SMD:C_0603_1608Metric_Pad1.05x0.95mm_HandSolder
- C10, C11, C12, C13, C14, C17, C18, C19, C22, C3, C6, C7, C8: footprint Capacitor_SMD:C_1206_3216Metric_Pad1.42x1.75mm_HandSolder -> Capacitor_SMD:C_0603_1608Metric_Pad1.05x0.95mm_HandSolder; moved to B.Cu
- C20, C21, R4, R5, R6, R8, R9: moved to B.Cu
- C4: footprint Capacitor_THT:CP_Radial_D4.0mm_P2.00mm -> Capacitor_SMD:C_1206_3216Metric_Pad1.42x1.75mm_HandSolder
- F1: footprint Fuse:Fuseholder_Cylinder-5x20mm_Schurter_FAB_0031-355x_Horizontal_Closed -> Fuse:Fuseholder_Cylinder-5x20mm_Schurter_0031_8201_Horizontal_Open
- moved C18 349.0 mm to (15.2, 41.9), turned to 90 degrees
- moved R8 339.2 mm to (22.9, 79.4), turned to 90 degrees
- moved C12 318.0 mm to (30.5, 36.8)
- moved C22 318.0 mm to (38.1, 74.3), turned to 270 degrees
- moved C14 313.5 mm to (30.1, 79.4)
- moved C13 310.2 mm to (50.8, 19.1), turned to 270 degrees
- moved C7 307.7 mm to (52.7, 49.9), turned to 90 degrees
- moved C10 305.4 mm to (50.6, 72.4), turned to 180 degrees
- moved C16 296.2 mm to (46.6, 61.0), turned to 180 degrees
- moved C15 295.9 mm to (46.6, 55.9)
- moved C20 294.7 mm to (53.8, 32.4)
- moved C21 294.7 mm to (53.8, 38.1), turned to 180 degrees
- moved C11 289.8 mm to (52.7, 46.1), turned to 90 degrees
- moved C17 286.9 mm to (80.6, 72.4)
- moved C6 286.8 mm to (61.6, 49.5), turned to 180 degrees
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Connections:
- D4 pad 1: +5V -> +3V3
- J1 pad 1: +5V -> Net-(J1-Pad1)
- J1 pad 3: GND -> Net-(J1-Pad3)
- J8 pad 1: /MikrokontrolerAtmega/ESP_RX -> /Moduł WiFi/ESP_RX
- J8 pad 8: /MikrokontrolerAtmega/ESP_TX -> /Moduł WiFi/ESP_TX
- J9 pad 2: /MikrokontrolerAtmega/ESP_RX -> /Moduł WiFi/ESP_RX
- J9 pad 3: /MikrokontrolerAtmega/ESP_TX -> /Moduł WiFi/ESP_TX
- R8 pad 1: +5V -> +3V3
- U3 pad 30: /MikrokontrolerAtmega/ESP_TX -> /MikrokontrolerAtmega/ESP_TX_HIGH
- U3 pad 31: /MikrokontrolerAtmega/ESP_RX -> /MikrokontrolerAtmega/ESP_RX_HIGH
Routing:
- net /MikrokontrolerAtmega/uC_MOSI: track 0.00 -> 48.3 mm, vias 0 -> 1
- net /MikrokontrolerAtmega/uC_MISO: track 0.00 -> 48.3 mm
- net /MikrokontrolerAtmega/uC_SCK: track 0.00 -> 46.4 mm
- net Net-(BT1-Pad1): track 0.00 -> 41.5 mm, vias 0 -> 1
- net +5V: track 0.00 -> 33.7 mm, vias 0 -> 2
- net /MikrokontrolerAtmega/uC_RST: track 0.00 -> 32.6 mm
- net +3V3: track 0.00 -> 26.2 mm, vias 0 -> 2
- net /MikrokontrolerAtmega/uC_GPIO3: track 0.00 -> 13.8 mm, vias 0 -> 1
- net /MikrokontrolerAtmega/RTC_SCL: track 0.00 -> 12.0 mm, vias 0 -> 1
- net /MikrokontrolerAtmega/uC_GPIO2: track 0.00 -> 11.5 mm, vias 0 -> 1
- net /MikrokontrolerAtmega/uC_GPIO0: track 0.00 -> 11.1 mm, vias 0 -> 1
- net Net-(F1-Pad2): track 0.00 -> 11.0 mm
- net /MikrokontrolerAtmega/uC_GPIO1: track 0.00 -> 10.4 mm, vias 0 -> 1
- net /MikrokontrolerAtmega/RTC_SDA: track 0.00 -> 9.94 mm
- net Net-(C20-Pad2): track 0.00 -> 6.04 mm
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
Commit message: layout2
Parts:
- R1: moved to B.Cu
- moved H4 1.17 mm to (17.5, 15.4)
- moved H3 0.57 mm to (17.5, 79.9)
- moved H2 0.36 mm to (114.6, 79.6)
- moved H1 0.28 mm to (114.6, 15.1)
- moved R7 0.25 mm to (68.2, 40.9)
Connections:
- C10 pad 1: +3V3 -> +5V
Routing:
- net +5V: track 33.7 -> 319.5 mm, vias 2 -> 11
- net +3V3: track 26.2 -> 187.9 mm, vias 2 -> 5
- net /MikrokontrolerAtmega/uC_RST: track 32.6 -> 103.6 mm, vias 0 -> 2
- net /Moduł WiFi/ESP_RST: track 0.00 -> 69.9 mm
- net /MikrokontrolerAtmega/LED_DATA: track 0.00 -> 52.5 mm, vias 0 -> 1
- net /MikrokontrolerAtmega/ESP_RX_HIGH: track 0.00 -> 47.3 mm, vias 0 -> 1
- net /Sensory/PIR_OUT: track 0.00 -> 37.8 mm, vias 0 -> 1
- net /MikrokontrolerAtmega/ESP_TX_HIGH: track 0.00 -> 37.4 mm, vias 0 -> 1
- net /Moduł WiFi/ESP_TX: track 0.00 -> 37.1 mm, vias 0 -> 1
- net /MikrokontrolerAtmega/uC_MISO: track 48.3 -> 84.1 mm
- net /MikrokontrolerAtmega/DHT22_DATA: track 0.00 -> 33.1 mm
- net /Moduł WiFi/ESP_GPIO0: track 0.00 -> 33.1 mm
- net GND: track 0.00 -> 28.1 mm, vias 0 -> 6
- net Net-(RV1-Pad2): track 0.00 -> 21.3 mm, vias 0 -> 1
- net /Moduł WiFi/ESP_RX: track 0.00 -> 16.9 mm
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- added copper zone on B.Cu, net GND
- added copper zone on F.Cu, net GND

Commit message: layout3
Parts:
- moved RV1 1.91 mm to (68.6, 70.5)
- moved R4 1.40 mm to (108.6, 78.0)
- moved C19 1.28 mm to (100.2, 78.1)
- moved SW1 1.02 mm to (97.0, 75.8)
- moved R5 0.85 mm to (92.1, 78.7)
Routing:
- net /MikrokontrolerAtmega/LIGHT_SENSOR_OUT: track 5.34 -> 8.15 mm
- net Net-(RV1-Pad2): track 21.3 -> 19.4 mm
- net /MikrokontrolerAtmega/uC_RST: track 103.6 -> 102.6 mm

Commit message: l
Parts:
- C15, C16, C20, C21: footprint Capacitor_SMD:C_1206_3216Metric_Pad1.42x1.75mm_HandSolder -> Capacitor_SMD:C_0603_1608Metric_Pad1.05x0.95mm_HandSolder
- R1, R10, R11, R12, R13, R2, R3, R4, R5, R6, R7, R8, R9: footprint Resistor_SMD:R_1206_3216Metric_Pad1.42x1.75mm_HandSolder -> Resistor_SMD:R_0603_1608Metric_Pad1.05x0.95mm_HandSolder
- moved C14 1.20 mm to (30.5, 78.2)
- moved R8 1.20 mm to (23.2, 78.2)
- moved R9 1.20 mm to (38.5, 78.2)
- moved SW2 1.20 mm to (27.1, 75.7)
- moved J1 1.02 mm to (104.5, 16.0)
- moved J2 0.63 mm to (18.4, 25.4)
- moved C22 0.38 mm to (38.5, 74.3)
Routing:
- net Net-(C16-Pad1): track 16.3 -> 21.7 mm
- net Net-(C15-Pad2): track 13.1 -> 18.4 mm
- net +5V: track 319.5 -> 322.8 mm
- net /Moduł WiFi/ESP_RST: track 69.9 -> 67.6 mm
- net /MikrokontrolerAtmega/RTC_SCL: track 12.0 -> 13.8 mm
- net /MikrokontrolerAtmega/RTC_SDA: track 9.94 -> 10.8 mm
- net Net-(R5-Pad1): track 11.3 -> 12.0 mm
- net /MikrokontrolerAtmega/uC_RST: track 102.6 -> 103.2 mm
- net Net-(R9-Pad1): track 11.6 -> 12.2 mm
- net Net-(D2-Pad2): track 3.38 -> 3.99 mm
- net Net-(D1-Pad2): track 3.38 -> 3.99 mm
- net Net-(C21-Pad1): track 5.79 -> 6.40 mm
- net Net-(C20-Pad2): track 6.04 -> 6.66 mm
- net /Moduł WiFi/ESP_TX: track 37.1 -> 37.7 mm
- net /MikrokontrolerAtmega/ESP_TX_HIGH: track 37.4 -> 38.0 mm
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
Commit message: ll
Parts:
- moved BT1 6.00 mm to (90.8, 35.9)
- moved C10 6.00 mm to (50.6, 66.4)
- moved C14 6.00 mm to (30.5, 72.2)
- moved C17 6.00 mm to (80.6, 66.4)
- moved C19 6.00 mm to (100.2, 72.1)
- moved C22 6.00 mm to (38.5, 68.3)
- moved D3 6.00 mm to (104.1, 64.5)
- moved D4 6.00 mm to (26.0, 64.5)
- moved H2 6.00 mm to (114.6, 73.6)
- moved H3 6.00 mm to (17.5, 73.9)
- moved J3 6.00 mm to (77.5, 71.5)
- moved J4 6.00 mm to (64.4, 71.5)
- moved J5 6.00 mm to (47.6, 71.5)
- moved J6 6.00 mm to (109.2, 44.8)
- moved R4 6.00 mm to (108.6, 72.0)
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Routing:
- net /MikrokontrolerAtmega/uC_MISO: track 84.1 -> 45.8 mm
- net +5V: track 322.8 -> 314.6 mm
- net GND: track 28.1 -> 20.4 mm
- net /Sensory/PIR_OUT: track 37.8 -> 31.9 mm
- net Net-(RV1-Pad2): track 19.4 -> 14.1 mm
- net /MikrokontrolerAtmega/uC_SCK: track 46.4 -> 43.9 mm
- net /MikrokontrolerAtmega/uC_MOSI: track 48.3 -> 50.8 mm
- net Net-(BT1-Pad1): track 41.7 -> 39.2 mm
- net /MikrokontrolerAtmega/uC_RST: track 103.2 -> 101.2 mm
- net /MikrokontrolerAtmega/DHT22_DATA: track 33.1 -> 32.5 mm

Commit message: layout4
Parts:
- added R14: 10k, Resistor_SMD:R_0603_1608Metric_Pad1.05x0.95mm_HandSolder, F.Cu at (37.5, 33.1)
- C1: moved to B.Cu
- C12: moved to F.Cu
- F1: footprint Fuse:Fuseholder_Cylinder-5x20mm_Schurter_0031_8201_Horizontal_Open -> Fuse:Fuse_Littelfuse_372_D8.50mm
- J2: value Input_Supply+12V -> Input_Supply+5V
- J6: value AVR-ISP-10 -> AVR-ISP-6; footprint Connector_IDC:IDC-Header_2x05_P2.54mm_Vertical -> Connector_IDC:IDC-Header_2x03_P2.54mm_Vertical
- moved U1 74.1 mm to (30.4, 22.2), turned to 0 degrees
- moved J1 70.4 mm to (34.2, 16.0)
- moved R1 68.5 mm to (32.9, 23.5), turned to 270 degrees
- moved C1 59.2 mm to (41.1, 24.9)
- moved J6 24.4 mm to (95.5, 24.6), turned to 180 degrees
- moved J7 13.3 mm to (70.7, 62.0), turned to 90 degrees
- moved R4 12.7 mm to (96.8, 67.2)
- moved R5 11.9 mm to (80.1, 72.3)
- moved SW1 10.7 mm to (86.4, 69.8)
- moved C19 10.6 mm to (89.6, 72.1)
- moved D3 10.5 mm to (93.6, 64.6)
- moved H1 10.0 mm to (104.6, 15.1)
- moved H2 10.0 mm to (104.6, 73.6)
- moved C12 8.52 mm to (22.2, 39.0), turned to 90 degrees
- moved J3 7.86 mm to (69.6, 71.5)
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Connections:
- F1 pad 2: Net-(F1-Pad2) -> +5VA
- J1 pad 1: Net-(J1-Pad1) -> GND
- J1 pad 3: Net-(J1-Pad3) -> +5VA
- J2 pad 1: Net-(F1-Pad2) -> +5VA
- J6 pad 1: /MikrokontrolerAtmega/uC_MOSI -> /MikrokontrolerAtmega/uC_MISO
- J6 pad 3: Net-(J6-Pad3) -> /MikrokontrolerAtmega/uC_SCK
- J6 pad 4: GND -> /MikrokontrolerAtmega/uC_MOSI
- SW3 pad 1: +3V3 -> /Moduł WiFi/ESP_GPIO2
- SW3 pad 3: Net-(SW3-Pad3) -> GND
- SW4 pad 1: GND -> /Moduł WiFi/ESP_GPIO2
- SW4 pad 3: Net-(SW4-Pad3) -> GND
Routing:
- net /Moduł WiFi/ESP_GPIO2: track 0.00 -> 55.4 mm, vias 0 -> 1
- net /MikrokontrolerAtmega/uC_MOSI: track 50.8 -> 80.7 mm, vias 1 -> 0
- net +5VA: track 0.00 -> 21.4 mm
- net /MikrokontrolerAtmega/uC_GPIO3: track 13.8 -> 32.7 mm
- net +5V: track 314.6 -> 298.0 mm
- net /MikrokontrolerAtmega/uC_GPIO2: track 11.5 -> 27.0 mm
- net /MikrokontrolerAtmega/uC_RST: track 101.2 -> 115.1 mm, vias 2 -> 1
- net /MikrokontrolerAtmega/uC_GPIO1: track 10.4 -> 22.5 mm
- net /MikrokontrolerAtmega/uC_MISO: track 45.8 -> 57.6 mm, vias 0 -> 1
- net Net-(F1-Pad2): track 11.0 -> 0.00 mm
- net /MikrokontrolerAtmega/uC_SCK: track 43.9 -> 54.7 mm
- net GND: track 20.4 -> 30.9 mm, vias 6 -> 4
- net /MikrokontrolerAtmega/uC_GPIO0: track 11.1 -> 20.2 mm
- net /MikrokontrolerAtmega/DHT22_DATA: track 32.5 -> 23.9 mm
- net +3V3: track 188.4 -> 182.2 mm, vias 5 -> 8
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- added copper zone on B.Cu, net +5VA
- added copper zone on F.Cu, net +5VA
