File: PONG_Display/PONG_Display.kicad_pcb (KiCad board)
At the start: 2 copper layers, 68 parts, among them J1 LED_Display_Conn, J2 Input_Supply+5V, J3 DHT22_Conn, J4 LightSensor_Conn, J5 PIR_Sensor_Conn, J6 AVR-ISP-6, J7 Conn_01x04, J8 ESP_Conn, J9 ESP_Prog_Conn, Q1 BSS138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

Commit message: layout5
Other:
- board text added: "GPIO 0"
- board text added: "GPIO 1"
- board text added: "GPIO 2"
- board text added: "GPIO 3"
Changed lines of the file:
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@@
   (general
     (thickness 1.6)
-    (drawings 38)
+    (drawings 42)
     (tracks 542)
     (zones 0)
@@
   )
   (setup
-    (last_trace_width 1)
+    (last_trace_width 0.25)
     (user_trace_width 0.3)
     (user_trace_width 0.5)
@@
     )
   )
+  (gr_text "GPIO 3" (at 78.105 57.15 90) (layer F.SilkS)
+    (effects (font (size 1 1) (thickness 0.15)))
+  )
+  (gr_text "GPIO 2" (at 75.565 57.15 90) (layer F.SilkS)
+    (effects (font (size 1 1) (thickness 0.15)))
+  )
+  (gr_text "GPIO 1" (at 73.025 57.15 90) (layer F.SilkS)
+    (effects (font (size 1 1) (thickness 0.15)))
+  )
+  (gr_text "GPIO 0" (at 70.485 57.15 90) (layer F.SilkS)
+    (effects (font (size 1 1) (thickness 0.15)))
+  )
   (gr_text GND (at 21.0185 46.1645) (layer F.SilkS)
     (effects (font (size 1 1) (thickness 0.15)))
@@
   (segment (start 63.825 65.461) (end 64.643 64.643) (width 0.5) (layer B.Cu) (net 17) (status 20))
   (segment (start 63.825 71.47) (end 63.825 65.461) (width 0.5) (layer B.Cu) (net 17) (status 10))
-  (segment (start 17.78 25.4) (end 17.96 25.4) (width 2) (layer F.Cu) (net 48) (status 30))
   (segment (start 58.795 44.01) (end 58.795 46.095) (width 0.5) (layer F.Cu) (net 18) (status 10))
   (via (at 59.055 46.355) (size 0.8) (drill 0.4) (layers F.Cu B.Cu) (net 18))
@@
   (segment (start 36.83 52.705) (end 35.925 52.705) (width 0.5) (layer B.Cu) (net 47) (status 20))
   (segment (start 36.6525 57.15) (end 37.265 57.15) (width 1) (layer B.Cu) (net 47) (status 10))
+  (segment (start 17.78 25.4) (end 17.96 25.4) (width 2) (layer F.Cu) (net 48) (status 30))
   (segment (start 38.227 13.843) (end 26.162 13.843) (width 1) (layer F.Cu) (net 48))
   (segment (start 40.5765 16.1925) (end 38.227 13.843) (width 1) (layer F.Cu) (net 48))

Commit message: laayout6
Parts:
- J1: footprint TerminalBlock:TerminalBlock_bornier-3_P5.08mm -> TerminalBlock_RND:TerminalBlock_RND_205-00002_1x03_P5.00mm_Horizontal
- J2: footprint TerminalBlock:TerminalBlock_bornier-2_P5.08mm -> TerminalBlock_RND:TerminalBlock_RND_205-00001_1x02_P5.00mm_Horizontal
- J4: footprint TerminalBlock_Phoenix:TerminalBlock_Phoenix_PT-1,5-2-3.5-H_1x02_P3.50mm_Horizontal -> TerminalBlock_Phoenix:TerminalBlock_Phoenix_PT-1,5-3-3.5-H_1x03_P3.50mm_Horizontal
- moved J4 3.81 mm to (56.5, 71.5)
- moved J5 3.17 mm to (44.5, 71.5)
- moved C1 1.09 mm to (40.6, 27.3)
- moved U1 1.08 mm to (30.4, 24.8)
- moved J3 1.02 mm to (68.6, 71.5)
- moved R1 0.95 mm to (32.9, 26.0)
- moved J2 0.64 mm to (18.4, 26.0)
Routing:
- net +5V: track 298.6 -> 296.2 mm
- net /Sensory/PIR_OUT: track 31.9 -> 34.0 mm
- net /MikrokontrolerAtmega/LIGHT_SENSOR_OUT: track 7.17 -> 8.74 mm
- net Net-(R1-Pad1): track 2.85 -> 1.98 mm
- net /Wyswietlacz LED/LED_DATA_ISO: track 14.6 -> 15.2 mm
- net +5VA: track 20.7 -> 20.6 mm, vias 35 -> 44
- net (no net): vias 0 -> 1

Commit message: layout7
Routing:
- net +5V: track 296.2 -> 294.8 mm
- net /Moduł WiFi/ESP_GPIO2: track 55.4 -> 54.4 mm
- net Net-(R1-Pad1): track 1.98 -> 2.70 mm
Other:
- board outline added: 95.2 x 66.4 mm

Commit message: layout8
Parts:
- added L1: 10u, Inductor_SMD:L_1008_2520Metric, F.Cu at (73.4, 47.6)
- added REF**: L_Axial_L7.0mm_D3.3mm_P5.08mm_Vertical_Fastron_MICC, Inductor_THT:L_Axial_L7.0mm_D3.3mm_P5.08mm_Vertical_Fastron_MICC, F.Cu at (73.6, 50.1)
- moved C10 5.59 mm to (45.0, 67.0), turned to 0 degrees
Connections:
- J5 pad 1: GND -> +5V
- J5 pad 3: +5V -> GND
Routing:
- net +5V: track 294.8 -> 306.7 mm
- net Net-(C8-Pad1): track 3.51 -> 10.1 mm, vias 1 -> 2
- net /MikrokontrolerAtmega/uC_RST: track 115.1 -> 109.7 mm
- net /Sensory/PIR_OUT: track 34.0 -> 32.2 mm
- net /Moduł WiFi/ESP_GPIO2: track 54.4 -> 53.0 mm
- net /MikrokontrolerAtmega/uC_GPIO3: track 32.7 -> 33.6 mm
- net /Moduł WiFi/ESP_TX: track 36.0 -> 35.1 mm
- net GND: track 25.8 -> 26.7 mm, vias 4 -> 38
- net /MikrokontrolerAtmega/uC_SCK: track 54.7 -> 55.3 mm
- net (no net): vias 1 -> 0
Other:
- board text added: "Mański, Mikos, Pliszka, Sokołowski, Tyburski"
- board text added: "PONG_Display v1.0.0"
- board text added: "Projekt grupowy 2020/21 WETI PG"
- board text added: "Reset Atmega"
- board text removed: "Reset atmega"

Commit message: layout8
Parts:
- removed REF**: L_Axial_L7.0mm_D3.3mm_P5.08mm_Vertical_Fastron_MICC, Inductor_THT:L_Axial_L7.0mm_D3.3mm_P5.08mm_Vertical_Fastron_MICC
- added SW5: SW_Push_SPDT, LIB_PONG_Display:SPDT_switch, F.Cu at (79.2, 31.2)
- added SW6: SW_Push_SPDT, LIB_PONG_Display:SPDT_switch, F.Cu at (15.5, 62.7)
- C8: moved to F.Cu
- moved C18 22.7 mm to (23.6, 63.0), turned to 90 degrees
- moved J9 15.2 mm to (19.3, 53.3), turned to 180 degrees
- moved C8 1.17 mm to (68.1, 49.3)
- moved L1 0.74 mm to (74.2, 47.6)
- moved C12 0.63 mm to (22.9, 38.9)
Connections:
- J6 pad 2: +5V -> Net-(J6-Pad2)
- J9 pad 1: +3V3 -> Net-(J9-Pad1)
Routing:
- net +5V: track 306.7 -> 282.9 mm
- net Net-(J6-Pad2): track 0.00 -> 19.4 mm
- net Net-(J9-Pad1): track 0.00 -> 11.6 mm
- net /Moduł WiFi/ESP_RX: track 17.7 -> 26.7 mm
- net GND: track 26.7 -> 30.1 mm, vias 38 -> 39
- net /Moduł WiFi/ESP_TX: track 35.1 -> 31.8 mm
- net Net-(BT1-Pad1): track 39.2 -> 36.3 mm
- net Net-(C8-Pad1): track 10.1 -> 8.13 mm, vias 2 -> 0
- net /MikrokontrolerAtmega/ESP_RX_HIGH: track 47.6 -> 47.0 mm
Other:
- board text added: "Wył."
- board text added: "Wł."
- board text added: "Zas. z prog."
