File: PONG_Display/PONG_Display.kicad_pcb (KiCad board)
At the start: 2 copper layers, 95.2 x 66.4 mm, 71 parts, among them J1 LED_Display_Conn, J2 Input_Supply+5V, J3 DHT22_Conn, J4 LightSensor_Conn, J5 PIR_Sensor_Conn, J6 AVR-ISP-6, J7 Conn_01x04, J8 ESP_Conn, J9 ESP_Prog_Conn, Q1 BSS138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

Commit message: Layout 11
Parts:
- D1, D2: footprint Diode_SMD:D_1206_3216Metric_Pad1.42x1.75mm_HandSolder -> Diode_SMD:D_0805_2012Metric_Pad1.15x1.40mm_HandSolder

Commit message: layout 12
Routing:
- net /MikrokontrolerAtmega/LED_DATA: track 52.1 -> 42.6 mm
- net GND: track 30.1 -> 25.4 mm
- net +5V: track 283.7 -> 282.8 mm
- net +3V3: track 170.5 -> 169.6 mm

Commit message: layout 11
Parts:
- C11, C7: moved to F.Cu
- turned C7 to 270 degrees
Routing:
- net +5V: track 282.8 -> 280.0 mm, vias 9 -> 7
- net GND: track 25.4 -> 26.9 mm, vias 41 -> 42
