File: PONG_Display/PONG_Display_z_przelotkami.kicad_pcb (KiCad board)
At the start: 2 copper layers, 68 parts, among them J1 LED_Display_Conn, J2 Input_Supply+5V, J3 DHT22_Conn, J4 LightSensor_Conn, J5 PIR_Sensor_Conn, J6 AVR-ISP-6, J7 Conn_01x04, J8 ESP_Conn, J9 ESP_Prog_Conn, Q1 BSS138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

Commit message: layout5
Routing:
- net /MikrokontrolerAtmega/ESP_RX_HIGH: track 47.6 -> 47.1 mm
- net GND: vias 4 -> 325
- net (no net): vias 0 -> 1
