File: PONG_Pcb/PONG_Display.kicad_pcb (KiCad board)
At the start: 2 copper layers, 95.2 x 66.4 mm, 71 parts, among them J1 LED_Display_Conn, J2 Input_Supply+5V, J3 DHT22_Conn, J4 LightSensor_Conn, J5 PIR_Sensor_Conn, J6 AVR-ISP-6, J7 Conn_01x04, J8 ESP_Conn, J9 ESP_Prog_Conn, Q1 BSS138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

Commit message: Drobne poprawki
Parts:
- removed SW6: SW_Push_SPDT, LIB_PONG_Display:SPDT_switch
- added D5: GREEN_LED, Diode_SMD:D_0805_2012Metric_Pad1.15x1.40mm_HandSolder, F.Cu at (19.3, 69.8)
- added R15: 5R1, Resistor_SMD:R_0603_1608Metric_Pad1.05x0.95mm_HandSolder, F.Cu at (23.9, 69.2)
- moved SW4 38.5 mm to (15.5, 62.7), turned to 90 degrees
- moved R14 7.43 mm to (30.1, 32.3), turned to 180 degrees
Connections:
- J9 pad 1: Net-(J9-Pad1) -> +3V3
- R14 pad 2: /Moduł WiFi/ESP_GPIO2 -> Net-(R14-Pad2)
- SW3 pad 1: /Moduł WiFi/ESP_GPIO2 -> Net-(R14-Pad2)
- SW4 pad 1: /Moduł WiFi/ESP_GPIO2 -> Net-(R14-Pad2)
Routing:
- net Net-(R14-Pad2): track 0.00 -> 46.3 mm
- net /Moduł WiFi/ESP_GPIO2: track 53.0 -> 32.2 mm
- net Net-(J9-Pad1): track 11.6 -> 0.00 mm
- net Net-(D5-Pad2): track 0.00 -> 3.64 mm
- net /Moduł WiFi/ESP_GPIO0: track 30.0 -> 27.9 mm
- net /Moduł WiFi/ESP_TX: track 31.4 -> 30.2 mm
- net +3V3: track 169.6 -> 168.9 mm
Other:
- board text added: "+3.3V"
- board text added: "Programowanie"
- board text added: "WiFi"
- board text removed: "3.3V"

Commit message: Pliki produkcyjne
Parts:
- C13, C20, C21, C22, C3, R9: moved to F.Cu
- moved C3 32.2 mm to (50.8, 15.0)
- moved C5 30.7 mm to (57.4, 25.7), turned to 270 degrees
- moved U2 30.5 mm to (52.1, 20.8)
- moved C4 30.5 mm to (52.1, 27.9)
- moved D1 11.2 mm to (64.5, 22.9)
- moved D2 11.2 mm to (69.6, 22.9)
- moved R2 11.2 mm to (64.5, 18.0)
- moved R3 11.2 mm to (69.6, 18.0)
- moved C13 8.73 mm to (59.4, 20.3)
- moved C2 8.39 mm to (77.0, 20.1)
- moved C10 2.60 mm to (47.5, 66.3)
- moved R5 2.16 mm to (82.3, 72.3)
- moved C6 1.33 mm to (62.0, 48.3)
- moved R1 0.89 mm to (32.9, 26.9)
- moved U1 0.89 mm to (30.4, 25.7)
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Routing:
- net +3V3: track 168.9 -> 143.4 mm, vias 8 -> 7
- net +5V: track 280.0 -> 287.5 mm, vias 7 -> 5
- net GND: track 26.9 -> 22.7 mm
- net /Moduł WiFi/ESP_RST: track 62.1 -> 65.5 mm
- net +5VA: track 20.6 -> 23.7 mm
- net /Wyswietlacz LED/LED_DATA_ISO: track 15.2 -> 17.6 mm
- net Net-(R5-Pad1): track 13.2 -> 11.1 mm
- net /Moduł WiFi/ESP_TX: track 30.2 -> 31.0 mm
- net Net-(BT1-Pad1): track 36.3 -> 37.0 mm
Other:
- board text added: "."
- board text added: "MISO"
- board text added: "MOSI"
- board text added: "RST"
- board text added: "SCK"
