File: PONG_Pcb/PONG_Display.kicad_pcb (KiCad board)
At the start: 2 copper layers, 95.2 x 66.4 mm, 74 parts, among them J1 LED_Display_Conn, J2 Input_Supply+5V, J3 DHT22_Conn, J4 LightSensor_Conn, J5 PIR_Sensor_Conn, J6 AVR-ISP-6, J7 Conn_01x04, J8 ESP_Conn, J9 ESP_Prog_Conn, Q1 BSS138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

Commit message: Ostatnia wersja
Parts:
- added TP1: TestPoint, TestPoint:TestPoint_Loop_D1.80mm_Drill1.0mm_Beaded, F.Cu at (70.1, 37.8)
- added TP2: TestPoint, TestPoint:TestPoint_Loop_D1.80mm_Drill1.0mm_Beaded, F.Cu at (77.0, 40.9)
- added TP3: TestPoint, TestPoint:TestPoint_Loop_D1.80mm_Drill1.0mm_Beaded, F.Cu at (79.8, 66.3)
- added TP4: TestPoint, TestPoint:TestPoint_Loop_D1.80mm_Drill1.0mm_Beaded, F.Cu at (18.8, 39.1)
- added TP5: TestPoint, TestPoint:TestPoint_Loop_D1.80mm_Drill1.0mm_Beaded, F.Cu at (39.6, 37.3)
- D6: footprint Diode_THT:D_DO-41_SOD81_P10.16mm_Horizontal -> Diode_SMD:D_SMC-RM10_Universal_Handsoldering
- moved D6 4.75 mm to (44.2, 16.0)
- moved C5 2.05 mm to (62.0, 25.4)
- moved U2 1.80 mm to (56.4, 20.1)
- moved C3 1.78 mm to (55.1, 14.5)
- moved R7 1.14 mm to (67.1, 40.9)
- moved C14 0.35 mm to (30.5, 71.9)
Routing:
- net /MikrokontrolerAtmega/RTC_SDA: track 10.8 -> 21.2 mm, vias 0 -> 1
- net /MikrokontrolerAtmega/DHT22_DATA: track 23.5 -> 33.3 mm
- net /Moduł WiFi/ESP_TX: track 31.0 -> 38.7 mm, vias 1 -> 2
- net /Moduł WiFi/ESP_RX: track 26.7 -> 31.2 mm
- net +5V: track 287.0 -> 290.9 mm
- net /MikrokontrolerAtmega/RTC_SCL: track 13.8 -> 16.4 mm
- net Net-(C8-Pad1): track 6.38 -> 7.18 mm
- net /MikrokontrolerAtmega/uC_RST: track 107.3 -> 106.5 mm
- net +3V3: track 147.0 -> 146.4 mm
- net Net-(R14-Pad2): track 46.3 -> 46.8 mm
- net GND: vias 45 -> 44

Commit message: poprawki koncowe
Parts:
- removed C1: 100n, Capacitor_SMD:C_0603_1608Metric_Pad1.05x0.95mm_HandSolder
- removed R16: 470R, Resistor_SMD:R_0603_1608Metric_Pad1.05x0.95mm_HandSolder
- removed U1: PC817, Package_DIP:DIP-4_W7.62mm
- D5: value GREEN_LED -> BLUE_LED
- R1: value 180R -> 10k
- R15, R3: value 5R1 -> 330R
- moved R1 31.4 mm to (19.3, 56.3), turned to 0 degrees
- moved C15 6.01 mm to (52.5, 54.6), turned to 270 degrees
- moved C16 5.95 mm to (52.5, 61.8), turned to 270 degrees
- moved Y1 4.70 mm to (48.0, 55.9)
- moved J1 0.13 mm to (34.2, 17.5)
Connections:
- J1 pad 2: /Wyswietlacz LED/LED_DATA_ISO -> /MikrokontrolerAtmega/LED_DATA
- R1 pad 1: Net-(R1-Pad1) -> +3V3
- R1 pad 2: /MikrokontrolerAtmega/LED_DATA -> Net-(R1-Pad2)
- SW4 pad 1: Net-(R14-Pad2) -> Net-(R1-Pad2)
Routing:
- net Net-(R14-Pad2): track 46.8 -> 4.31 mm
- net +5V: track 290.9 -> 280.3 mm
- net Net-(R1-Pad2): track 0.00 -> 10.5 mm
- net /Wyswietlacz LED/LED_DATA_ISO: track 10.4 -> 0.00 mm
- net /MikrokontrolerAtmega/LED_DATA: track 44.4 -> 52.3 mm
- net Net-(C1-Pad1): track 6.56 -> 0.00 mm
- net Net-(C16-Pad1): track 21.7 -> 16.7 mm
- net Net-(C15-Pad2): track 18.4 -> 14.2 mm
- net +3V3: track 146.4 -> 149.7 mm
- net Net-(R1-Pad1): track 2.45 -> 0.00 mm
- net GND: vias 44 -> 43
