File: PONG_Pcb/PONG_Display.sch (KiCad schematic (older format))
At the start: 4 parts

Commit message: Drobne poprawki
Other:
- note removed: "1)wybór 5V czy 12V\n2)Poziomy logiczne TX i RX\n3)stany na pinach -\n> czy programowo\n4)Jakie piny na GPIO uC\n5)GPIO od ESP czy potrzebne \n6)Jaka prędkość I2C \n->rezystory 2k/10k\n7)Przypisać piny ESP"
- note removed: "To do:\n"
Changed lines of the file:
@@
 F7 "ESP_TX_HIGH" I L 8400 2500 50
 $EndSheet
-Text Notes 950  1150 0    197  Italic 39
-To do:\n
-Text Notes 700  2500 0    79   ~ 0
-1)wybór 5V czy 12V\n2)Poziomy logiczne TX i RX\n3)stany na pinach -\n> czy programowo\n4)Jakie piny na GPIO uC\n5)GPIO od ESP czy potrzebne \n6)Jaka prędkość I2C \n->rezystory 2k/10k\n7)Przypisać piny ESP
 $EndSCHEMATC

Commit message: poprawki koncowe
Changed lines of the file:
@@
 $Descr A4 11693 8268
 encoding utf-8
-Sheet 1 6
+Sheet 1 5
 Title ""
 Date ""
@@
 $EndDescr
 $Sheet
-S 8800 4400 900  1250
-U 5E80C133
-F0 "Wyswietlacz LED" 50
-F1 "LED.sch" 50
-F2 "LED_DATA" I L 8800 4900 50
-$EndSheet
-$Sheet
-S 2650 4050 1100 1150
+S 4350 6200 1100 1150
 U 5E80B14C
 F0 "Power Supply" 50
@@
 $EndSheet
 Wire Wire Line
-	7200 2350 8400 2350
+	6750 3350 7950 3350
 Wire Wire Line
-	7200 2500 8400 2500
+	6750 3500 7950 3500
 Wire Wire Line
-	3850 2650 5400 2650
+	3400 3650 4950 3650
 Wire Wire Line
-	5400 2800 3850 2800
-Wire Wire Line
-	7200 3300 8000 3300
-Wire Wire Line
-	8000 3300 8000 4900
-Wire Wire Line
-	8000 4900 8800 4900
+	4950 3800 3400 3800
 $Comp
 L Mechanical:MountingHole H?
@@
 $EndComp
 Wire Wire Line
-	5400 2500 3850 2500
+	4950 3500 3400 3500
 Text Notes 7600 7500 0    50   ~ 0
 Wyświetlacz ping-pong - schemat główny
 $Sheet
-S 2650 1950 1200 1200
+S 2200 2950 1200 1200
 U 5E80B6DE
 F0 "Sensory" 50
 F1 "sensors.sch" 50
-F2 "DHT22_DATA" I R 3850 2650 50
-F3 "LIGHT_SENSOR_OUT" I R 3850 2500 50
-F4 "PIR_OUT" I R 3850 2800 50
+F2 "DHT22_DATA" I R 3400 3650 50
+F3 "LIGHT_SENSOR_OUT" I R 3400 3500 50
+F4 "PIR_OUT" I R 3400 3800 50
 $EndSheet
 $Sheet
-S 5400 1900 1800 1500
+S 4950 2900 1800 1500
 U 5E80B18F
 F0 "MikrokontrolerAtmega" 50
 F1 "microcontroler.sch" 50
-F2 "LIGHT_SENSOR_OUT" I L 5400 2500 50
-F3 "PIR_SENSOR_OUT" I L 5400 2800 50
-F4 "DHT22_DATA" I L 5400 2650 50
-F5 "ESP_RST" I R 7200 2950 50
-F6 "LED_DATA" I R 7200 3300 50
-F7 "ESP_TX_HIGH" I R 7200 2500 50
-F8 "ESP_RX_HIGH" I R 7200 2350 50
+F2 "LIGHT_SENSOR_OUT" I L 4950 3500 50
+F3 "PIR_SENSOR_OUT" I L 4950 3800 50
+F4 "DHT22_DATA" I L 4950 3650 50
+F5 "ESP_RST" I R 6750 3950 50
+F6 "ESP_TX_HIGH" I R 6750 3500 50
+F7 "ESP_RX_HIGH" I R 6750 3350 50
 $EndSheet
 Wire Wire Line
-	7200 2950 8400 2950
+	6750 3950 7950 3950
 $Sheet
-S 8400 1950 1350 1500
+S 7950 2950 1350 1500
 U 5E80B1F8
 F0 "Moduł WiFi" 50
 F1 "esp.sch" 50
-F2 "ESP_RST" I L 8400 2950 50
-F3 "ESP_CH_PD" I L 8400 3100 50
-F4 "ESP_GPIO0" I L 8400 2650 50
-F5 "ESP_GPIO2" I L 8400 2800 50
-F6 "ESP_RX_HIGH" I L 8400 2350 50
-F7 "ESP_TX_HIGH" I L 8400 2500 50
+F2 "ESP_RST" I L 7950 3950 50
+F3 "ESP_RX_HIGH" I L 7950 3350 50
+F4 "ESP_TX_HIGH" I L 7950 3500 50
 $EndSheet
 $EndSCHEMATC
