File: PONG_Pcb/microcontroler.sch (KiCad schematic (older format))
At the start: 32 parts, among them J6 AVR-ISP-6, J7 Conn_01x04, SW1 SW_Push, SW5 SW_Push_SPDT, U3 ATmega328P-AU, U4 MCP79400, Y1 16MHz, Y2 32,768kHz

Commit message: Ostatnia wersja
Parts:
- added TP1, TP2: TestPoint, TestPoint:TestPoint_Loop_D1.80mm_Drill1.0mm_Beaded, symbol Connector:TestPoint
Connections:
- net RTC_SCL: now also TP1.1
- net RTC_SDA: now also TP2.1
Changed lines of the file:
@@
 Wire Wire Line
 	2050 6850 2300 6850
-Wire Wire Line
-	2050 6750 2300 6750
-Wire Wire Line
-	2050 6650 2300 6650
-Wire Wire Line
-	2050 6550 2300 6550
 Text Notes 7750 7500 0    50   ~ 0
 Schemat mikrokontrolera
@@
 $EndComp
 Wire Wire Line
-	8250 1700 8650 1700
+	7800 1700 8000 1700
 Wire Wire Line
 	9150 1800 8900 1800
@@
 Text Label 3550 2600 0    50   ~ 0
 uC_MOSI
-Text Label 2300 6550 0    50   ~ 0
+Text Label 2850 6550 0    50   ~ 0
 uC_MISO
-Text Label 2300 6650 0    50   ~ 0
+Text Label 2850 6650 0    50   ~ 0
 uC_MOSI
-Text Label 2300 6750 0    50   ~ 0
+Text Label 2850 6750 0    50   ~ 0
 uC_SCK
 Text Label 2300 6850 0    50   ~ 0
@@
 NoConn ~ 3400 4700
 NoConn ~ 9150 2000
-Text Label 8250 1700 2    50   ~ 0
+Text Label 7800 1700 2    50   ~ 0
 RTC_SCL
-Text Label 8250 1800 2    50   ~ 0
+Text Label 7800 1800 2    50   ~ 0
 RTC_SDA
 Text HLabel 3550 2400 2    50   Input ~ 0
@@
 	1550 6100 1550 6250
 NoConn ~ 2000 6200
+$Comp
+L Connector:TestPoint TP2
+U 1 1 5EC52676
+P 8250 1350
+F 0 "TP2" H 8308 1468 50  0000 L CNN
+F 1 "TestPoint" H 8308 1377 50  0000 L CNN
+F 2 "TestPoint:TestPoint_Loop_D1.80mm_Drill1.0mm_Beaded" H 8450 1350 50  0001 C CNN
+F 3 "~" H 8450 1350 50  0001 C CNN
+	1    8250 1350
+	1    0    0    -1
+$EndComp
+$Comp
+L Connector:TestPoint TP1
+U 1 1 5EC534E4
+P 8000 1100
+F 0 "TP1" H 8058 1218 50  0000 L CNN
+F 1 "TestPoint" H 8058 1127 50  0000 L CNN
+F 2 "TestPoint:TestPoint_Loop_D1.80mm_Drill1.0mm_Beaded" H 8200 1100 50  0001 C CNN
+F 3 "~" H 8200 1100 50  0001 C CNN
+	1    8000 1100
+	1    0    0    -1
+$EndComp
+Wire Wire Line
+	8250 1350 8250 1800
+Connection ~ 8250 1800
+Wire Wire Line
+	8250 1800 7800 1800
+Wire Wire Line
+	8000 1100 8000 1700
+Connection ~ 8000 1700
+Wire Wire Line
+	8000 1700 8650 1700
+Wire Wire Line
+	2050 6550 2850 6550
+Wire Wire Line
+	2050 6650 2850 6650
+Wire Wire Line
+	2050 6750 2850 6750
 $EndSCHEMATC

Commit message: poprawki koncowe
Parts:
- added J1: LED_Display_Conn, TerminalBlock_RND:TerminalBlock_RND_205-00002_1x03_P5.00mm_Horizontal, symbol Connector_Generic:Conn_01x03
- U3: symbol PONG_Display-rescue:ATmega328P-AU-MCU_Microchip_ATmega -> MCU_Microchip_ATmega:ATmega328P-AU
Connections:
- net GND: now also J1.1 (Pin_1)
- net LED_DATA: now also J1.2 (Pin_2)
- new net +5VA: J1.3 (Pin_3)
Other:
- note added: "Złącze wyjścia na wyświetlacz"
Changed lines of the file:
@@
 $Descr A4 11693 8268
 encoding utf-8
-Sheet 5 6
+Sheet 4 5
 Title ""
 Date ""
@@
 Schemat mikrokontrolera
 $Comp
-L PONG_Display-rescue:ATmega328P-AU-MCU_Microchip_ATmega U3
+L MCU_Microchip_ATmega:ATmega328P-AU U3
 U 1 1 5E85008B
 P 2800 3500
@@
 Text Label 7800 1800 2    50   ~ 0
 RTC_SDA
-Text HLabel 3550 2400 2    50   Input ~ 0
-LED_DATA
 Wire Wire Line
 	3400 3800 6150 3800
-Wire Wire Line
-	3550 2400 3400 2400
 $Comp
 L power:+5V #PWR056
@@
 Wire Wire Line
 	2050 6750 2850 6750
+$Comp
+L Connector_Generic:Conn_01x03 J?
+U 1 1 600C6715
+P 9800 5050
+AR Path="/5E80CCDD/600C6715" Ref="J?"  Part="1"
+AR Path="/5E80C133/600C6715" Ref="J?"  Part="1"
+AR Path="/5E80B18F/600C6715" Ref="J1"  Part="1"
+F 0 "J1" H 9880 5092 50  0000 L CNN
+F 1 "LED_Display_Conn" H 9880 5001 50  0000 L CNN
+F 2 "TerminalBlock_RND:TerminalBlock_RND_205-00002_1x03_P5.00mm_Horizontal" H 9800 5050 50  0001 C CNN
+F 3 "~" H 9800 5050 50  0001 C CNN
+	1    9800 5050
+	1    0    0    1
+$EndComp
+Text Notes 9100 4300 0    50   ~ 0
+Złącze wyjścia na wyświetlacz
+Text Label 8900 5050 0    50   ~ 0
+LED_DATA
+Wire Wire Line
+	8900 5050 9600 5050
+$Comp
+L power:GND #PWR?
+U 1 1 600C671E
+P 9550 5350
+AR Path="/5E80C133/600C671E" Ref="#PWR?"  Part="1"
+AR Path="/5E80B18F/600C671E" Ref="#PWR0109"  Part="1"
+F 0 "#PWR0109" H 9550 5100 50  0001 C CNN
+F 1 "GND" H 9555 5177 50  0000 C CNN
+F 2 "" H 9550 5350 50  0001 C CNN
+F 3 "" H 9550 5350 50  0001 C CNN
+	1    9550 5350
+	1    0    0    -1
+$EndComp
+Wire Wire Line
+	9550 4750 9550 4950
+Wire Wire Line
+	9550 4950 9600 4950
+Wire Wire Line
+	9550 5350 9550 5150
+Wire Wire Line
+	9550 5150 9600 5150
+$Comp
+L power:+5VA #PWR?
+U 1 1 600C6728
+P 9550 4750
+AR Path="/5E80C133/600C6728" Ref="#PWR?"  Part="1"
+AR Path="/5E80B18F/600C6728" Ref="#PWR0110"  Part="1"
+F 0 "#PWR0110" H 9550 4600 50  0001 C CNN
+F 1 "+5VA" H 9565 4923 50  0000 C CNN
+F 2 "" H 9550 4750 50  0001 C CNN
+F 3 "" H 9550 4750 50  0001 C CNN
+	1    9550 4750
+	1    0    0    -1
+$EndComp
+Text Label 4250 2400 0    50   ~ 0
+LED_DATA
+Wire Wire Line
+	3400 2400 4250 2400
+Wire Notes Line
+	8500 4050 8500 6200
+Wire Notes Line
+	8500 6200 10950 6200
+Wire Notes Line
+	10950 6200 10950 4050
+Wire Notes Line
+	10950 4050 8500 4050
 $EndSCHEMATC
